File: 9v_iso/9v_iso.kicad_pcb (KiCad board)
At the start: 2 copper layers, 56 x 34 mm, 15 parts, among them J1 Conn_01x02, J2 Conn_01x02, J3 Conn_01x03, U1 ICZ_SINGLE

Commit message: Checkpoint.
Parts:
- removed JP1: SolderJumper_3_Open, Jumper:SolderJumper-3_P1.3mm_Open_RoundedPad1.0x1.5mm_NumberLabels
- J3: value Conn_01x03 -> DNI
- moved J3 1.27 mm to (73.7, 54.6)
Routing:
- net Net-(J3-Pad2): track 23.9 -> 18.3 mm
- net /Vin_filtered: track 42.2 -> 40.9 mm
Other:
- board text added: "ISOLATED 9V REV 1.0 MURGATROID HEAVY INDUSTRIES, LTD (C) 2022"
- board text added: "REMOTE ON/OFF"

Commit message: checkpoint
Parts:
- added R1: DNI/0, Resistor_SMD:R_0805_2012Metric_Pad1.20x1.40mm_HandSolder, F.Cu at (73.9, 59.7)
Connections:
- U1 pad 3: Net-(J3-Pad2) -> Net-(U1-Pad3)
Routing:
- net Net-(J3-Pad2): track 18.3 -> 5.83 mm
- net Net-(U1-Pad3): track 0.00 -> 12.4 mm, vias 0 -> 1
Other:
- board size 56 x 34 mm -> 60 x 38 mm
