File: projects/ddf_small_array/ddf_small_array.kicad_pcb (KiCad board)
At the start: 2 copper layers, 46 parts, among them J1 Conn_Coaxial, J2 Conn_Coaxial, J3 Conn_Coaxial, J4 Conn_Coaxial, J5 Conn_Coaxial, J6 RJ45_Shielded

Commit message: Checkpoint on new design.
Parts:
- removed C10, C11, C12, C13: C, Capacitor_SMD:C_0805_2012Metric_Pad1.18x1.45mm_HandSolder
- removed R10, R11, R12, R13, R14, R15, R7, R8, R9: R, Resistor_SMD:R_0805_2012Metric_Pad1.20x1.40mm_HandSolder
- added L5: L, Inductor_SMD:L_0805_2012Metric_Pad1.15x1.40mm_HandSolder, F.Cu at (103.6, 239.4)
- moved C2 382.3 mm to (249.4, 395.8)
- moved J3 365.8 mm to (410.0, 250.0)
- moved D3 362.3 mm to (401.2, 258.0)
- moved R3 348.2 mm to (401.8, 241.6)
- moved R5 335.1 mm to (369.4, 191.6)
- moved C6 330.5 mm to (234.8, 364.3)
- moved L3 330.3 mm to (233.0, 376.8)
- moved D5 314.6 mm to (371.9, 166.2)
- moved C3 310.8 mm to (401.2, 247.6)
- moved R2 307.2 mm to (238.4, 409.6)
- moved J2 290.1 mm to (249.5, 410.0)
- moved R6 282.9 mm to (383.2, 144.6)
- moved L4 282.3 mm to (399.0, 236.0)
- moved D7 276.6 mm to (377.0, 171.3)
- moved C7 268.0 mm to (407.5, 230.0)
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Connections:
- C2 pad 1: GND -> Net-(C2-Pad1)
- C4 pad 1: GND -> Net-(C4-Pad1)
- C4 pad 2: Net-(C2-Pad2) -> Net-(C4-Pad2)
- C5 pad 1: Net-(C5-Pad1) -> /NORTH
- C5 pad 2: Net-(C5-Pad2) -> GND
- C6 pad 1: GND -> /SOUTH
- C6 pad 2: Net-(C2-Pad2) -> GND
- C7 pad 1: Net-(C7-Pad1) -> /EAST
- C7 pad 2: Net-(C7-Pad2) -> GND
- C8 pad 1: GND -> /WEST
- C8 pad 2: Net-(C2-Pad2) -> GND
- C9 pad 1: /NORTH -> Net-(C9-Pad1)
- C9 pad 2: GND -> Net-(C9-Pad2)
- D1 pad 1: Net-(C1-Pad1) -> Net-(D1-Pad1)
- D1 pad 2: Net-(D1-Pad2) -> Net-(C1-Pad1)
- D2 pad 1: Net-(C3-Pad1) -> Net-(D2-Pad1)
- D2 pad 2: Net-(D2-Pad2) -> Net-(C2-Pad1)
- D3 pad 1: Net-(C5-Pad1) -> Net-(D3-Pad1)
- D3 pad 2: Net-(D3-Pad2) -> Net-(C3-Pad1)
- D4 pad 1: Net-(C7-Pad1) -> Net-(D4-Pad1)
- D4 pad 2: Net-(D4-Pad2) -> Net-(C4-Pad1)
- D5 pad 1: Net-(C13-Pad1) -> Net-(C9-Pad1)
- D5 pad 2: Net-(D1-Pad2) -> Net-(D1-Pad1)
- D6 pad 1: Net-(C13-Pad1) -> Net-(C9-Pad1)
- D6 pad 2: Net-(D2-Pad2) -> Net-(D2-Pad1)
- D7 pad 1: Net-(C13-Pad1) -> Net-(C9-Pad1)
- D7 pad 2: Net-(D3-Pad2) -> Net-(D3-Pad1)
- D8 pad 1: Net-(C13-Pad1) -> Net-(C9-Pad1)
- D8 pad 2: Net-(D4-Pad2) -> Net-(D4-Pad1)
- J2 pad 1: Net-(C3-Pad2) -> Net-(C2-Pad2)
- J3 pad 1: Net-(C5-Pad2) -> Net-(C3-Pad2)
- J4 pad 1: Net-(C7-Pad2) -> Net-(C4-Pad2)
- J5 pad 1: Net-(C13-Pad2) -> Net-(C9-Pad2)
- L1 pad 2: /NORTH -> Net-(C9-Pad1)
- L2 pad 1: Net-(L2-Pad1) -> Net-(C1-Pad1)
- L2 pad 2: /SOUTH -> /NORTH
- L3 pad 1: Net-(L3-Pad1) -> Net-(C2-Pad1)
- L3 pad 2: /EAST -> /SOUTH
- L4 pad 1: Net-(L4-Pad1) -> Net-(C3-Pad1)
- L4 pad 2: /WEST -> /EAST
- R2 pad 1: Net-(C3-Pad2) -> Net-(C2-Pad2)
- R3 pad 1: Net-(C5-Pad2) -> Net-(C3-Pad2)
- R4 pad 1: Net-(C7-Pad2) -> Net-(C4-Pad2)
- R5 pad 1: Net-(C1-Pad1) -> Net-(L1-Pad1)
- R5 pad 2: Net-(C2-Pad2) -> GND
- R6 pad 1: Net-(C3-Pad1) -> Net-(C9-Pad2)
- R6 pad 2: Net-(C2-Pad2) -> GND
Routing:
- added copper zone on F.Cu, net GND
Other:
- board outline added: 400 x 400 mm

Commit message: checkpoint; need to use em solver now.
Parts:
- added C10: C, Capacitor_SMD:C_0402_1005Metric_Pad0.74x0.62mm_HandSolder, F.Cu at (380.0, 120.8)
- added L6: L, Inductor_SMD:L_0402_1005Metric_Pad0.77x0.64mm_HandSolder, F.Cu at (378.2, 121.8)
- C1, C2, C3, C4, C5, C6, C7, C8, C9: footprint Capacitor_SMD:C_0805_2012Metric_Pad1.18x1.45mm_HandSolder -> Capacitor_SMD:C_0402_1005Metric
- D1, D2, D3, D4, D5, D6, D7, D8: footprint Diode_SMD:D_SOD-523 -> Diode_SMD:D_SOD-323
- L1, L2, L3, L4, L5: footprint Inductor_SMD:L_0805_2012Metric_Pad1.15x1.40mm_HandSolder -> Inductor_SMD:L_0402_1005Metric
- R1, R2, R3, R4, R5, R6: footprint Resistor_SMD:R_0805_2012Metric_Pad1.20x1.40mm_HandSolder -> Resistor_SMD:R_0402_1005Metric
- moved L1 172.8 mm to (257.6, 257.6), turned to 135 degrees
- moved C9 160.5 mm to (257.0, 243.0), turned to 45 degrees
- moved D8 154.4 mm to (240.0, 250.0), turned to 180 degrees
- moved D6 153.1 mm to (250.0, 260.0), turned to -90 degrees
- moved D5 142.5 mm to (250.0, 240.0), turned to 90 degrees
- moved D7 141.0 mm to (260.0, 250.0)
- moved R5 129.2 mm to (259.4, 259.4), turned to -45 degrees
- moved D2 54.4 mm to (250.0, 402.2), turned to -90 degrees
- moved C6 43.7 mm to (253.5, 403.8), turned to -90 degrees
- moved L3 32.6 mm to (252.0, 403.3)
- moved R6 26.1 mm to (380.7, 118.6), turned to 135 degrees
- moved C7 23.8 mm to (403.8, 253.5)
- moved C4 19.0 mm to (95.2, 250.0), turned to 180 degrees
- moved L4 16.6 mm to (403.3, 252.0), turned to -90 degrees
- moved C8 15.3 mm to (96.2, 246.5), turned to 180 degrees
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Connections:
- net /EAST renamed /E_BIAS_IN
- net /NORTH renamed /N_BIAS_IN
- net /SOUTH renamed /S_BIAS_IN
- net /WEST renamed /W_BIAS_IN
- net Net-(C1-Pad1) renamed /N_BIAS
- net Net-(C1-Pad2) renamed /N_ANT
- net Net-(C2-Pad1) renamed /S_BIAS
- net Net-(C2-Pad2) renamed /S_ANT
- net Net-(C3-Pad1) renamed /E_BIAS
- net Net-(C3-Pad2) renamed /E_ANT
- net Net-(C4-Pad1) renamed /W_BIAS
- net Net-(C4-Pad2) renamed /W_ANT
- net Net-(C9-Pad1) renamed /RF_COM
- net Net-(D1-Pad1) renamed /N_RF_TO_COM
- net Net-(D2-Pad1) renamed /S_RF_TO_COM
- net Net-(D3-Pad1) renamed /E_RF_TO_COM
- net Net-(D4-Pad1) renamed /W_RF_TO_COM
- J5 pad 1: Net-(C9-Pad2) -> /RF_OUT
- R6 pad 1: Net-(C9-Pad2) -> /RF_OUT
Routing:
- net Net-(C9-Pad2): track 0.00 -> 170.4 mm
- net /W_RF_TO_COM: track 0.00 -> 140.1 mm
- net /N_RF_TO_COM: track 0.00 -> 140.1 mm
- net /S_RF_TO_COM: track 0.00 -> 140.1 mm
- net /E_RF_TO_COM: track 0.00 -> 140.1 mm
- net /RF_COM: track 0.00 -> 55.5 mm
- net /RF_OUT: track 0.00 -> 9.52 mm
- net /S_ANT: track 0.00 -> 5.63 mm
- net /E_ANT: track 0.00 -> 5.63 mm
- net /W_ANT: track 0.00 -> 5.63 mm
- net /N_ANT: track 0.00 -> 5.63 mm
- net /W_BIAS: track 0.00 -> 2.53 mm
- net /S_BIAS: track 0.00 -> 2.53 mm
- net /N_BIAS: track 0.00 -> 2.53 mm
- net /E_BIAS: track 0.00 -> 2.53 mm
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- added copper zone on B.Cu, net GND
