File: projects/ddf_small_array/ddf_small_array.kicad_sch (KiCad schematic)
At the start: 46 parts, among them J1 Conn_Coaxial, J2 Conn_Coaxial, J3 Conn_Coaxial, J4 Conn_Coaxial, J5 Conn_Coaxial, J6 RJ45_Shielded

Commit message: Checkpoint on new design.
Parts:
- removed C5, C6, C7, C8: C, Capacitor_SMD:C_0805_2012Metric_Pad1.18x1.45mm_HandSolder, symbol Device:C
- removed L2: L, Inductor_SMD:L_0805_2012Metric_Pad1.15x1.40mm_HandSolder, symbol Device:L
- removed R10, R11, R12, R13, R14, R6, R7, R8, R9: R, Resistor_SMD:R_0805_2012Metric_Pad1.20x1.40mm_HandSolder, symbol Device:R
- added L1, L5: L, Inductor_SMD:L_0805_2012Metric_Pad1.15x1.40mm_HandSolder, symbol Device:L
- renumbered C9 to C5, C10 to C6, C11 to C7, C12 to C8, C13 to C9, L1 to L2, R15 to R6
Connections:
- net EAST: now also L4.2; no longer L3.2
- net GND: now also R5.2; no longer C2.1, C4.1
- net SOUTH: now also L3.2
- net WEST: now also L5.2; no longer L4.2
- net at C9.1, D5.1 (K), D6.1 (K)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: now also L1.2
- net at D5.2 (A): now also D1.1 (K); no longer D1.2 (A)
- net at D2.2 (A): now also C2.1, L3.1; no longer D6.2 (A)
- net at D4.1 (K): now also D8.2 (A)
- net at J4.1 (In), R4.1: now also C4.2
- net at L4.1: now also C3.1, D3.2 (A)
- net at D4.2 (A): now also C4.1, L5.1; no longer D8.2 (A)
- net at L2.1: now also C1.1, D1.2 (A)
- net at D2.1 (K): now also D6.2 (A); no longer C3.1
- net at D3.1 (K): now also D7.2 (A)
- net at J3.1 (In), R3.1: now also C3.2
- net at J2.1 (In), R2.1: now also C2.2; no longer C3.2
- new net: L1.1, R5.1

Commit message: checkpoint; need to use em solver now.
Parts:
- added C10: C, Capacitor_SMD:C_0402_1005Metric_Pad0.74x0.62mm_HandSolder, symbol Device:C
- added L6: L, Inductor_SMD:L_0402_1005Metric_Pad0.77x0.64mm_HandSolder, symbol Device:L
- C1, C2, C3, C4, C5, C6, C7, C8, C9: footprint Capacitor_SMD:C_0805_2012Metric_Pad1.18x1.45mm_HandSolder -> Capacitor_SMD:C_0402_1005Metric
- D1, D2, D3, D4, D5, D6, D7, D8: footprint Diode_SMD:D_SOD-523 -> Diode_SMD:D_SOD-323
- L1, L2, L3, L4, L5: footprint Inductor_SMD:L_0805_2012Metric_Pad1.15x1.40mm_HandSolder -> Inductor_SMD:L_0402_1005Metric
- R1, R2, R3, R4, R5, R6: footprint Resistor_SMD:R_0805_2012Metric_Pad1.20x1.40mm_HandSolder -> Resistor_SMD:R_0402_1005Metric
Connections:
- net GND: now also C10.2
- net RF_OUT: now reaches J5.1 (In), R6.1
- net RF_OUT: now also C10.1, L6.2; no longer C9.2
- net RF_COM: now reaches C9.1, D5.1 (K), D6.1 (K), D7.1 (K), D8.1 (K), L1.2
- net N_RF_TO_COM: now reaches D1.1 (K), D5.2 (A)
- net N_BIAS: now reaches C1.1, D1.2 (A), L2.1
- net E_BIAS: now reaches C3.1, D3.2 (A), L4.1
- net E_ANT: now reaches C3.2, J3.1 (In), R3.1
- net W_RF_TO_COM: now reaches D4.1 (K), D8.2 (A)
- net W_BIAS: now reaches C4.1, D4.2 (A), L5.1
- net E_RF_TO_COM: now reaches D3.1 (K), D7.2 (A)
- net N_ANT: now reaches C1.2, J1.1 (In), R1.1
- net S_BIAS: now reaches C2.1, D2.2 (A), L3.1
- net S_ANT: now reaches C2.2, J2.1 (In), R2.1
- net S_RF_TO_COM: now reaches D2.1 (K), D6.2 (A)
- net W_ANT: now reaches C4.2, J4.1 (In), R4.1
- net EAST renamed E_BIAS_IN
- net NORTH renamed N_BIAS_IN
- net SOUTH renamed S_BIAS_IN
- net WEST renamed W_BIAS_IN
- new net: C9.2, L6.1
Other:
- moved on the sheet: J5, R6
