File: projects/ddf_big_array/ddf_big_array.kicad_pcb (KiCad board)
At the start: 2 copper layers, 55 parts, among them J1 Conn_Coaxial, J101 Conn_Coaxial, J102 Conn_Coaxial, J2 Conn_Coaxial, J201 Conn_Coaxial, J202 Conn_Coaxial, J3 Conn_Coaxial, J301 Conn_Coaxial, J302 Conn_Coaxial, J4 Conn_Coaxial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

Commit message: Checkpoint.
Parts:
- moved C101 12.9 mm to (27.2, 35.0)
- moved R101 10.0 mm to (25.0, 35.6), turned to -90 degrees
- moved D101 9.75 mm to (31.5, 35.0)
- moved L101 9.59 mm to (29.3, 35.6), turned to -90 degrees
- moved J101 2.80 mm to (20.0, 35.0)
- moved J102 1.12 mm to (38.0, 35.0)
Connections:
- net Net-(J101-Pad2) renamed /N_ANT_GND
- net Net-(J201-Pad2) renamed /E_ANT_GND
- net Net-(J301-Pad2) renamed /S_ANT_GND
- net Net-(J401-Pad2) renamed /W_ANT_GND
Routing:
- net Net-(C101-Pad1): track 0.00 -> 6.63 mm
- net Net-(D101-Pad2): track 0.00 -> 5.80 mm
- net Net-(C101-Pad2): track 0.00 -> 3.06 mm
- added copper zone on B.Cu, net /N_ANT_GND
