File: projects/ddf_big_array_antterm/ddf_big_array_antterm.kicad_pcb (KiCad board)
At the start: 2 copper layers, 55 parts, among them J1 Conn_Coaxial, J101 Conn_Coaxial, J102 Conn_Coaxial, J2 Conn_Coaxial, J201 Conn_Coaxial, J202 Conn_Coaxial, J3 Conn_Coaxial, J301 Conn_Coaxial, J302 Conn_Coaxial, J4 Conn_Coaxial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

Commit message: Checkpoint.
Parts:
- removed the C1 at (199.6, 28.2)
- removed C2, C201, C3, C301, C4, C401, C5, C6, C7, C8, C9: C, Capacitor_SMD:C_0402_1005Metric_Pad0.74x0.62mm_HandSolder
- removed the D1 at (183.7, 27.4)
- removed D2, D201, D3, D301, D4, D401: D, Diode_SMD:D_SOD-523
- removed the J1 at (171.8, 27.2)
- removed the J2 at (171.5, 39.5)
- removed J201, J301, J401: Conn_Coaxial, Connector_Coaxial:SMA_Amphenol_132134_Vertical
- removed J202, J3, J302, J4, J402: Conn_Coaxial, Connector_Coaxial:SMA_Amphenol_132203-12_Horizontal
- removed J5: Conn_Coaxial, Connector_Coaxial:SMA_Molex_73251-2200_Horizontal
- removed J6, J7: RJ45_Shielded, Connector_RJ:RJ45_Wuerth_7499010001A_Horizontal
- removed J8: Conn_01x05_Male, Connector_PinHeader_2.54mm:PinHeader_1x05_P2.54mm_Vertical
- removed the L1 at (189.2, 26.6)
- removed L2, L201, L3, L301, L4, L401, L5: L, Inductor_SMD:L_0402_1005Metric_Pad0.77x0.64mm_HandSolder
- removed the R1 at (194.6, 28.4)
- removed R2, R201, R3, R301, R4, R401, R5: R, Resistor_SMD:R_0402_1005Metric_Pad0.72x0.64mm_HandSolder
- added H1: MountingHole, MountingHole:MountingHole_3.2mm_M3, F.Cu at (124.0, 84.0)
- added H2: MountingHole, MountingHole:MountingHole_3.2mm_M3, F.Cu at (86.0, 46.0)
- added H3: MountingHole, MountingHole:MountingHole_3.2mm_M3, F.Cu at (86.0, 84.0)
- added H4: MountingHole, MountingHole:MountingHole_3.2mm_M3, F.Cu at (124.0, 46.0)
- moved J2 91.1 mm to (124.0, 65.0)
- moved C1 90.0 mm to (112.0, 65.0)
- moved D1 90.0 mm to (116.3, 65.0)
- moved J1 90.0 mm to (104.8, 65.0)
- moved L1 90.0 mm to (114.1, 65.6)
- moved R1 90.0 mm to (109.8, 65.6)
- renumbered C101 to C1, D101 to D1, J101 to J1, J102 to J2, L101 to L1, R101 to R1
Connections:
- J1 pad 2: /N_ANT_GND -> GND
- J2 pad 2: /N_ANT_GND -> GND
- L1 pad 2: /N_ANT_GND -> GND
- R1 pad 2: /N_ANT_GND -> GND
Routing:
- net Net-(D1-Pad2): track 5.80 -> 7.02 mm
- added copper zone on B.Cu, net GND
- added copper zone on F.Cu, net GND
- removed copper zone on B.Cu, net /N_ANT_GND
Other:
- board outline added: 50 x 50 mm
- board text added: "TO DO: Set trace width for microstrip (remove top fill) or coplanar (stitch) Fix refdes Check against posible case (or plan for 3d print) Add artwork"

Commit message: Checkpoint.
Other:
- board text added: "ANT"
- board text added: "Murgatroid Heavy Industries, LLC"
- board text added: "OUT"

Commit message: Closing on release quality.
Parts:
- C1: value C -> 390p NP0; footprint Capacitor_SMD:C_0402_1005Metric_Pad0.74x0.62mm_HandSolder -> Capacitor_SMD:C_0603_1608Metric_Pad1.08x0.95mm_HandSolder
- D1: value D -> SMP1340
- H1, H2, H3, H4: footprint MountingHole:MountingHole_3.2mm_M3 -> MountingHole:MountingHole_3.2mm_M3_Pad_TopBottom
- J1: footprint Connector_Coaxial:SMA_Amphenol_132134_Vertical -> ch:SMA_Molex-73391-0070_Vertical
- J2: footprint Connector_Coaxial:SMA_Amphenol_132203-12_Horizontal -> ch:SMA_Molex_73251-2200_Horizontal
- L1: value L -> 510n; footprint Inductor_SMD:L_0402_1005Metric_Pad0.77x0.64mm_HandSolder -> ch:Coilcraft-0402HL-hand-solder
- R1: value R -> 1M
- moved L1 1.05 mm to (115.2, 65.6)
- moved D1 0.85 mm to (117.2, 65.0)
- moved R1 0.85 mm to (110.7, 65.6)
- moved C1 0.85 mm to (112.8, 65.0)
- moved J1 0.20 mm to (105.0, 65.0)
Connections:
- net Net-(C1-Pad1) renamed /ANT
- net Net-(C1-Pad2) renamed /RET
- net Net-(D1-Pad2) renamed /OUT
Routing:
- net GND: track 0.00 -> 2.13 mm, vias 0 -> 2
- net /OUT: track 7.02 -> 6.15 mm
- net /ANT: track 6.63 -> 7.28 mm
- added copper zone on In1.Cu, net GND
- added copper zone on In2.Cu, net GND
- removed copper zone on F.Cu, net GND
Other:
- copper layers 2 -> 4
- board text added: "50Z SE for JLC7628: 11.55 mil for microstrip per JLCPCB calculator"
- board text added: "Stack up per JLC04161H-7628 layer {dblquote}F.Silkscreen{dblquote} type {dblquote}Top Silk Screen{dblquote} Color {dblquote}Not specified{dblquote} Material {dblquote}Not specified{dblquote} layer {dblquote}F.Paste{dblquote} type {dblquote}Top Solder Paste{dblquote} layer {dblquote}F.Mask{dblquote} type {dblquote}Top Solder Mask{dblquote} Color {dblquote}Not specified{dblquote} Thickness 0.0127 m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"
- board text added: "ddf_big_array_antterm v1.0 ch@murgatroid.com"
- board text removed: "TO DO: Set trace width for microstrip (remove top fill) or coplanar (stitch) Fix refdes Check against posible case (or plan for 3d print) Add artwork"

Commit message: interim snapshot
Parts:
- C1: value 390p NP0 -> 390p NP0 50V; footprint Capacitor_SMD:C_0603_1608Metric_Pad1.08x0.95mm_HandSolder -> Capacitor_SMD:C_0402_1005Metric
- L1: value 510n -> 560n; footprint ch:Coilcraft-0402HL-hand-solder -> ch:IMC1008
- R1: value 1M -> 100K; footprint Resistor_SMD:R_0402_1005Metric_Pad0.72x0.64mm_HandSolder -> Resistor_SMD:R_0603_1608Metric
- moved D1 1.10 mm to (118.2, 65.0)
- moved L1 0.66 mm to (115.2, 66.2)
- moved C1 0.35 mm to (112.5, 65.0)
- moved R1 0.27 mm to (110.5, 65.8)
Routing:
- net /RET: track 2.98 -> 4.57 mm
- net /OUT: track 6.15 -> 5.05 mm
- net GND: track 2.13 -> 2.84 mm

Commit message: release candidate
Routing:
- net GND: vias 2 -> 180
- added copper zone on F.Cu, net GND

Commit message: release candidate
Parts:
- added R2: 100K, Resistor_SMD:R_0603_1608Metric, F.Cu at (119.0, 65.8)
- moved D1 1.38 mm to (116.9, 65.0)
- moved L1 1.12 mm to (114.1, 66.2)
- moved C1 0.75 mm to (111.8, 65.0)
- moved R1 0.50 mm to (110.0, 65.8)
Routing:
- net /OUT: track 5.05 -> 6.37 mm
- net /ANT: track 7.01 -> 6.24 mm
- net GND: track 2.84 -> 3.52 mm, vias 180 -> 181
- net /RET: track 4.57 -> 3.94 mm
Changed lines of the file:
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@@
   (net 4 "GND")
   (footprint "Resistor_SMD:R_0603_1608Metric" (layer "F.Cu")
-    (at 110.5 65.83 -90)
+    (at 119 65.8125 -90)
     (descr "Resistor SMD 0603 (1608 Metric), square (rectangular) end terminal, IPC_7351 nominal, (Body size source: IPC-SM-782 page 72, https://www.pcb-3d.com/wordpress/wp-content/uploads/ipc-sm-782a_amendment_1_and_2.pdf), generated with kicad-footprint-generator")
     (tags "resistor")
+    (property "LCSC" "C14675")
+    (property "MFG" "UNI-ROYAL")
+    (property "MPN" "RC0603FR-07100KL")
     (property "Sheetfile" "ddf_big_array_antterm.kicad_sch")
     (property "Sheetname" "")
     (attr smd)
-    (fp_text reference "R1" (at 5.67 -0.6) (layer "F.SilkS")
+    (fp_text reference "R2" (at 5.6875 0.5) (layer "F.SilkS")
+      (effects (font (size 1 1) (thickness 0.15)))
+    )
+    (fp_text value "100K" (at 0 1.43 90) (layer "F.Fab")
+      (effects (font (size 1 1) (thickness 0.15)))
+    )
+    (fp_text user "${REFERENCE}" (at 0 0 90) (layer "F.Fab")
+      (effects (font (size 0.4 0.4) (thickness 0.06)))
+    )
+    (fp_line (start -0.237258 0.5225) (end 0.237258 0.5225) (layer "F.SilkS") (width 0.12))
+    (fp_line (start -0.237258 -0.5225) (end 0.237258 -0.5225) (layer "F.SilkS") (width 0.12))
+    (fp_line (start 1.48 -0.73) (end 1.48 0.73) (layer "F.CrtYd") (width 0.05))
+    (fp_line (start -1.48 -0.73) (end 1.48 -0.73) (layer "F.CrtYd") (width 0.05))
+    (fp_line (start 1.48 0.73) (end -1.48 0.73) (layer "F.CrtYd") (width 0.05))
+    (fp_line (start -1.48 0.73) (end -1.48 -0.73) (layer "F.CrtYd") (width 0.05))
+    (fp_line (start -0.8 -0.4125) (end 0.8 -0.4125) (layer "F.Fab") (width 0.1))
+    (fp_line (start 0.8 -0.4125) (end 0.8 0.4125) (layer "F.Fab") (width 0.1))
+    (fp_line (start 0.8 0.4125) (end -0.8 0.4125) (layer "F.Fab") (width 0.1))
+    (fp_line (start -0.8 0.4125) (end -0.8 -0.4125) (layer "F.Fab") (width 0.1))
+    (pad "1" smd roundrect (at -0.825 0 270) (size 0.8 0.95) (layers "F.Cu" "F.Paste" "F.Mask") (roundrect_rratio 0.25)
+      (net 3 "/OUT") (pintype "passive"))
+    (pad "2" smd roundrect (at 0.825 0 270) (size 0.8 0.95) (layers "F.Cu" "F.Paste" "F.Mask") (roundrect_rratio 0.25)
+      (net 4 "GND") (pintype "passive"))
+    (model "${KICAD6_3DMODEL_DIR}/Resistor_SMD.3dshapes/R_0603_1608Metric.wrl"
+      (offset (xyz 0 0 0))
+      (scale (xyz 1 1 1))
+      (rotate (xyz 0 0 0))
+    )
+  )
+  (footprint "Resistor_SMD:R_0603_1608Metric" (layer "F.Cu")
+    (at 110 65.8125 -90)
+    (descr "Resistor SMD 0603 (1608 Metric), square (rectangular) end terminal, IPC_7351 nominal, (Body size source: IPC-SM-782 page 72, https://www.pcb-3d.com/wordpress/wp-content/uploads/ipc-sm-782a_amendment_1_and_2.pdf), generated with kicad-footprint-generator")
+    (tags "resistor")
+    (property "LCSC" "C14675")
+    (property "MFG" "UNI-ROYAL")
+    (property "MPN" "RC0603FR-07100KL")
+    (property "Sheetfile" "ddf_big_array_antterm.kicad_sch")
+    (property "Sheetname" "")
+    (attr smd)
+    (fp_text reference "R1" (at 5.67 -0.25) (layer "F.SilkS")
       (effects (font (size 1 1) (thickness 0.15)))
     )
@@
     (property "Sheetname" "")
     (attr through_hole)
-    (fp_text reference "J2" (at 4.8 0) (layer "F.SilkS")
+    (fp_text reference "J2" (at 5.25 2.5) (layer "F.SilkS")
       (effects (font (size 1 1) (thickness 0.15)))
     )
@@
   )
   (footprint "Capacitor_SMD:C_0402_1005Metric" (layer "F.Cu")
-    (at 112.5 65)
+    (at 111.75 65)
     (descr "Capacitor SMD 0402 (1005 Metric), square (rectangular) end terminal, IPC_7351 nominal, (Body size source: IPC-SM-782 page 76, https://www.pcb-3d.com/wordpress/wp-content/uploads/ipc-sm-782a_amendment_1_and_2.pdf), generated with kicad-footprint-generator")
     (tags "capacitor")
+    (property "LCSC" "C162100")
+    (property "MFG" "Murata")
+    (property "MPN" "GRM1555C1H391FA01D")
     (property "Sheetfile" "ddf_big_array_antterm.kicad_sch")
     (property "Sheetname" "")
     (attr smd)
-    (fp_text reference "C1" (at 0.75 6.5) (layer "F.SilkS")
+    (fp_text reference "C1" (at 0.5 6.5) (layer "F.SilkS")
       (effects (font (size 1 1) (thickness 0.15)))
     )
@@
   )
   (footprint "Diode_SMD:D_SOD-523" (layer "F.Cu")
-    (at 118.25 65)
+    (at 116.875 65)
     (descr "http://www.diodes.com/datasheets/ap02001.pdf p.144")
     (tags "Diode SOD523")
-    (property "MPN" "SMP1340-007LF")
+    (property "MFG" "Skyworks")
+    (property "MPN" "SMP1340-079LF")
     (property "Sheetfile" "ddf_big_array_antterm.kicad_sch")
     (property "Sheetname" "")
     (attr smd)
-    (fp_text reference "D1" (at -1 6.5) (layer "F.SilkS")
+    (fp_text reference "D1" (at -0.625 6.5) (layer "F.SilkS")
       (effects (font (size 1 1) (thickness 0.15)))
     )
@@
     (property "Sheetname" "")
     (attr through_hole)
-    (fp_text reference "J1" (at 0.25 4.75) (layer "F.SilkS")
+    (fp_text reference "J1" (at -2.5 5.25) (layer "F.SilkS")
       (effects (font (size 1 1) (thickness 0.15)))
     )
@@
   )
   (footprint "ch:IMC1008" (layer "F.Cu")
-    (at 115.25 66.25 -90)
+    (at 114.125 66.25 -90)
     (descr "Inductor SMD 1008 (2520 Metric), square (rectangular) end terminal, IPC_7351 nominal, (Body size source: https://ecsxtal.com/store/pdf/ECS-MPI2520-SMD-POWER-INDUCTOR.pdf), generated with kicad-footprint-generator")
     (tags "inductor")
+    (property "MFG" "Vishay Dale")
     (property "MPN" "IMC1008ERR56J")
     (property "Sheetfile" "ddf_big_array_antterm.kicad_sch")
@@
       (net 4 "GND") (pinfunction "1") (pintype "input"))
   )
-  (gr_rect (start 109.75 70.484) (end 118.5 72.5) (layer "F.SilkS") (width 0.15) (fill none))
+  (gr_rect (start 109 70.484) (end 119.75 72.5) (layer "F.SilkS") (width 0.15) (fill none))
   (gr_poly
     (pts
@@
     (effects (font (size 1 1) (thickness 0.15)) (justify left))
   )
-  (segment (start 105 65) (end 110.495 65) (width 0.29337) (layer "F.Cu") (net 1))
-  (segment (start 110.5 65.005) (end 112.015 65.005) (width 0.29337) (layer "F.Cu") (net 1))
-  (segment (start 112.98 65) (end 115.25 65) (width 0.29337) (layer "F.Cu") (net 2))
-  (segment (start 117.55 65) (end 115.25 65) (width 0.29337) (layer "F.Cu") (net 2))
-  (segment (start 124 65) (end 118.95 65) (width 0.29337) (layer "F.Cu") (net 3))
-  (segment (start 115.25 67.5) (end 115.25 69) (width 0.25) (layer "F.Cu") (net 4))
-  (segment (start 110.5 66.655) (end 110.5 68) (width 0.25) (layer "F.Cu") (net 4))
+  (segment (start 105 65) (end 109.9875 65) (width 0.29337) (layer "F.Cu") (net 1))
+  (segment (start 111.27 65) (end 110.0125 65) (width 0.29337) (layer "F.Cu") (net 1))
+  (segment (start 116.175 65) (end 114.125 65) (width 0.29337) (layer "F.Cu") (net 2))
+  (segment (start 112.23 65) (end 114.125 65) (width 0.29337) (layer "F.Cu") (net 2))
+  (segment (start 117.575 65) (end 118.975 65) (width 0.29337) (layer "F.Cu") (net 3))
+  (segment (start 124 65) (end 119.025 65) (width 0.29337) (layer "F.Cu") (net 3))
+  (segment (start 119 67.75) (end 119 66.6375) (width 0.25) (layer "F.Cu") (net 4))
+  (segment (start 114.125 68.8) (end 114.125 67.5) (width 0.25) (layer "F.Cu") (net 4))
+  (segment (start 110 67.75) (end 110 66.6375) (width 0.25) (layer "F.Cu") (net 4))
+  (via (at 119 67.75) (size 0.8) (drill 0.4) (layers "F.Cu" "B.Cu") (free) (net 4))
   (via (at 112 87) (size 0.8) (drill 0.4) (layers "F.Cu" "B.Cu") (free) (net 4))
   (via (at 97 42) (size 0.8) (drill 0.4) (layers "F.Cu" "B.Cu") (free) (net 4))
@@
   (via (at 101 86) (size 0.8) (drill 0.4) (layers "F.Cu" "B.Cu") (free) (net 4))
   (via (at 89 42) (size 0.8) (drill 0.4) (layers "F.Cu" "B.Cu") (free) (net 4))
-  (via (at 110.5 68) (size 0.8) (drill 0.4) (layers "F.Cu" "B.Cu") (free) (net 4))
+  (via (at 110 67.75) (size 0.8) (drill 0.4) (layers "F.Cu" "B.Cu") (free) (net 4))
   (via (at 93 42) (size 0.8) (drill 0.4) (layers "F.Cu" "B.Cu") (free) (net 4))
   (via (at 92 43) (size 0.8) (drill 0.4) (layers "F.Cu" "B.Cu") (free) (net 4))
@@
   (via (at 105 88) (size 0.8) (drill 0.4) (layers "F.Cu" "B.Cu") (free) (net 4))
   (via (at 82 49) (size 0.8) (drill 0.4) (layers "F.Cu" "B.Cu") (free) (net 4))
+  (via (at 114.125 68.8) (size 0.8) (drill 0.4) (layers "F.Cu" "B.Cu") (free) (net 4))
   (via (at 126 77) (size 0.8) (drill 0.4) (layers "F.Cu" "B.Cu") (free) (net 4))
   (via (at 83 58) (size 0.8) (drill 0.4) (layers "F.Cu" "B.Cu") (free) (net 4))
@@
   (via (at 127 76) (size 0.8) (drill 0.4) (layers "F.Cu" "B.Cu") (free) (net 4))
   (via (at 95 42) (size 0.8) (drill 0.4) (layers "F.Cu" "B.Cu") (free) (net 4))
-  (via (at 115.25 69) (size 0.8) (drill 0.4) (layers "F.Cu" "B.Cu") (free) (net 4))
   (via (at 94 87) (size 0.8) (drill 0.4) (layers "F.Cu" "B.Cu") (free) (net 4))
   (via (at 103 86) (size 0.8) (drill 0.4) (layers "F.Cu" "B.Cu") (free) (net 4))
