File: projects/ddf_big_array_antterm/ddf_big_array_antterm.kicad_sch (KiCad schematic)
At the start: 75 parts, among them J1 Conn_Coaxial, J101 Conn_Coaxial, J102 Conn_Coaxial, J2 Conn_Coaxial, J201 Conn_Coaxial, J202 Conn_Coaxial, J3 Conn_Coaxial, J301 Conn_Coaxial, J302 Conn_Coaxial, J4 Conn_Coaxial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

Commit message: Checkpoint.
Parts:
- removed C1, C2, C201, C3, C301, C4, C401, C5, C6, C7, C8, C9: C, Capacitor_SMD:C_0402_1005Metric_Pad0.74x0.62mm_HandSolder, symbol Device:C
- removed D1, D2, D201, D3, D301, D4, D401: D, Diode_SMD:D_SOD-523, symbol Device:D
- removed H? (x16): MountingHole, symbol Mechanical:MountingHole
- removed J1, J2, J202, J3, J302, J4, J402: Conn_Coaxial, Connector_Coaxial:SMA_Amphenol_132203-12_Horizontal, symbol Connector:Conn_Coaxial
- removed J201, J301, J401: Conn_Coaxial, Connector_Coaxial:SMA_Amphenol_132134_Vertical, symbol Connector:Conn_Coaxial
- removed J5: Conn_Coaxial, Connector_Coaxial:SMA_Molex_73251-2200_Horizontal, symbol Connector:Conn_Coaxial
- removed J6, J7: RJ45_Shielded, Connector_RJ:RJ45_Wuerth_7499010001A_Horizontal, symbol Connector:RJ45_Shielded
- removed J8: Conn_01x05_Male, Connector_PinHeader_2.54mm:PinHeader_1x05_P2.54mm_Vertical, symbol Connector:Conn_01x05_Male
- removed L1, L2, L201, L3, L301, L4, L401, L5: L, Inductor_SMD:L_0402_1005Metric_Pad0.77x0.64mm_HandSolder, symbol Device:L
- removed R1, R2, R201, R3, R301, R4, R401, R5: R, Resistor_SMD:R_0402_1005Metric_Pad0.72x0.64mm_HandSolder, symbol Device:R
- H1: renamed from H101; footprint (none) -> MountingHole:MountingHole_3.2mm_M3
- H2: renamed from H102; footprint (none) -> MountingHole:MountingHole_3.2mm_M3
- H3: renamed from H103; footprint (none) -> MountingHole:MountingHole_3.2mm_M3
- H4: renamed from H104; footprint (none) -> MountingHole:MountingHole_3.2mm_M3
- renumbered C101 to C1, D101 to D1, J101 to J1, J102 to J2, L101 to L1, R101 to R1
Connections:
- net N_ANT_GND is gone; now on net GND: J1.2 (Ext), J2.2 (Ext), L1.2, R1.2
Other:
- note removed: "Ltune/Ctune"
- note removed: "RJ45 T-568B 2/1 OR/ORWH 6/3 GR/GRWH 4/5 BL/BLWH 8/7 BR/BRWH"
- moved on the sheet: C1, D1, H1, H2, H3, H4, J1, J2, L1, R1

Commit message: Closing on release quality.
Parts:
- C1: value C -> 390p NP0; footprint Capacitor_SMD:C_0402_1005Metric_Pad0.74x0.62mm_HandSolder -> Capacitor_SMD:C_0603_1608Metric_Pad1.08x0.95mm_HandSolder
- D1: value D -> SMP1340
- H1, H2, H3, H4: footprint MountingHole:MountingHole_3.2mm_M3 -> MountingHole:MountingHole_3.2mm_M3_Pad_TopBottom; symbol Mechanical:MountingHole -> Mechanical:MountingHole_Pad
- J1: footprint Connector_Coaxial:SMA_Amphenol_132134_Vertical -> ch:SMA_Molex-73391-0070_Vertical
- J2: footprint Connector_Coaxial:SMA_Amphenol_132203-12_Horizontal -> ch:SMA_Molex_73251-2200_Horizontal
- L1: value L -> 510n; footprint Inductor_SMD:L_0402_1005Metric_Pad0.77x0.64mm_HandSolder -> ch:Coilcraft-0402HL-hand-solder
- R1: value R -> 100K
Connections:
- net GND: now also H1.1, H2.1, H3.1, H4.1
- net ANT: now reaches C1.1, J1.1 (In), R1.1
- net RET: now reaches C1.2, D1.1 (K), L1.1
- net OUT: now reaches D1.2 (A), J2.1 (In)
Other:
- note added: "510nH @ 144MHz => 461R 510nH @ 440MHz => 1410R 390pF @ 144MHz => 2.89R 390pF @ 440MHz => 0.93R"
- note added: "PIN: Skyworks SMP1340-079LF (SC-79/SOD-523) 1.2R@10mA@100MHz 0.3pF@5V@1MHz 50V 250mW https://www.skyworksinc.com/-/media/SkyWorks/Documents/Products/101-200/SMP1340_Series_200051U.pdf"
- note added: "RF Choke: CoilCraft 0402HL-511XJR 510nH Q=12@25MHz SRF=450MHz DCR=3.50R Irms=150mA https://www.coilcraft.com/en-us/products/rf/ceramic-core-chip-inductors/0402-(1005)/0402hl https://www.coilcraft.com/getmedia/e87228f8-e1c6-4958-ae62-6930ea641edb/0402hl.pdf"
- note added: "RF DC Blocking Cap: VJ HIFREQ Series https://www.vishay.com/docs/45258/vjhifreqseries.pdf"
- moved on the sheet: C1, D1, J1, J2, L1, R1

Commit message: interim snapshot
Parts:
- C1: value 390p NP0 -> 390p NP0 50V; footprint Capacitor_SMD:C_0603_1608Metric_Pad1.08x0.95mm_HandSolder -> Capacitor_SMD:C_0402_1005Metric
- D1: MPN (none) -> SMP1340-007LF
- L1: value 510n -> 560n; footprint ch:Coilcraft-0402HL-hand-solder -> ch:IMC1008; MPN (none) -> IMC1008ERR56J
- R1: footprint Resistor_SMD:R_0402_1005Metric_Pad0.72x0.64mm_HandSolder -> Resistor_SMD:R_0603_1608Metric
Other:
- note removed: "510nH @ 144MHz => 461R 510nH @ 440MHz => 1410R 390pF @ 144MHz => 2.89R 390pF @ 440MHz => 0.93R"
- note removed: "RF Choke: CoilCraft 0402HL-511XJR 510nH Q=12@25MHz SRF=450MHz DCR=3.50R Irms=150mA https://www.coilcraft.com/en-us/products/rf/ceramic-core-chip-inductors/0402-(1005)/0402hl https://www.coilcraft.com/getmedia/e87228f8-e1c6-4958-ae62-6930ea641edb/0402hl.pdf"
- note removed: "RF DC Blocking Cap: VJ HIFREQ Series https://www.vishay.com/docs/45258/vjhifreqseries.pdf"
Changed lines of the file:
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@@
     (stroke (width 0) (type default) (color 0 0 0 0))
   )
-  (text "510nH @ 144MHz => 461R\n510nH @ 440MHz => 1410R\n\n390pF @ 144MHz => 2.89R\n390pF @ 440MHz => 0.93R"
-    (at 130.175 46.99 0)
-    (effects (font (size 1.27 1.27)) (justify left bottom))
-  )
-  (text "RF DC Blocking Cap: VJ HIFREQ Series\n\nhttps://www.vishay.com/docs/45258/vjhifreqseries.pdf\n"
-    (at 93.218 97.282 0)
-    (effects (font (size 1.27 1.27)) (justify left bottom))
-  )
   (text "PIN: Skyworks SMP1340-079LF (SC-79/SOD-523)\n\n1.2R@10mA@100MHz 0.3pF@5V@1MHz 50V 250mW\n\nhttps://www.skyworksinc.com/-/media/SkyWorks/Documents/Products/101-200/SMP1340_Series_200051U.pdf"
-    (at 93.218 113.538 0)
-    (effects (font (size 1.27 1.27)) (justify left bottom))
-  )
-  (text "RF Choke: CoilCraft 0402HL-511XJR\n\n510nH Q=12@25MHz SRF=450MHz DCR=3.50R Irms=150mA\n\nhttps://www.coilcraft.com/en-us/products/rf/ceramic-core-chip-inductors/0402-(1005)/0402hl\nhttps://www.coilcraft.com/getmedia/e87228f8-e1c6-4958-ae62-6930ea641edb/0402hl.pdf\n"
-    (at 92.71 86.36 0)
+    (at 130.048 61.976 0)
     (effects (font (size 1.27 1.27)) (justify left bottom))
   )
@@
       (effects (font (size 1.27 1.27)) (justify left))
     )
-    (property "Footprint" "Resistor_SMD:R_0402_1005Metric_Pad0.72x0.64mm_HandSolder" (id 2) (at 57.912 43.815 90)
+    (property "Footprint" "Resistor_SMD:R_0603_1608Metric" (id 2) (at 57.912 43.815 90)
       (effects (font (size 1.27 1.27)) hide)
     )
@@
       (effects (font (size 1.27 1.27)) hide)
     )
+    (property "MPN" "SMP1340-007LF" (id 4) (at 81.915 38.735 0)
+      (effects (font (size 1.27 1.27)) hide)
+    )
     (pin "1")
     (pin "2")
@@
   (symbol (lib_id "Device:L") (at 74.295 43.815 0) (unit 1)
     (in_bom yes) (on_board yes) (fields_autoplaced)
-    (property "Reference" "L1" (id 0) (at 75.565 42.5449 0)
-      (effects (font (size 1.27 1.27)) (justify left))
-    )
-    (property "Value" "510n" (id 1) (at 75.565 45.0849 0)
-      (effects (font (size 1.27 1.27)) (justify left))
-    )
-    (property "Footprint" "ch:Coilcraft-0402HL-hand-solder" (id 2) (at 74.295 43.815 0)
+    (property "Reference" "L1" (id 0) (at 76.2 42.5449 0)
+      (effects (font (size 1.27 1.27)) (justify left))
+    )
+    (property "Value" "560n" (id 1) (at 76.2 45.0849 0)
+      (effects (font (size 1.27 1.27)) (justify left))
+    )
+    (property "Footprint" "ch:IMC1008" (id 2) (at 74.295 43.815 0)
       (effects (font (size 1.27 1.27)) hide)
     )
     (property "Datasheet" "~" (id 3) (at 74.295 43.815 0)
+      (effects (font (size 1.27 1.27)) hide)
+    )
+    (property "MPN" "IMC1008ERR56J" (id 4) (at 74.295 43.815 0)
       (effects (font (size 1.27 1.27)) hide)
     )
@@
     (in_bom yes) (on_board yes) (fields_autoplaced)
     (property "Reference" "C1" (id 0) (at 67.945 31.75 90))
-    (property "Value" "390p NP0" (id 1) (at 67.945 34.29 90))
-    (property "Footprint" "Capacitor_SMD:C_0603_1608Metric_Pad1.08x0.95mm_HandSolder" (id 2) (at 71.755 37.7698 0)
+    (property "Value" "390p NP0 50V" (id 1) (at 67.945 34.29 90))
+    (property "Footprint" "Capacitor_SMD:C_0402_1005Metric" (id 2) (at 71.755 37.7698 0)
       (effects (font (size 1.27 1.27)) hide)
     )
@@
     )
     (path "/ede5ab0d-9d11-4b47-8d0f-090cf3e9d513"
-      (reference "C1") (unit 1) (value "390p NP0") (footprint "Capacitor_SMD:C_0603_1608Metric_Pad1.08x0.95mm_HandSolder")
+      (reference "C1") (unit 1) (value "390p NP0 50V") (footprint "Capacitor_SMD:C_0402_1005Metric")
     )
     (path "/8959787f-6134-42a9-bd2d-e7f7a1af74c6"
@@
     )
     (path "/ab276e50-f838-4362-9aac-7d16f40393c4"
-      (reference "L1") (unit 1) (value "510n") (footprint "ch:Coilcraft-0402HL-hand-solder")
+      (reference "L1") (unit 1) (value "560n") (footprint "ch:IMC1008")
     )
     (path "/7af88a3a-2b90-481e-8799-91d38c39a62b"
-      (reference "R1") (unit 1) (value "100K") (footprint "Resistor_SMD:R_0402_1005Metric_Pad0.72x0.64mm_HandSolder")
-    )
-  )
+      (reference "R1") (unit 1) (value "100K") (footprint "Resistor_SMD:R_0603_1608Metric")
+    )
+  )

Commit message: release candidate
Parts:
- added R2: 100K, Resistor_SMD:R_0603_1608Metric, symbol Device:R
- C1: LCSC (none) -> C162100; MFG (none) -> Murata; MPN (none) -> GRM1555C1H391FA01D
- D1: MFG (none) -> Skyworks; MPN SMP1340-007LF -> SMP1340-079LF
- L1: MFG (none) -> Vishay Dale
- R1: LCSC (none) -> C14675; MFG (none) -> UNI-ROYAL; MPN (none) -> RC0603FR-07100KL
Connections:
- net GND: now also R2.2
- net OUT: now also R2.1
Other:
- note added: "560nH @ 144MHz => Z=506Ω 560nH @ 440MHz => Z=1547Ω 390pF @ 144MHz => Z=2.84Ω 390pF @ 440MHz => Z=0.928Ω"
- note added: "RF Choke: Vishay IMC-1008 High Frequency, Surface Mount Inductors https://www.vishay.com/docs/34041/imc1008.pdf PIN Diode: Skyworks SMP1340-079LF (SC-79/SOD-523) 1.2R@10mA@100MHz 0.3pF@5V@1MHz 50V 250mW https://www.skyworksinc.com/-/media/SkyWorks/Documents/Products/101-200/SMP1340_Series_200051U.pdf"
- note removed: "PIN: Skyworks SMP1340-079LF (SC-79/SOD-523) 1.2R@10mA@100MHz 0.3pF@5V@1MHz 50V 250mW https://www.skyworksinc.com/-/media/SkyWorks/Documents/Products/101-200/SMP1340_Series_200051U.pdf"
- moved on the sheet: C1, D1, J1, J2, L1, R1

Commit message: release candidate
Parts:
- H1, H2, H3: now left out of the parts list
Changed lines of the file:
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@@
   )
   (symbol (lib_id "Mechanical:MountingHole_Pad") (at 48.006 170.434 0) (unit 1)
-    (in_bom yes) (on_board yes)
+    (in_bom no) (on_board yes)
     (property "Reference" "H1" (id 0) (at 50.546 169.1639 0)
       (effects (font (size 1.27 1.27)) (justify left))
@@
   )
   (symbol (lib_id "Mechanical:MountingHole_Pad") (at 65.151 170.434 0) (unit 1)
-    (in_bom yes) (on_board yes) (fields_autoplaced)
+    (in_bom no) (on_board yes) (fields_autoplaced)
     (property "Reference" "H2" (id 0) (at 67.691 169.1639 0)
       (effects (font (size 1.27 1.27)) (justify left))
@@
   )
   (symbol (lib_id "Mechanical:MountingHole_Pad") (at 82.296 170.434 0) (unit 1)
-    (in_bom yes) (on_board yes) (fields_autoplaced)
+    (in_bom no) (on_board yes) (fields_autoplaced)
     (property "Reference" "H3" (id 0) (at 84.836 169.1639 0)
       (effects (font (size 1.27 1.27)) (justify left))

Commit message: release candidate
Parts:
- H4: now left out of the parts list
Changed lines of the file:
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@@
   )
   (symbol (lib_id "Mechanical:MountingHole_Pad") (at 99.314 170.434 0) (unit 1)
-    (in_bom yes) (on_board yes) (fields_autoplaced)
+    (in_bom no) (on_board yes) (fields_autoplaced)
     (property "Reference" "H4" (id 0) (at 101.854 169.1639 0)
       (effects (font (size 1.27 1.27)) (justify left))

Commit message: release candidate
Parts:
- removed R1, R2: 100K, Resistor_SMD:R_0603_1608Metric, symbol Device:R
- added D2, D3: ESD7951ST5G, Diode_SMD:D_SOD-923, symbol Device:D_TVS
Connections:
- net ANT: now also D2.2 (A2)
- net GND: now also D2.1 (A1), D3.1 (A1)
- net OUT: now also D3.2 (A2)
Other:
- moved on the sheet: C1, D1, J2, L1

Commit message: release candidate
Parts:
- J1: LCSC (none) -> C2874833
- J2: LCSC (none) -> C1509208
Changed lines of the file:
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@@
       (effects (font (size 1.27 1.27)) hide)
     )
-    (property "Datasheet" "~" (id 3) (at 57.15 44.45 0)
+    (property "Datasheet" "https://www.onsemi.com/pdf/datasheet/esd7951s-d.pdf" (id 3) (at 57.15 44.45 0)
       (effects (font (size 1.27 1.27)) hide)
     )
@@
     )
     (property "Datasheet" " ~" (id 3) (at 125.73 39.37 0)
+      (effects (font (size 1.27 1.27)) hide)
+    )
+    (property "LCSC" "C1509208" (id 4) (at 125.73 39.37 0)
       (effects (font (size 1.27 1.27)) hide)
     )
@@
       (effects (font (size 1.27 1.27)) hide)
     )
+    (property "LCSC" "C2874833" (id 4) (at 48.26 39.37 0)
+      (effects (font (size 1.27 1.27)) hide)
+    )
     (pin "1")
     (pin "2")
@@
       (effects (font (size 1.27 1.27)) hide)
     )
-    (property "Datasheet" "~" (id 3) (at 118.11 44.45 0)
+    (property "Datasheet" "https://www.onsemi.com/pdf/datasheet/esd7951s-d.pdf" (id 3) (at 118.11 44.45 0)
       (effects (font (size 1.27 1.27)) hide)
     )
