File: projects/ddf_big_array_antsw/ddf_big_array_antsw.kicad_sch (KiCad schematic)
At the start: 75 parts, among them J1 Conn_Coaxial, J101 Conn_Coaxial, J102 Conn_Coaxial, J2 Conn_Coaxial, J201 Conn_Coaxial, J202 Conn_Coaxial, J3 Conn_Coaxial, J301 Conn_Coaxial, J302 Conn_Coaxial, J4 Conn_Coaxial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

Commit message: Checkpoint.
Parts:
- removed C101, C201, C301, C401: C, Capacitor_SMD:C_0402_1005Metric_Pad0.74x0.62mm_HandSolder, symbol Device:C
- removed D101, D201, D301, D401: D, Diode_SMD:D_SOD-523, symbol Device:D
- removed H101, H102, H103, H104, H? (x12): MountingHole, symbol Mechanical:MountingHole
- removed J101, J201, J301, J401: Conn_Coaxial, Connector_Coaxial:SMA_Amphenol_132134_Vertical, symbol Connector:Conn_Coaxial
- removed J102, J202, J302, J402: Conn_Coaxial, Connector_Coaxial:SMA_Amphenol_132203-12_Horizontal, symbol Connector:Conn_Coaxial
- removed J7: RJ45_Shielded, Connector_RJ:RJ45_Wuerth_7499010001A_Horizontal, symbol Connector:RJ45_Shielded
- removed J8: Conn_01x05_Male, Connector_PinHeader_2.54mm:PinHeader_1x05_P2.54mm_Vertical, symbol Connector:Conn_01x05_Male
- removed L101, L201, L301, L401: L, Inductor_SMD:L_0402_1005Metric_Pad0.77x0.64mm_HandSolder, symbol Device:L
- removed R101, R201, R301, R401: R, Resistor_SMD:R_0402_1005Metric_Pad0.72x0.64mm_HandSolder, symbol Device:R
- added C10: C, Capacitor_SMD:C_0402_1005Metric_Pad0.74x0.62mm_HandSolder, symbol Device:C
- added R6: R, Resistor_SMD:R_0402_1005Metric_Pad0.72x0.64mm_HandSolder, symbol Device:R
- H1, H2, H3, H4: renamed from H?; footprint (none) -> MountingHole:MountingHole_3.2mm_M3
- J5: footprint Connector_Coaxial:SMA_Molex_73251-2200_Horizontal -> Connector_Coaxial:SMA_Amphenol_132203-12_Horizontal
- J6: footprint Connector_RJ:RJ45_Wuerth_7499010001A_Horizontal -> Connector_RJ:RJ45_Amphenol_RJHSE5380
Connections:
- net GND: now also C10.2, R6.2; no longer J6.SH
- new net: C10.1, J6.SH, R6.1
Other:
- note added: "RJ45 T-568B 2/1 OR-OR/WH 6/3 GR-GR/WH 4/5 BL-BL/WH 8/7 BR-BR/WH"
- note removed: "RJ45 T-568B 2/1 OR/ORWH 6/3 GR/GRWH 4/5 BL/BLWH 8/7 BR/BRWH"
- moved on the sheet: H1, H2, H3, H4, J6

Commit message: Checkpoint.
Parts:
- C10, C5, C6, C7, C8, C9: footprint Capacitor_SMD:C_0402_1005Metric_Pad0.74x0.62mm_HandSolder -> Capacitor_SMD:C_0603_1608Metric_Pad1.08x0.95mm_HandSolder
- R1, R2, R3, R4, R6: footprint Resistor_SMD:R_0402_1005Metric_Pad0.72x0.64mm_HandSolder -> Resistor_SMD:R_0603_1608Metric_Pad0.98x0.95mm_HandSolder
Changed lines of the file:
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@@
       (effects (font (size 1.27 1.27)) (justify left))
     )
-    (property "Footprint" "Capacitor_SMD:C_0402_1005Metric_Pad0.74x0.62mm_HandSolder" (id 2) (at 176.2252 101.6 0)
+    (property "Footprint" "Capacitor_SMD:C_0603_1608Metric_Pad1.08x0.95mm_HandSolder" (id 2) (at 176.2252 101.6 0)
       (effects (font (size 1.27 1.27)) hide)
     )
@@
     (property "Reference" "R3" (id 0) (at 143.51 99.06 90))
     (property "Value" "R" (id 1) (at 143.51 101.6 90))
-    (property "Footprint" "Resistor_SMD:R_0402_1005Metric_Pad0.72x0.64mm_HandSolder" (id 2) (at 143.51 107.188 90)
+    (property "Footprint" "Resistor_SMD:R_0603_1608Metric_Pad0.98x0.95mm_HandSolder" (id 2) (at 143.51 107.188 90)
       (effects (font (size 1.27 1.27)) hide)
     )
@@
       (effects (font (size 1.27 1.27)) (justify left))
     )
-    (property "Footprint" "Capacitor_SMD:C_0402_1005Metric_Pad0.74x0.62mm_HandSolder" (id 2) (at 263.2202 61.595 0)
+    (property "Footprint" "Capacitor_SMD:C_0603_1608Metric_Pad1.08x0.95mm_HandSolder" (id 2) (at 263.2202 61.595 0)
       (effects (font (size 1.27 1.27)) hide)
     )
@@
       (effects (font (size 1.27 1.27)) (justify left))
     )
-    (property "Footprint" "Capacitor_SMD:C_0402_1005Metric_Pad0.74x0.62mm_HandSolder" (id 2) (at 134.3152 158.75 0)
+    (property "Footprint" "Capacitor_SMD:C_0603_1608Metric_Pad1.08x0.95mm_HandSolder" (id 2) (at 134.3152 158.75 0)
       (effects (font (size 1.27 1.27)) hide)
     )
@@
     (property "Reference" "R1" (id 0) (at 143.51 24.13 90))
     (property "Value" "R" (id 1) (at 143.51 26.67 90))
-    (property "Footprint" "Resistor_SMD:R_0402_1005Metric_Pad0.72x0.64mm_HandSolder" (id 2) (at 143.51 32.258 90)
+    (property "Footprint" "Resistor_SMD:R_0603_1608Metric_Pad0.98x0.95mm_HandSolder" (id 2) (at 143.51 32.258 90)
       (effects (font (size 1.27 1.27)) hide)
     )
@@
     (property "Reference" "R2" (id 0) (at 143.51 60.96 90))
     (property "Value" "R" (id 1) (at 143.51 63.5 90))
-    (property "Footprint" "Resistor_SMD:R_0402_1005Metric_Pad0.72x0.64mm_HandSolder" (id 2) (at 143.51 69.088 90)
+    (property "Footprint" "Resistor_SMD:R_0603_1608Metric_Pad0.98x0.95mm_HandSolder" (id 2) (at 143.51 69.088 90)
       (effects (font (size 1.27 1.27)) hide)
     )
@@
       (effects (font (size 1.27 1.27)) (justify left))
     )
-    (property "Footprint" "Capacitor_SMD:C_0402_1005Metric_Pad0.74x0.62mm_HandSolder" (id 2) (at 134.3152 77.47 0)
+    (property "Footprint" "Capacitor_SMD:C_0603_1608Metric_Pad1.08x0.95mm_HandSolder" (id 2) (at 134.3152 77.47 0)
       (effects (font (size 1.27 1.27)) hide)
     )
@@
       (effects (font (size 1.27 1.27)) (justify left))
     )
-    (property "Footprint" "Resistor_SMD:R_0402_1005Metric_Pad0.72x0.64mm_HandSolder" (id 2) (at 252.222 58.42 90)
+    (property "Footprint" "Resistor_SMD:R_0603_1608Metric_Pad0.98x0.95mm_HandSolder" (id 2) (at 252.222 58.42 90)
       (effects (font (size 1.27 1.27)) hide)
     )
@@
       (effects (font (size 1.27 1.27)) (justify left))
     )
-    (property "Footprint" "Capacitor_SMD:C_0402_1005Metric_Pad0.74x0.62mm_HandSolder" (id 2) (at 134.3152 115.57 0)
+    (property "Footprint" "Capacitor_SMD:C_0603_1608Metric_Pad1.08x0.95mm_HandSolder" (id 2) (at 134.3152 115.57 0)
       (effects (font (size 1.27 1.27)) hide)
     )
@@
       (effects (font (size 1.27 1.27)) (justify left))
     )
-    (property "Footprint" "Capacitor_SMD:C_0402_1005Metric_Pad0.74x0.62mm_HandSolder" (id 2) (at 134.3152 40.64 0)
+    (property "Footprint" "Capacitor_SMD:C_0603_1608Metric_Pad1.08x0.95mm_HandSolder" (id 2) (at 134.3152 40.64 0)
       (effects (font (size 1.27 1.27)) hide)
     )
@@
     (property "Reference" "R4" (id 0) (at 143.51 142.24 90))
     (property "Value" "R" (id 1) (at 143.51 144.78 90))
-    (property "Footprint" "Resistor_SMD:R_0402_1005Metric_Pad0.72x0.64mm_HandSolder" (id 2) (at 143.51 150.368 90)
+    (property "Footprint" "Resistor_SMD:R_0603_1608Metric_Pad0.98x0.95mm_HandSolder" (id 2) (at 143.51 150.368 90)
       (effects (font (size 1.27 1.27)) hide)
     )
@@
     )
     (path "/ebee6295-95a0-4b78-820c-724e9fe8bc5d"
-      (reference "C5") (unit 1) (value "C") (footprint "Capacitor_SMD:C_0402_1005Metric_Pad0.74x0.62mm_HandSolder")
+      (reference "C5") (unit 1) (value "C") (footprint "Capacitor_SMD:C_0603_1608Metric_Pad1.08x0.95mm_HandSolder")
     )
     (path "/b70c6f80-9f0b-49ff-9760-23326927c8f4"
-      (reference "C6") (unit 1) (value "C") (footprint "Capacitor_SMD:C_0402_1005Metric_Pad0.74x0.62mm_HandSolder")
+      (reference "C6") (unit 1) (value "C") (footprint "Capacitor_SMD:C_0603_1608Metric_Pad1.08x0.95mm_HandSolder")
     )
     (path "/ea6d3061-13c4-4746-914e-a9591b4c7d84"
-      (reference "C7") (unit 1) (value "C") (footprint "Capacitor_SMD:C_0402_1005Metric_Pad0.74x0.62mm_HandSolder")
+      (reference "C7") (unit 1) (value "C") (footprint "Capacitor_SMD:C_0603_1608Metric_Pad1.08x0.95mm_HandSolder")
     )
     (path "/3e60d1a2-bbc3-478a-bd1a-757741907e9c"
-      (reference "C8") (unit 1) (value "C") (footprint "Capacitor_SMD:C_0402_1005Metric_Pad0.74x0.62mm_HandSolder")
+      (reference "C8") (unit 1) (value "C") (footprint "Capacitor_SMD:C_0603_1608Metric_Pad1.08x0.95mm_HandSolder")
     )
     (path "/11144e59-10a0-41f7-a9d6-bbbd2d208879"
-      (reference "C9") (unit 1) (value "C") (footprint "Capacitor_SMD:C_0402_1005Metric_Pad0.74x0.62mm_HandSolder")
+      (reference "C9") (unit 1) (value "C") (footprint "Capacitor_SMD:C_0603_1608Metric_Pad1.08x0.95mm_HandSolder")
     )
     (path "/2ba52fdd-6a8d-41ac-bb4a-7a0252982099"
-      (reference "C10") (unit 1) (value "C") (footprint "Capacitor_SMD:C_0402_1005Metric_Pad0.74x0.62mm_HandSolder")
+      (reference "C10") (unit 1) (value "C") (footprint "Capacitor_SMD:C_0603_1608Metric_Pad1.08x0.95mm_HandSolder")
     )
     (path "/57fb8ada-7623-4a7f-90a6-450a79e03e45"
@@
     )
     (path "/57956bab-b0fc-4027-bfc7-29ac34f67c29"
-      (reference "R1") (unit 1) (value "R") (footprint "Resistor_SMD:R_0402_1005Metric_Pad0.72x0.64mm_HandSolder")
+      (reference "R1") (unit 1) (value "R") (footprint "Resistor_SMD:R_0603_1608Metric_Pad0.98x0.95mm_HandSolder")
     )
     (path "/972d5e10-1a1c-4b23-a90f-f4f171587b05"
-      (reference "R2") (unit 1) (value "R") (footprint "Resistor_SMD:R_0402_1005Metric_Pad0.72x0.64mm_HandSolder")
+      (reference "R2") (unit 1) (value "R") (footprint "Resistor_SMD:R_0603_1608Metric_Pad0.98x0.95mm_HandSolder")
     )
     (path "/24cc2e59-0230-478d-b9ef-ad89fb1b17c0"
-      (reference "R3") (unit 1) (value "R") (footprint "Resistor_SMD:R_0402_1005Metric_Pad0.72x0.64mm_HandSolder")
+      (reference "R3") (unit 1) (value "R") (footprint "Resistor_SMD:R_0603_1608Metric_Pad0.98x0.95mm_HandSolder")
     )
     (path "/fdad155e-2f66-4e23-8c55-b0a7057b87ce"
-      (reference "R4") (unit 1) (value "R") (footprint "Resistor_SMD:R_0402_1005Metric_Pad0.72x0.64mm_HandSolder")
+      (reference "R4") (unit 1) (value "R") (footprint "Resistor_SMD:R_0603_1608Metric_Pad0.98x0.95mm_HandSolder")
     )
     (path "/0d7b6121-7f90-44b2-bdc3-d3f8e3779c1e"
@@
     )
     (path "/bae019c3-57d4-4c72-832f-fab263ff9cca"
-      (reference "R6") (unit 1) (value "R") (footprint "Resistor_SMD:R_0402_1005Metric_Pad0.72x0.64mm_HandSolder")
-    )
-  )
+      (reference "R6") (unit 1) (value "R") (footprint "Resistor_SMD:R_0603_1608Metric_Pad0.98x0.95mm_HandSolder")
+    )
+  )

Commit message: Closing on release quality.
Parts:
- C1, C2, C3, C4: value C -> 390p NP0; footprint Capacitor_SMD:C_0402_1005Metric_Pad0.74x0.62mm_HandSolder -> Capacitor_SMD:C_0603_1608Metric_Pad1.08x0.95mm_HandSolder
- C10: value C -> 1n
- C5, C6, C7, C8: value C -> 1n NP0
- C9: value C -> Ctune; footprint Capacitor_SMD:C_0603_1608Metric_Pad1.08x0.95mm_HandSolder -> Capacitor_SMD:C_0402_1005Metric_Pad0.74x0.62mm_HandSolder
- D1, D2, D3, D4: value D -> SMP1340
- H1, H2, H3, H4: footprint MountingHole:MountingHole_3.2mm_M3 -> MountingHole:MountingHole_3.2mm_M3_Pad_TopBottom; symbol Mechanical:MountingHole -> Mechanical:MountingHole_Pad
- J1, J2, J3, J4, J5: footprint Connector_Coaxial:SMA_Amphenol_132203-12_Horizontal -> ch:SMA_Molex_73251-2200_Horizontal
- L1, L2, L3, L4: value L -> 510n; footprint Inductor_SMD:L_0402_1005Metric_Pad0.77x0.64mm_HandSolder -> ch:Coilcraft-0402HL-hand-solder
- L5: value L -> Ltune
- R5, R6: value R -> 100K
Connections:
- net GND: now also H1.1, H2.1, H3.1, H4.1
- net S_SW: now reaches C3.1, D3.2 (A), L3.1
- net E_SW: now reaches C2.1, D2.2 (A), L2.1
- net W_SW: now reaches C4.1, D4.2 (A), L4.1
- net RJ_SHIELD: now reaches C10.1, J6.SH, R6.1
- net N_IN: now reaches D1.1 (K), J1.1 (In)
- net E_IN: now reaches D2.1 (K), J2.1 (In)
- net N_SW: now reaches C1.1, D1.2 (A), L1.1
- net S_IN: now reaches D3.1 (K), J3.1 (In)
- net W_IN: now reaches D4.1 (K), J4.1 (In)
Other:
- note added: "510nH @ 144MHz => 461R 510nH @ 440MHz => 1410R 390pF @ 144MHz => 2.89R 390pF @ 440MHz => 0.93R"
- note added: "PIN Diodes: Skyworks SMP1340-079LF (SC-79/SOD-523) 1.2R@10mA@100MHz 0.3pF@5V@1MHz 50V 250mW https://www.skyworksinc.com/-/media/SkyWorks/Documents/Products/101-200/SMP1340_Series_200051U.pdf"
- note added: "RF Chokes: CoilCraft 0402HL-511XJR 510nH Q=12@25MHz SRF=450MHz DCR=3.50R Irms=150mA https://www.coilcraft.com/en-us/products/rf/ceramic-core-chip-inductors/0402-(1005)/0402hl https://www.coilcraft.com/getmedia/e87228f8-e1c6-4958-ae62-6930ea641edb/0402hl.pdf"
- note added: "RF DC Block Caps: VJ HIFREQ Series https://www.vishay.com/docs/45258/vjhifreqseries.pdf"
- note added: "RJ45 T-568B 2/1 OR-OR/WH => W 6/3 GR-GR/WH => E 4/5 BL-BL/WH => S 8/7 BR-BR/WH => N"
- note removed: "Ltune/Ctune"
- note removed: "RJ45 T-568B 2/1 OR-OR/WH 6/3 GR-GR/WH 4/5 BL-BL/WH 8/7 BR-BR/WH"
- moved on the sheet: C1, C10, C2, C3, C4, C5, C6, C7, C8, C9, D1, D2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

Commit message: interim snapshot
Parts:
- C1, C10, C2, C3, C4, C5, C6, C7, C8: footprint Capacitor_SMD:C_0603_1608Metric_Pad1.08x0.95mm_HandSolder -> Capacitor_SMD:C_0603_1608Metric
- C9: footprint Capacitor_SMD:C_0402_1005Metric_Pad0.74x0.62mm_HandSolder -> Capacitor_SMD:C_0603_1608Metric
- L1, L2, L3, L4: value 510n -> 560n; footprint ch:Coilcraft-0402HL-hand-solder -> ch:IMC1008; MPN (none) -> IMC1008ERR56J
Changed lines of the file:
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@@
     (property "Reference" "C3" (id 0) (at 58.42 99.695 90))
     (property "Value" "390p NP0" (id 1) (at 58.42 102.235 90))
-    (property "Footprint" "Capacitor_SMD:C_0603_1608Metric_Pad1.08x0.95mm_HandSolder" (id 2) (at 62.23 106.3498 0)
+    (property "Footprint" "Capacitor_SMD:C_0603_1608Metric" (id 2) (at 62.23 106.3498 0)
       (effects (font (size 1.27 1.27)) hide)
     )
@@
     (in_bom yes) (on_board yes) (fields_autoplaced)
     (property "Reference" "L3" (id 0) (at 85.09 95.885 90))
-    (property "Value" "510n" (id 1) (at 85.09 98.425 90))
-    (property "Footprint" "ch:Coilcraft-0402HL-hand-solder" (id 2) (at 85.09 102.235 0)
+    (property "Value" "560n" (id 1) (at 85.09 98.425 90))
+    (property "Footprint" "ch:IMC1008" (id 2) (at 85.09 102.235 0)
       (effects (font (size 1.27 1.27)) hide)
     )
@@
       (effects (font (size 1.27 1.27)) hide)
     )
+    (property "MPN" "IMC1008ERR56J" (id 4) (at 85.09 102.235 90)
+      (effects (font (size 1.27 1.27)) hide)
+    )
     (pin "1")
     (pin "2")
@@
     (in_bom yes) (on_board yes) (fields_autoplaced)
     (property "Reference" "L2" (id 0) (at 85.09 57.785 90))
-    (property "Value" "510n" (id 1) (at 85.09 60.325 90))
-    (property "Footprint" "ch:Coilcraft-0402HL-hand-solder" (id 2) (at 85.09 64.135 0)
+    (property "Value" "560n" (id 1) (at 85.09 60.325 90))
+    (property "Footprint" "ch:IMC1008" (id 2) (at 85.09 64.135 0)
       (effects (font (size 1.27 1.27)) hide)
     )
@@
       (effects (font (size 1.27 1.27)) hide)
     )
+    (property "MPN" "IMC1008ERR56J" (id 4) (at 85.09 64.135 90)
+      (effects (font (size 1.27 1.27)) hide)
+    )
     (pin "1")
     (pin "2")
@@
       (effects (font (size 1.27 1.27)) (justify left))
     )
-    (property "Footprint" "Capacitor_SMD:C_0402_1005Metric_Pad0.74x0.62mm_HandSolder" (id 2) (at 126.9492 98.806 0)
+    (property "Footprint" "Capacitor_SMD:C_0603_1608Metric" (id 2) (at 126.9492 98.806 0)
       (effects (font (size 1.27 1.27)) hide)
     )
@@
     (in_bom yes) (on_board yes) (fields_autoplaced)
     (property "Reference" "L4" (id 0) (at 85.09 139.065 90))
-    (property "Value" "510n" (id 1) (at 85.09 141.605 90))
-    (property "Footprint" "ch:Coilcraft-0402HL-hand-solder" (id 2) (at 85.09 145.415 0)
+    (property "Value" "560n" (id 1) (at 85.09 141.605 90))
+    (property "Footprint" "ch:IMC1008" (id 2) (at 85.09 145.415 0)
       (effects (font (size 1.27 1.27)) hide)
     )
     (property "Datasheet" "~" (id 3) (at 85.09 145.415 0)
+      (effects (font (size 1.27 1.27)) hide)
+    )
+    (property "MPN" "IMC1008ERR56J" (id 4) (at 85.09 145.415 90)
       (effects (font (size 1.27 1.27)) hide)
     )
@@
       (effects (font (size 1.27 1.27)) (justify left))
     )
-    (property "Footprint" "Capacitor_SMD:C_0603_1608Metric_Pad1.08x0.95mm_HandSolder" (id 2) (at 264.6172 64.516 0)
+    (property "Footprint" "Capacitor_SMD:C_0603_1608Metric" (id 2) (at 264.6172 64.516 0)
       (effects (font (size 1.27 1.27)) hide)
     )
@@
       (effects (font (size 1.27 1.27)) (justify left))
     )
-    (property "Footprint" "Capacitor_SMD:C_0603_1608Metric_Pad1.08x0.95mm_HandSolder" (id 2) (at 92.4052 155.575 0)
+    (property "Footprint" "Capacitor_SMD:C_0603_1608Metric" (id 2) (at 92.4052 155.575 0)
       (effects (font (size 1.27 1.27)) hide)
     )
@@
     (property "Reference" "C1" (id 0) (at 58.42 24.765 90))
     (property "Value" "390p NP0" (id 1) (at 58.42 27.305 90))
-    (property "Footprint" "Capacitor_SMD:C_0603_1608Metric_Pad1.08x0.95mm_HandSolder" (id 2) (at 62.23 31.4198 0)
+    (property "Footprint" "Capacitor_SMD:C_0603_1608Metric" (id 2) (at 62.23 31.4198 0)
       (effects (font (size 1.27 1.27)) hide)
     )
@@
     (property "Reference" "C4" (id 0) (at 58.42 142.875 90))
     (property "Value" "390p NP0" (id 1) (at 58.42 145.415 90))
-    (property "Footprint" "Capacitor_SMD:C_0603_1608Metric_Pad1.08x0.95mm_HandSolder" (id 2) (at 62.23 149.5298 0)
+    (property "Footprint" "Capacitor_SMD:C_0603_1608Metric" (id 2) (at 62.23 149.5298 0)
       (effects (font (size 1.27 1.27)) hide)
     )
@@
       (effects (font (size 1.27 1.27)) (justify left))
     )
-    (property "Footprint" "Capacitor_SMD:C_0603_1608Metric_Pad1.08x0.95mm_HandSolder" (id 2) (at 92.4052 74.295 0)
+    (property "Footprint" "Capacitor_SMD:C_0603_1608Metric" (id 2) (at 92.4052 74.295 0)
       (effects (font (size 1.27 1.27)) hide)
     )
@@
     (in_bom yes) (on_board yes) (fields_autoplaced)
     (property "Reference" "L1" (id 0) (at 85.09 20.955 90))
-    (property "Value" "510n" (id 1) (at 85.09 23.495 90))
-    (property "Footprint" "ch:Coilcraft-0402HL-hand-solder" (id 2) (at 85.09 27.305 0)
+    (property "Value" "560n" (id 1) (at 85.09 23.495 90))
+    (property "Footprint" "ch:IMC1008" (id 2) (at 85.09 27.305 0)
       (effects (font (size 1.27 1.27)) hide)
     )
     (property "Datasheet" "~" (id 3) (at 85.09 27.305 0)
+      (effects (font (size 1.27 1.27)) hide)
+    )
+    (property "MPN" "IMC1008ERR56J" (id 4) (at 85.09 27.305 90)
       (effects (font (size 1.27 1.27)) hide)
     )
@@
       (effects (font (size 1.27 1.27)) (justify left))
     )
-    (property "Footprint" "Capacitor_SMD:C_0603_1608Metric_Pad1.08x0.95mm_HandSolder" (id 2) (at 92.4052 112.395 0)
+    (property "Footprint" "Capacitor_SMD:C_0603_1608Metric" (id 2) (at 92.4052 112.395 0)
       (effects (font (size 1.27 1.27)) hide)
     )
@@
       (effects (font (size 1.27 1.27)) (justify left))
     )
-    (property "Footprint" "Capacitor_SMD:C_0603_1608Metric_Pad1.08x0.95mm_HandSolder" (id 2) (at 92.4052 37.465 0)
+    (property "Footprint" "Capacitor_SMD:C_0603_1608Metric" (id 2) (at 92.4052 37.465 0)
       (effects (font (size 1.27 1.27)) hide)
     )
@@
     (property "Reference" "C2" (id 0) (at 58.42 61.595 90))
     (property "Value" "390p NP0" (id 1) (at 58.42 64.135 90))
-    (property "Footprint" "Capacitor_SMD:C_0603_1608Metric_Pad1.08x0.95mm_HandSolder" (id 2) (at 62.23 68.2498 0)
+    (property "Footprint" "Capacitor_SMD:C_0603_1608Metric" (id 2) (at 62.23 68.2498 0)
       (effects (font (size 1.27 1.27)) hide)
     )
@@
     )
     (path "/6fc91c3d-5283-48aa-86c9-0a0b148ec670"
-      (reference "C1") (unit 1) (value "390p NP0") (footprint "Capacitor_SMD:C_0603_1608Metric_Pad1.08x0.95mm_HandSolder")
+      (reference "C1") (unit 1) (value "390p NP0") (footprint "Capacitor_SMD:C_0603_1608Metric")
     )
     (path "/f5df2f96-0b2b-44c4-a278-36079decc514"
-      (reference "C2") (unit 1) (value "390p NP0") (footprint "Capacitor_SMD:C_0603_1608Metric_Pad1.08x0.95mm_HandSolder")
+      (reference "C2") (unit 1) (value "390p NP0") (footprint "Capacitor_SMD:C_0603_1608Metric")
     )
     (path "/0aaa5383-0b9c-4781-b683-e869fc7ad4ed"
-      (reference "C3") (unit 1) (value "390p NP0") (footprint "Capacitor_SMD:C_0603_1608Metric_Pad1.08x0.95mm_HandSolder")
+      (reference "C3") (unit 1) (value "390p NP0") (footprint "Capacitor_SMD:C_0603_1608Metric")
     )
     (path "/7ac55616-5762-4d3f-9ce0-3ea65a5449ac"
-      (reference "C4") (unit 1) (value "390p NP0") (footprint "Capacitor_SMD:C_0603_1608Metric_Pad1.08x0.95mm_HandSolder")
+      (reference "C4") (unit 1) (value "390p NP0") (footprint "Capacitor_SMD:C_0603_1608Metric")
     )
     (path "/ebee6295-95a0-4b78-820c-724e9fe8bc5d"
-      (reference "C5") (unit 1) (value "1n NP0") (footprint "Capacitor_SMD:C_0603_1608Metric_Pad1.08x0.95mm_HandSolder")
+      (reference "C5") (unit 1) (value "1n NP0") (footprint "Capacitor_SMD:C_0603_1608Metric")
     )
     (path "/b70c6f80-9f0b-49ff-9760-23326927c8f4"
-      (reference "C6") (unit 1) (value "1n NP0") (footprint "Capacitor_SMD:C_0603_1608Metric_Pad1.08x0.95mm_HandSolder")
+      (reference "C6") (unit 1) (value "1n NP0") (footprint "Capacitor_SMD:C_0603_1608Metric")
     )
     (path "/ea6d3061-13c4-4746-914e-a9591b4c7d84"
-      (reference "C7") (unit 1) (value "1n NP0") (footprint "Capacitor_SMD:C_0603_1608Metric_Pad1.08x0.95mm_HandSolder")
+      (reference "C7") (unit 1) (value "1n NP0") (footprint "Capacitor_SMD:C_0603_1608Metric")
     )
     (path "/3e60d1a2-bbc3-478a-bd1a-757741907e9c"
-      (reference "C8") (unit 1) (value "1n NP0") (footprint "Capacitor_SMD:C_0603_1608Metric_Pad1.08x0.95mm_HandSolder")
+      (reference "C8") (unit 1) (value "1n NP0") (footprint "Capacitor_SMD:C_0603_1608Metric")
     )
     (path "/11144e59-10a0-41f7-a9d6-bbbd2d208879"
-      (reference "C9") (unit 1) (value "Ctune") (footprint "Capacitor_SMD:C_0402_1005Metric_Pad0.74x0.62mm_HandSolder")
+      (reference "C9") (unit 1) (value "Ctune") (footprint "Capacitor_SMD:C_0603_1608Metric")
     )
     (path "/2ba52fdd-6a8d-41ac-bb4a-7a0252982099"
-      (reference "C10") (unit 1) (value "1n") (footprint "Capacitor_SMD:C_0603_1608Metric_Pad1.08x0.95mm_HandSolder")
+      (reference "C10") (unit 1) (value "1n") (footprint "Capacitor_SMD:C_0603_1608Metric")
     )
     (path "/57fb8ada-7623-4a7f-90a6-450a79e03e45"
@@
     )
     (path "/c9c40959-458e-4364-833a-949b622eda4f"
-      (reference "L1") (unit 1) (value "510n") (footprint "ch:Coilcraft-0402HL-hand-solder")
+      (reference "L1") (unit 1) (value "560n") (footprint "ch:IMC1008")
     )
     (path "/1112b7d9-fa55-49d2-a6fe-e666f391852c"
-      (reference "L2") (unit 1) (value "510n") (footprint "ch:Coilcraft-0402HL-hand-solder")
+      (reference "L2") (unit 1) (value "560n") (footprint "ch:IMC1008")
     )
     (path "/0bf0be6f-2f84-49d1-8431-ab84e97b20e6"
-      (reference "L3") (unit 1) (value "510n") (footprint "ch:Coilcraft-0402HL-hand-solder")
+      (reference "L3") (unit 1) (value "560n") (footprint "ch:IMC1008")
     )
     (path "/1d8d01e5-72bc-4f45-8e6e-c4ea6d79abeb"
-      (reference "L4") (unit 1) (value "510n") (footprint "ch:Coilcraft-0402HL-hand-solder")
+      (reference "L4") (unit 1) (value "560n") (footprint "ch:IMC1008")
     )
     (path "/c9df7f03-6d00-45e4-8f3a-2c2397f8bcdc"

Commit message: checkpoint
Parts:
- added J7: 5_Port_50Z_RF_Junction, ch:5 Port 50Z RF Junction, symbol ch:5_Port_50Z_RF_Junction
Connections:
- removed net RF_COM: C1.2, C2.2, C3.2, C4.2, L5.1
- new net E_SW_DCB: C2.2, J7.2 (Pin_2)
- new net N_SW_DCB: C1.2, J7.1 (Pin_1)
- new net S_SW_DCB: C3.2, J7.4 (Pin_4)
- new net TUNE: J7.3 (Pin_3), L5.1
- new net W_SW_DCB: C4.2, J7.5 (Pin_5)
Other:
- moved on the sheet: C1, C10, C2, C3, C4, C5, C6, C7, C8, C9, D1, D2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
