File: projects/ddf_big_array_antsw/ddf_big_array_antsw.kicad_sch (KiCad schematic)
At the start: 36 parts, among them J1 Conn_Coaxial, J2 Conn_Coaxial, J3 Conn_Coaxial, J4 Conn_Coaxial, J5 Conn_Coaxial, J6 RJ45_Shielded, J7 5_Port_50Z_RF_Junction

Commit message: release candidate
Parts:
- added R1, R3, R5, R7: 100K, Resistor_SMD:R_0603_1608Metric, symbol Device:R
- C1, C2, C3, C4: value 390p NP0 -> 390p NP0 50V; LCSC (none) -> C162100; MFG (none) -> Murata; MPN (none) -> GRM1555C1H391FA01D
- C10: value 1n -> 1n NP0 50V; LCSC (none) -> C77026; MFG (none) -> Murata; MPN (none) -> GRM1885C1H102JA01D
- C5, C6, C7, C8: value 1n NP0 -> 1n NP0 50V; LCSC (none) -> C77026; MFG (none) -> Murata; MPN (none) -> GRM1885C1H102JA01D
- C9: value Ctune -> DNP
- D1, D2, D3, D4: MFG (none) -> Skyworks; MPN (none) -> SMP1340-079LF
- H1, H2, H3, H4: now left out of the parts list
- L1, L2, L3, L4: MFG (none) -> Vishay Dale
- L5: value Ltune -> 0R; LCSC (none) -> C17168; MFG (none) -> UNI-ROYAL; MPN (none) -> 0402WGF0000TCE
- R10: renamed from R6; footprint Resistor_SMD:R_0603_1608Metric_Pad0.98x0.95mm_HandSolder -> Resistor_SMD:R_0603_1608Metric; LCSC (none) -> C14675; MFG (none) -> Yageo; MPN (none) -> RC0603FR-07100KL
- R2: renamed from R1; value R -> 270; LCSC (none) -> C137754; MFG (none) -> Yageo; MPN (none) -> RC0603FR-07270RL
- R4: renamed from R2; value R -> 270; LCSC (none) -> C137754; MFG (none) -> Yageo; MPN (none) -> RC0603FR-07270RL
- R6: renamed from R3; value R -> 270; LCSC (none) -> C137754; MFG (none) -> Yageo; MPN (none) -> RC0603FR-07270RL
- R8: renamed from R4; value R -> 270; LCSC (none) -> C137754; MFG (none) -> Yageo; MPN (none) -> RC0603FR-07270RL
- R9: renamed from R5; footprint Resistor_SMD:R_0402_1005Metric_Pad0.72x0.64mm_HandSolder -> Resistor_SMD:R_0603_1608Metric; LCSC (none) -> C14675; MFG (none) -> Yageo; MPN (none) -> RC0603FR-07100KL
Connections:
- net E_IN: now also R3.1
- net GND: now also R1.2, R3.2, R5.2, R7.2
- net N_IN: now also R1.1
- net S_IN: now also R5.1
- net W_IN: now also R7.1
Other:
- note added: "560nH @ 144MHz => Z=506Ω 560nH @ 440MHz => Z=1547Ω 390pF @ 144MHz => Z=2.84Ω 390pF @ 440MHz => Z=0.928Ω"
- note added: "RF Choke: Vishay IMC-1008 High Frequency, Surface Mount Inductors https://www.vishay.com/docs/34041/imc1008.pdf PIN Diode: Skyworks SMP1340-079LF (SC-79/SOD-523) 1.2R@10mA@100MHz 0.3pF@5V@1MHz 50V 250mW https://www.skyworksinc.com/-/media/SkyWorks/Documents/Products/101-200/SMP1340_Series_200051U.pdf"
- note removed: "510nH @ 144MHz => 461R 510nH @ 440MHz => 1410R 390pF @ 144MHz => 2.89R 390pF @ 440MHz => 0.93R"
- note removed: "PIN Diodes: Skyworks SMP1340-079LF (SC-79/SOD-523) 1.2R@10mA@100MHz 0.3pF@5V@1MHz 50V 250mW https://www.skyworksinc.com/-/media/SkyWorks/Documents/Products/101-200/SMP1340_Series_200051U.pdf"
- note removed: "RF Chokes: CoilCraft 0402HL-511XJR 510nH Q=12@25MHz SRF=450MHz DCR=3.50R Irms=150mA https://www.coilcraft.com/en-us/products/rf/ceramic-core-chip-inductors/0402-(1005)/0402hl https://www.coilcraft.com/getmedia/e87228f8-e1c6-4958-ae62-6930ea641edb/0402hl.pdf"
- note removed: "RF DC Block Caps: VJ HIFREQ Series https://www.vishay.com/docs/45258/vjhifreqseries.pdf"
- moved on the sheet: C1, C2, C3, C4, C6, C7, D1, D3, D4, J1, J3, J4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

Commit message: release candidate
Parts:
- added D5, D6, D7, D8, D9: ESD7951ST5G, Diode_SMD:D_SOD-923, symbol Device:D_TVS
- added U1: SMDB05, Package_SO:SO-8_3.9x4.9mm_P1.27mm, symbol ch:TVS 4x Unidir
Connections:
- net E_BIAS: now also U1.2 (B1)
- net E_IN: now also D6.2 (A2)
- net GND: now also D5.1 (A1), D6.1 (A1), D7.1 (A1), D8.1 (A1), D9.1 (A1), U1.5 (D2), U1.6 (C2), U1.7 (B2), U1.8 (A2)
- net N_BIAS: now also U1.1 (A1)
- net N_IN: now also D5.2 (A2)
- net RF_OUT: now also D9.2 (A2)
- net S_BIAS: now also U1.3 (C1)
- net S_IN: now also D7.2 (A2)
- net W_BIAS: now also U1.4 (D1)
- net W_IN: now also D8.2 (A2)
Other:
- note added: "RF Choke: Vishay IMC-1008 High Frequency, Surface Mount Inductors PIN Diode: Skyworks SMP1340-079LF (SC-79/SOD-523) 1.2R@10mA@100MHz 0.3pF@5V@1MHz 50V 250mW"
- note removed: "RF Choke: Vishay IMC-1008 High Frequency, Surface Mount Inductors https://www.vishay.com/docs/34041/imc1008.pdf PIN Diode: Skyworks SMP1340-079LF (SC-79/SOD-523) 1.2R@10mA@100MHz 0.3pF@5V@1MHz 50V 250mW https://www.skyworksinc.com/-/media/SkyWorks/Documents/Products/101-200/SMP1340_Series_200051U.pdf"
- moved on the sheet: C1, C2, C3, C4, C5, C6, C7, C8, C9, D1, D2, D3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

Commit message: release candidate
Parts:
- added FB1, FB2, FB3, FB4: 600R @ 100 MHz, Inductor_SMD:L_0603_1608Metric, symbol Device:FerriteBead_Small
- C9: LCSC (none) -> DNP
- J1, J2, J3, J4, J5: LCSC (none) -> C1509208
- J6: LCSC (none) -> C464586
- U1: value SMDB05 -> SMDA05; LCSC (none) -> C1978067; MFG SMC -> Semtech; MPN SMDB05 -> SMDA05
Connections:
- net E_BIAS: now also FB2.1; no longer J6.6, U1.2 (B1)
- net N_BIAS: now also FB1.1; no longer J6.8, U1.1 (A1)
- net S_BIAS: now also FB3.1; no longer J6.4, U1.3 (C1)
- net W_BIAS: now also FB4.1; no longer J6.2, U1.4 (D1)
- new net: FB1.2, J6.8, U1.1 (A1)
- new net: FB3.2, J6.4, U1.3 (C1)
- new net: FB2.2, J6.6, U1.2 (B1)
- new net: FB4.2, J6.2, U1.4 (D1)
