File: projects/txrx_switcher/txrx_switcher.kicad_pcb (KiCad board)
At the start: 2 copper layers, 4 parts, among them K1 HF3-56, K2 HF3-56, Q1 IRF7309IPBF

Commit message: .
Parts:
- removed A1: Arduino_Nano_v3.x, Module:Arduino_Nano
- removed Q1: IRF7309IPBF, Package_SO:SOIC-8_3.9x4.9mm_P1.27mm
- renumbered K2 to K1, K1 to K2
Connections:
- net +VDC renamed Net-(D1-Pad1)
- K1 pad 11: Net-(K1-Pad11) -> GND
- K2 pad 11: Net-(K1-Pad11) -> GND
