File: projects/txrx_switcher/txrx_switcher.kicad_sch (KiCad schematic)
At the start: 12 parts, among them J1 Conn_Coaxial, J2 Conn_Coaxial, J3 Conn_Coaxial, J4 Conn_Coaxial, J5 Conn_Coaxial, J6 Conn_Coaxial, K1 HF3-56, K2 HF3-56, Q1 IRF7309IPBF

Commit message: .
Parts:
- removed A1: Arduino_Nano_v3.x, Module:Arduino_Nano, symbol MCU_Module:Arduino_Nano_v3.x
- removed Q1: IRF7309IPBF, Package_SO:SOIC-8_3.9x4.9mm_P1.27mm, symbol Transistor_FET:IRF7309IPBF
- added D2: D, symbol Device:D
- added Q?: DMP3013SFV, Package_SON:Diodes_PowerDI3333-8, symbol Transistor_FET:DMP3013SFV
- added R2: 5K, symbol Device:R
- added R3: 10, symbol Device:R
- R1: value 10K -> 5K
- renumbered J6 to J1, J4 to J2, J2 to J4, J1 to J5, J5 to J6, K2 to K1, K1 to K2
Connections:
- net +VDC: now also R3.1; no longer D1.1 (K), K1.1, K2.1
- net GND: now also D1.2 (A), K1.11, K2.11, D2.2 (A); no longer R1.2
- net RX/^TX renamed ^TX/RX
- new net: Q?.5 (D), R2.1, R3.2
- new net: Q?.4 (G), R1.2, R2.2
- new net: D1.1 (K), D2.1 (K), K1.1, K2.1, Q?.1 (S), Q?.2 (S), Q?.3 (S)
Other:
- moved on the sheet: D1, J1, J2, J3, J4, K1
