File: projects/z3817a_breakout/z3817a_breakout.kicad_sch (KiCad schematic)
At the start: 35 parts, among them J1 DB25_Male_MountingHoles, J10 Conn_Coaxial, J11 Conn_01x02, J12 Conn_Coaxial, J13 Conn_01x02, J14 Conn_01x02, J15 Conn_01x02, J16 Conn_01x02, J17 Conn_01x02, J2 Conn_01x02, J3 Conn_01x02, J4 Conn_01x03, J5 Conn_01x02, J6 Conn_01x03, J7 Conn_Coaxial, J8 Conn_Coaxial, J9 Conn_01x02, U1 L78L05_SOT89

Commit message: wip; busted
Parts:
- removed J15, J16: Conn_01x02, Connector_PinHeader_2.54mm:PinHeader_1x02_P2.54mm_Vertical, symbol Connector_Generic:Conn_01x02
- J1: value DB25_Male_MountingHoles -> Conn_01x02; footprint Connector_Dsub:DSUB-25_Female_Horizontal_P2.77x2.84mm_EdgePinOffset14.56mm_Housed_MountingHolesOffset8.20mm -> Connector_PinHeader_2.54mm:PinHeader_1x02_P2.54mm_Vertical
- J10: renamed from J8; value Conn_Coaxial -> Conn_01x02; footprint Connector_Coaxial:SMA_Amphenol_901-143_Horizontal -> Connector_Phoenix_MSTB:PhoenixContact_MSTBA_2,5_2-G-5,08_1x02_P5.08mm_Horizontal
- J11: renamed from J9; value Conn_01x02 -> DB25_Male_MountingHoles; footprint Connector_PinHeader_2.54mm:PinHeader_1x02_P2.54mm_Vertical -> Connector_Dsub:DSUB-25_Female_Horizontal_P2.77x2.84mm_EdgePinOffset14.56mm_Housed_MountingHolesOffset8.20mm
- J12: renamed from J10; footprint Connector_Coaxial:SMA_Amphenol_901-143_Horizontal -> Connector_Coaxial:SMA_Molex_73251-2200_Horizontal
- J13: renamed from J11; value Conn_01x02 -> Conn_Coaxial; footprint Connector_PinHeader_2.54mm:PinHeader_1x02_P2.54mm_Vertical -> Connector_Coaxial:SMA_Molex_73251-2200_Horizontal
- J14: renamed from J12; value Conn_Coaxial -> Conn_01x02; footprint Connector_Coaxial:SMA_Amphenol_901-143_Horizontal -> Connector_PinHeader_2.54mm:PinHeader_1x02_P2.54mm_Vertical
- J15: renamed from J17; footprint Connector_PinHeader_2.54mm:PinHeader_1x02_P2.54mm_Vertical -> Connector_Phoenix_MSTB:PhoenixContact_MSTBA_2,5_2-G-5,08_1x02_P5.08mm_Horizontal
- J2: value Conn_01x02 -> Conn_01x03; footprint Connector_PinHeader_2.54mm:PinHeader_1x02_P2.54mm_Vertical -> Connector_PinHeader_2.54mm:PinHeader_1x03_P2.54mm_Vertical
- J3: value Conn_01x02 -> Conn_Coaxial; footprint Connector_PinHeader_2.54mm:PinHeader_1x02_P2.54mm_Vertical -> Connector_Coaxial:SMA_Molex_73251-2200_Horizontal
- J4, J6: value Conn_01x03 -> Conn_01x02; footprint Connector_PinHeader_2.54mm:PinHeader_1x03_P2.54mm_Vertical -> Connector_PinHeader_2.54mm:PinHeader_1x02_P2.54mm_Vertical
- J7: value Conn_Coaxial -> Conn_01x02; footprint Connector_Coaxial:SMA_Amphenol_901-143_Horizontal -> Connector_PinHeader_2.54mm:PinHeader_1x02_P2.54mm_Vertical
- J8: renamed from J13; value Conn_01x02 -> Conn_01x03; footprint Connector_PinHeader_2.54mm:PinHeader_1x02_P2.54mm_Vertical -> Connector_PinHeader_2.54mm:PinHeader_1x03_P2.54mm_Vertical
- J9: renamed from J14; value Conn_01x02 -> Conn_Coaxial; footprint Connector_PinHeader_2.54mm:PinHeader_1x02_P2.54mm_Vertical -> Connector_Coaxial:SMA_Molex_73251-2200_Horizontal
- renumbered C3 to C2, C4 to C3, C5 to C4, R5 to R4, R6 to R5, R7 to R6
Connections:
- net +5V: now also J8.2 (Pin_2)
- net GND: no longer J8.2 (Pin_2)

Commit message: .
Parts:
- J1: value Conn_01x02 -> DB25_Male_MountingHoles; footprint Connector_PinHeader_2.54mm:PinHeader_1x02_P2.54mm_Vertical -> Connector_Dsub:DSUB-25_Female_Horizontal_P2.77x2.84mm_EdgePinOffset14.56mm_Housed_MountingHolesOffset8.20mm
- J10: value Conn_01x02 -> Conn_Coaxial; footprint Connector_Phoenix_MSTB:PhoenixContact_MSTBA_2,5_2-G-5,08_1x02_P5.08mm_Horizontal -> Connector_Coaxial:SMA_Molex_73251-2200_Horizontal
- J11: value DB25_Male_MountingHoles -> Conn_01x02; footprint Connector_Dsub:DSUB-25_Female_Horizontal_P2.77x2.84mm_EdgePinOffset14.56mm_Housed_MountingHolesOffset8.20mm -> Connector_PinHeader_2.54mm:PinHeader_1x02_P2.54mm_Vertical
- J13, J3, J9: value Conn_Coaxial -> Conn_01x02; footprint Connector_Coaxial:SMA_Molex_73251-2200_Horizontal -> Connector_PinHeader_2.54mm:PinHeader_1x02_P2.54mm_Vertical
- J14, J7: value Conn_01x02 -> Conn_Coaxial; footprint Connector_PinHeader_2.54mm:PinHeader_1x02_P2.54mm_Vertical -> Connector_Coaxial:SMA_Molex_73251-2200_Horizontal
- J2, J8: value Conn_01x03 -> Conn_01x02; footprint Connector_PinHeader_2.54mm:PinHeader_1x03_P2.54mm_Vertical -> Connector_PinHeader_2.54mm:PinHeader_1x02_P2.54mm_Vertical
- J4, J6: value Conn_01x02 -> Conn_01x03; footprint Connector_PinHeader_2.54mm:PinHeader_1x02_P2.54mm_Vertical -> Connector_PinHeader_2.54mm:PinHeader_1x03_P2.54mm_Vertical
Other:
- moved on the sheet: J10, J11, J12, J13, J14, J3, J4, J5, J7, JP1, JP2, R3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

Commit message: fixed
Parts:
- renumbered C2 to C1, C4 to C2, C1 to C4, J14 to J1, J7 to J10, J10 to J11, J6 to J13, J3 to J14, J11 to J15, J5 to J2, J4 to J3, J8 to J4, J13 to J5, J9 to J6, J2 to J7, J15 to J8, J1 to J9, JP2 to JP1, JP1 to JP2, R3 to R1, R6 to R3, R1 to R4, R4 to R6
