File: projects/z3817a_breakout/z3817a_breakout.kicad_pcb (KiCad board)
At the start: 2 copper layers, 76.2 x 76.2 mm, 35 parts, among them J1 DB25_Male_MountingHoles, J10 Conn_Coaxial, J11 Conn_01x02, J12 Conn_Coaxial, J13 Conn_01x02, J14 Conn_01x02, J15 Conn_01x02, J16 Conn_01x02, J17 Conn_01x02, J2 Conn_01x02, J3 Conn_01x02, J4 Conn_01x03, J5 Conn_01x02, J6 Conn_01x03, J7 Conn_Coaxial, J8 Conn_Coaxial, J9 Conn_01x02, U1 L78L05_SOT89

Commit message: wip; busted
Parts:
- removed C5: 0.1u 10V X7R, Capacitor_SMD:C_0805_2012Metric_Pad1.18x1.45mm_HandSolder
- removed J16: Conn_01x02, Connector_PinHeader_2.54mm:PinHeader_1x02_P2.54mm_Vertical
- removed the J3 at (91.4, 96.5)
- removed the R1 at (72.4, 90.8)
- added C4: 0.1u 10V X7R, Capacitor_SMD:C_0805_2012Metric_Pad1.18x1.45mm_HandSolder, F.Cu at (93.5, 60.0)
- added R6: DNI, Resistor_SMD:R_0603_1608Metric_Pad0.98x0.95mm_HandSolder, F.Cu at (151.5, 51.0)
- C1: renamed from C3; value 0.33u 50V X7R -> DNI
- C2: renamed from C4; value 22u 50V X7S -> 0.33u 50V X7R; footprint Capacitor_SMD:C_2220_5650Metric_Pad1.97x5.40mm_HandSolder -> Capacitor_SMD:C_0805_2012Metric_Pad1.18x1.45mm_HandSolder
- C3: renamed from C1; value DNI -> 22u 50V X7S; footprint Capacitor_SMD:C_0805_2012Metric_Pad1.18x1.45mm_HandSolder -> Capacitor_SMD:C_2220_5650Metric_Pad1.97x5.40mm_HandSolder
- J10: renamed from J17; footprint Connector_PinHeader_2.54mm:PinHeader_1x02_P2.54mm_Vertical -> Connector_Phoenix_MSTB:PhoenixContact_MSTBA_2,5_2-G-5,08_1x02_P5.08mm_Horizontal
- J12: renamed from J7; footprint Connector_Coaxial:SMA_Amphenol_901-143_Horizontal -> Connector_Coaxial:SMA_Molex_73251-2200_Horizontal
- J13: renamed from J8; footprint Connector_Coaxial:SMA_Amphenol_901-143_Horizontal -> Connector_Coaxial:SMA_Molex_73251-2200_Horizontal
- J15: footprint Connector_PinHeader_2.54mm:PinHeader_1x02_P2.54mm_Vertical -> Connector_Phoenix_MSTB:PhoenixContact_MSTBA_2,5_2-G-5,08_1x02_P5.08mm_Horizontal
- J3: renamed from J12; footprint Connector_Coaxial:SMA_Amphenol_901-143_Horizontal -> Connector_Coaxial:SMA_Molex_73251-2200_Horizontal
- J9: renamed from J10; footprint Connector_Coaxial:SMA_Amphenol_901-143_Horizontal -> Connector_Coaxial:SMA_Molex_73251-2200_Horizontal
- R3: renamed from R7; value DNI -> 33
- R4: renamed from R6; value DNI -> 33
- R5: value 33 -> DNI
- moved J6 66.8 mm to (101.6, 30.5)
- moved R5 63.7 mm to (134.0, 54.5)
- moved R1 51.3 mm to (72.4, 85.5), turned to 180 degrees
- moved C3 44.8 mm to (103.0, 54.5), turned to -90 degrees
- moved R3 41.1 mm to (81.5, 37.5)
- moved C1 37.7 mm to (72.5, 83.0)
- moved R4 33.6 mm to (145.5, 65.0), turned to 180 degrees
- moved J15 16.8 mm to (116.7, 46.5)
- moved C2 9.70 mm to (93.5, 52.0), turned to 0 degrees
- moved F1 9.09 mm to (106.5, 46.4)
- moved J10 6.72 mm to (116.7, 46.5), turned to 90 degrees
- moved J5 5.08 mm to (111.8, 30.5)
- moved JP1 2.18 mm to (78.0, 37.2)
- moved JP2 1.84 mm to (78.0, 89.8)
- moved J12 1.28 mm to (122.0, 80.0)
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- renumbered H4 to H1, H1 to H2, H2 to H4, J5 to J1, J1 to J11, J9 to J14, J4 to J2, J11 to J4, J13 to J5, J14 to J6, J2 to J7, J6 to J8, JP2 to JP1, JP1 to JP2, R3 to R1
Connections:
- C1 pad 1: /DCIn -> Net-(C1-Pad1)
- C3 pad 1: Net-(C1-Pad1) -> /DCIn
- J1 pad 1: GND2 -> Net-(J1-Pad1)
- J1 pad 2: GND2 -> /10MHZ_OUT_A+
- J10 pad 1: /DCIn0 -> /10MHZ_OUT_B+
- J10 pad 2: GND -> /10MHZ_OUT_B-
- J11 pad 0: Net-(C1-Pad1) -> (no net)
- J11 pad 1: Net-(J1-Pad1) -> /TIMEREF1_RXD_IN
- J11 pad 10: unconnected-(J1-Pad10) -> (no net)
- J11 pad 11: unconnected-(J1-Pad11) -> (no net)
- J11 pad 12: unconnected-(J1-Pad12) -> (no net)
- J11 pad 13: unconnected-(J1-Pad13) -> (no net)
- J11 pad 14: unconnected-(J1-Pad14) -> (no net)
- J11 pad 15: /10MHZ_OUT_A- -> (no net)
- J11 pad 16: /10MHZ_OUT_B- -> (no net)
- J11 pad 17: unconnected-(J1-Pad17) -> (no net)
- J11 pad 18: GND1 -> (no net)
- J11 pad 19: unconnected-(J1-Pad19) -> (no net)
- J11 pad 2: /10MHZ_OUT_A+ -> GND1
- J11 pad 20: GND2 -> (no net)
- J11 pad 21: Net-(J1-Pad1) -> (no net)
- J11 pad 22: /TIMEREF2_VALID_IN -> (no net)
- J11 pad 23: unconnected-(J1-Pad23) -> (no net)
- J11 pad 24: unconnected-(J1-Pad24) -> (no net)
- J11 pad 25: GND -> (no net)
- J11 pad 3: /10MHZ_OUT_B+ -> (no net)
- J11 pad 4: /TIMEREF1_RXD_IN -> (no net)
- J11 pad 5: /TIMEREF1_PPS_IN -> (no net)
- J11 pad 6: /TIMEREF2_RXD_IN -> (no net)
- J11 pad 7: /TIMEREF2_PPS_IN -> (no net)
- J11 pad 8: GND -> (no net)
- J11 pad 9: /TIMEREF1_VALID_IN -> (no net)
- J12 pad 1: /10MHZ_OUT_A+ -> /TIMEREF1_PPS_IN
- J12 pad 2: /10MHZ_OUT_A- -> GND1
- J13 pad 1: /10MHZ_OUT_B+ -> /TIMEREF2_RXD_IN
- J13 pad 2: /10MHZ_OUT_B- -> GND2
- J14 pad 1: /TIMEREF1_RXD_IN -> /TIMEREF2_PPS_IN
- J14 pad 2: GND1 -> GND2
- J15 pad 1: +5V -> /DCIn0
- J2 pad 1: Net-(J4-Pad1) -> Net-(J1-Pad1)
- J2 pad 2: /TIMEREF2_VALID_IN -> /DCIn
- J2 pad 3: GND2 -> (no net)
- J3 pad 1: /TIMEREF2_PPS_IN -> GND1
- J3 pad 2: GND2 -> GND1
- J4 pad 1: /TIMEREF2_RXD_IN -> Net-(J4-Pad1)
- J4 pad 2: GND2 -> /TIMEREF2_VALID_IN
- J5 pad 1: +5V -> GND2
- J5 pad 2: GND -> GND2
- J6 pad 1: GND -> Net-(J6-Pad1)
- J6 pad 2: GND -> /TIMEREF1_VALID_IN
- J7 pad 1: Net-(J1-Pad1) -> /10MHZ_OUT_A+
- J7 pad 2: /DCIn -> /10MHZ_OUT_A-
- J8 pad 1: Net-(J6-Pad1) -> +5V
- J8 pad 2: /TIMEREF1_VALID_IN -> +5V
- J8 pad 3: GND1 -> (no net)
- J9 pad 1: /TIMEREF1_PPS_IN -> GND
- J9 pad 2: GND1 -> GND
- JP1 pad 2: GND2 -> GND1
- JP2 pad 2: GND1 -> GND2
- R1 pad 1: +5V -> Net-(C1-Pad1)
- R1 pad 2: Net-(J4-Pad1) -> GND
- R3 pad 1: /10MHZ_OUT_B- -> +5V
- R3 pad 2: GND -> Net-(J4-Pad1)
- R4 pad 1: /10MHZ_OUT_A- -> +5V
- R4 pad 2: GND -> Net-(J6-Pad1)
- R5 pad 1: +5V -> /10MHZ_OUT_A-
- R5 pad 2: Net-(J6-Pad1) -> GND
Routing:
- net GND: track 0.00 -> 133.7 mm
- net GND1: track 34.4 -> 127.2 mm
- net Net-(C1-Pad1): track 64.1 -> 0.00 mm
- net /10MHZ_OUT_B-: track 64.1 -> 0.00 mm
- net /10MHZ_OUT_A-: track 61.3 -> 0.00 mm
- net /10MHZ_OUT_B+: track 58.1 -> 0.00 mm
- net Net-(J4-Pad1): track 3.81 -> 55.3 mm, vias 0 -> 1
- net /TIMEREF1_VALID_IN: track 49.4 -> 0.00 mm, vias 2 -> 0
- net +5V: track 107.5 -> 154.6 mm, vias 5 -> 10
- net Net-(J1-Pad1): track 35.6 -> 0.00 mm
- net /TIMEREF2_VALID_IN: track 35.4 -> 0.00 mm
- net /TIMEREF1_RXD_IN: track 34.0 -> 0.00 mm
- net /DCIn: track 46.2 -> 77.3 mm
- net GND2: track 30.6 -> 57.3 mm
- net /10MHZ_OUT_A+: track 56.3 -> 35.4 mm
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- added copper zone on B.Cu, net GND1
- added copper zone on B.Cu, net GND2
Other:
- board size 76.2 x 76.2 mm -> 77.3 x 76.2 mm
- board text added: "10 MHz A"
- board text added: "10 MHz B"
- board text added: "18-36V"
- board text added: "5V"
- board text added: "EN/OFF"
- board text added: "GND"
- board text added: "PPS_IN"
- board text added: "RETURN"
- board text added: "RXD_IN"
- board text added: "TIMEREF1"
- board text added: "TIMEREF2"

Commit message: .
Parts:
- removed the J10 at (116.7, 46.5)
- added J11: Conn_01x02, Connector_PinHeader_2.54mm:PinHeader_1x02_P2.54mm_Vertical, F.Cu at (92.0, 96.6)
- moved R4 66.9 mm to (83.4, 89.8), turned to -90 degrees
- moved R6 38.9 mm to (113.5, 59.4), turned to 180 degrees
- moved R5 37.8 mm to (113.5, 86.2), turned to 180 degrees
- turned C1 to 0 degrees
- turned C2 to 180 degrees
- turned R1 to 0 degrees
- renumbered J11 to J1, J13 to J10, J9 to J12, J4 to J13, J3 to J14, J7 to J2, J14 to J3, J2 to J4, J1 to J5, J8 to J6, J12 to J7, J5 to J8, J6 to J9, JP2 to JP1, JP1 to JP2
Connections:
- J1 pad 0: (no net) -> Net-(C1-Pad1)
- J1 pad 1: /TIMEREF1_RXD_IN -> Net-(J1-Pad1)
- J1 pad 10: (no net) -> unconnected-(J1-Pad10)
- J1 pad 11: (no net) -> unconnected-(J1-Pad11)
- J1 pad 12: (no net) -> unconnected-(J1-Pad12)
- J1 pad 13: (no net) -> unconnected-(J1-Pad13)
- J1 pad 14: (no net) -> unconnected-(J1-Pad14)
- J1 pad 15: (no net) -> /10MHZ_OUT_A-
- J1 pad 16: (no net) -> /10MHZ_OUT_B-
- J1 pad 17: (no net) -> unconnected-(J1-Pad17)
- J1 pad 18: (no net) -> GND1
- J1 pad 19: (no net) -> unconnected-(J1-Pad19)
- J1 pad 2: GND1 -> /10MHZ_OUT_A+
- J1 pad 20: (no net) -> GND2
- J1 pad 21: (no net) -> Net-(J1-Pad1)
- J1 pad 22: (no net) -> /TIMEREF2_VALID_IN
- J1 pad 23: (no net) -> unconnected-(J1-Pad23)
- J1 pad 24: (no net) -> unconnected-(J1-Pad24)
- J1 pad 25: (no net) -> GND
- J1 pad 3: (no net) -> /10MHZ_OUT_B+
- J1 pad 4: (no net) -> /TIMEREF1_RXD_IN
- J1 pad 5: (no net) -> /TIMEREF1_PPS_IN
- J1 pad 6: (no net) -> /TIMEREF2_RXD_IN
- J1 pad 7: (no net) -> /TIMEREF2_PPS_IN
- J1 pad 8: (no net) -> GND
- J1 pad 9: (no net) -> /TIMEREF1_VALID_IN
- J10 pad 1: /TIMEREF2_RXD_IN -> /10MHZ_OUT_B+
- J10 pad 2: GND2 -> /10MHZ_OUT_B-
- J12 pad 1: GND -> /TIMEREF1_PPS_IN
- J12 pad 2: GND -> GND1
- J13 pad 1: Net-(J4-Pad1) -> /TIMEREF2_RXD_IN
- J13 pad 2: /TIMEREF2_VALID_IN -> GND2
- J14 pad 1: GND1 -> /TIMEREF2_PPS_IN
- J14 pad 2: GND1 -> GND2
- J2 pad 1: /10MHZ_OUT_A+ -> Net-(J1-Pad1)
- J2 pad 2: /10MHZ_OUT_A- -> /DCIn
- J3 pad 1: /TIMEREF2_PPS_IN -> GND1
- J3 pad 2: GND2 -> GND1
- J4 pad 1: Net-(J1-Pad1) -> Net-(J4-Pad1)
- J4 pad 2: /DCIn -> /TIMEREF2_VALID_IN
- J4 pad 3: (no net) -> GND2
- J5 pad 1: Net-(J1-Pad1) -> GND2
- J5 pad 2: /10MHZ_OUT_A+ -> GND2
- J6 pad 1: +5V -> Net-(J6-Pad1)
- J6 pad 2: +5V -> /TIMEREF1_VALID_IN
- J6 pad 3: (no net) -> GND1
- J7 pad 1: /TIMEREF1_PPS_IN -> /10MHZ_OUT_A+
- J7 pad 2: GND1 -> /10MHZ_OUT_A-
- J8 pad 1: GND2 -> +5V
- J8 pad 2: GND2 -> +5V
- J9 pad 1: Net-(J6-Pad1) -> GND
- J9 pad 2: /TIMEREF1_VALID_IN -> GND
- JP1 pad 2: GND2 -> GND1
- JP2 pad 2: GND1 -> GND2
Routing:
- net GND: track 133.7 -> 0.00 mm
- net GND1: track 127.2 -> 34.4 mm
- net Net-(C1-Pad1): track 0.00 -> 63.8 mm
- net /10MHZ_OUT_B+: track 0.00 -> 58.6 mm, vias 0 -> 1
- net /10MHZ_OUT_B-: track 0.00 -> 58.4 mm, vias 0 -> 1
- net +5V: track 154.6 -> 97.1 mm, vias 10 -> 5
- net /10MHZ_OUT_A-: track 0.00 -> 57.3 mm, vias 0 -> 1
- net /TIMEREF1_RXD_IN: track 0.00 -> 49.7 mm, vias 0 -> 1
- net /TIMEREF1_VALID_IN: track 0.00 -> 49.4 mm, vias 0 -> 2
- net Net-(J4-Pad1): track 55.3 -> 6.28 mm
- net Net-(J1-Pad1): track 0.00 -> 35.4 mm
- net /DCIn: track 77.3 -> 42.0 mm
- net /TIMEREF2_VALID_IN: track 0.00 -> 35.4 mm
- net GND2: track 57.3 -> 30.6 mm
- net /10MHZ_OUT_A+: track 35.4 -> 55.8 mm, vias 0 -> 1
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
Commit message: fixed
Parts:
- R4: renamed from R1; value 33 -> DNI
- renumbered C2 to C1, C4 to C2, C1 to C4, J14 to J1, J7 to J10, J10 to J11, J6 to J13, J3 to J14, J11 to J15, J5 to J2, J4 to J3, J8 to J4, J13 to J5, J9 to J6, J2 to J7, J15 to J8, J1 to J9, JP2 to JP1, JP1 to JP2, R3 to R1, R6 to R3, R4 to R6

Commit message: .
Parts:
- removed J7: Conn_01x02, Connector_PinHeader_2.54mm:PinHeader_1x02_P2.54mm_Vertical
- removed R2: 0, Resistor_SMD:R_0603_1608Metric_Pad0.98x0.95mm_HandSolder
- moved ? 1.87 mm to (81.5, 89.9)
- moved J5 0.64 mm to (92.1, 30.5)
- moved R1 0.17 mm to (81.5, 37.3)
- moved J15 0.13 mm to (92.1, 96.5)
- moved JP1 0.09 mm to (78.0, 37.3)
- renumbered R6 to ?
Connections:
- J9 pad 1: Net-(J9-Pad1) -> /DCIn
- J9 pad 21: Net-(J9-Pad1) -> /DCIn
Routing:
- net Net-(J9-Pad1): track 35.4 -> 0.00 mm
- net /DCIn: track 42.0 -> 76.7 mm, vias 1 -> 0
- net +5V: track 97.1 -> 99.0 mm
- net /TIMEREF1_VALID_IN: track 49.4 -> 48.7 mm
- net GND2: track 30.6 -> 31.2 mm
- net /TIMEREF2_PPS_IN: track 40.2 -> 40.8 mm
- net GND: vias 0 -> 58

Commit message: .
Parts:
- J9: footprint Connector_Dsub:DSUB-25_Female_Horizontal_P2.77x2.84mm_EdgePinOffset14.56mm_Housed_MountingHolesOffset8.20mm -> Connector_Dsub:DSUB-25_Female_Horizontal_P2.77x2.84mm_EdgePinOffset7.70mm_Housed_MountingHolesOffset9.12mm
- moved R4 7.82 mm to (64.6, 85.0)
- moved C4 7.80 mm to (64.7, 83.1)
- moved J9 7.62 mm to (59.7, 80.0)
- moved C1 0.32 mm to (93.8, 52.0)
- moved C2 0.32 mm to (93.8, 60.0)
- gave numbers to parts that had none: 1
Connections:
- net Net-(C4-Pad1) renamed /CONNSHIELD
Routing:
- net /DCIn: track 76.7 -> 86.8 mm
- net /10MHZ_OUT_B-: track 58.4 -> 66.0 mm
- net /10MHZ_OUT_B+: track 58.6 -> 66.2 mm
- net /10MHZ_OUT_A+: track 55.8 -> 63.5 mm
- net /10MHZ_OUT_A-: track 57.3 -> 65.0 mm
- net /TIMEREF1_VALID_IN: track 48.7 -> 56.3 mm
- net /TIMEREF2_VALID_IN: track 35.4 -> 41.7 mm
- net GND2: track 31.2 -> 37.5 mm
- net /TIMEREF2_RXD_IN: track 49.0 -> 55.0 mm
- net /TIMEREF1_PPS_IN: track 35.4 -> 41.3 mm
- net /TIMEREF2_PPS_IN: track 40.8 -> 46.3 mm
- net GND1: track 34.4 -> 39.0 mm
- net /CONNSHIELD: track 63.8 -> 59.8 mm
- net /TIMEREF1_RXD_IN: track 49.7 -> 52.8 mm
- net GND: vias 58 -> 86
Other:
- board size 77.3 x 76.2 mm -> 77.3 x 76.3 mm
- board text added: "Murgatroid Heavy Industries, LLC"
- board text added: "Z3817A Interface V1.0 ch@murgatroid.com"
