File: projects/pdp11_front_panel/ltc.kicad_sch (KiCad schematic)
At the start: 7 parts

Commit message: .
Parts:
- added JP2: Jumper_2_Open, symbol Jumper:Jumper_2_Open
- Q3: renamed from Q?; value DNI/MMBT3904 -> 3904
- gave numbers to parts that had none: 6
Connections:
- net BEVENT_L: no longer names the net of Q3.3 (C), R20.2
- net BEVENT_L: now also JP2.1 (A)
