File: projects/pdp11_front_panel/debounced_switch.kicad_sch (KiCad schematic)
At the start: 5 parts, among them SW2 SW_SPDT, U4 SN74LVC1G14DBV, U5 SN74LVC1G14DBV

Commit message: wip
Parts:
- renumbered C5 to C1, C6 to C2, SW2 to SW1, U5 to U1, U4 to U2
Changed lines of the file:
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@@
+    (stroke (width 0) (type default))
+  )
+  (wire (pts (xy 80.01 109.22) (xy 82.55 109.22))
     (stroke (width 0) (type default))
   )
@@
     (stroke (width 0) (type default))
   )
+  (wire (pts (xy 82.55 109.22) (xy 82.55 114.3))
+    (stroke (width 0) (type default))
+  )
   (wire (pts (xy 97.79 81.28) (xy 104.14 81.28))
     (stroke (width 0) (type default))
@@
     (stroke (width 0) (type default))
   )
-  (wire (pts (xy 111.76 107.95) (xy 111.76 111.76))
+  (wire (pts (xy 111.76 107.95) (xy 111.76 114.3))
     (stroke (width 0) (type default))
   )
@@
     (effects (font (size 1.27 1.27)) (justify left))
   )
-  (hierarchical_label "GND" (shape passive) (at 111.76 111.76 270) (fields_autoplaced)
+  (hierarchical_label "GND" (shape passive) (at 80.01 109.22 180) (fields_autoplaced)
     (effects (font (size 1.27 1.27)) (justify right))
   )
   (symbol (lib_id "Device:C") (at 152.4 71.12 0) (unit 1)
     (in_bom yes) (on_board yes) (dnp no) (fields_autoplaced)
-    (property "Reference" "C6" (at 156.21 69.85 0)
+    (property "Reference" "C2" (at 156.21 69.85 0)
       (effects (font (size 1.27 1.27)) (justify left))
     )
@@
           (reference "C6") (unit 1)
         )
-        (path "/e63e39d7-6ac0-4ffd-8aa3-1841a4541b55/48ec5c41-bdf1-45f7-9034-4defa6aa7296"
+        (path "/e63e39d7-6ac0-4ffd-8aa3-1841a4541b55/25fe9e03-a231-44dc-96d1-9307cff67739"
           (reference "C8") (unit 1)
         )
@@
   (symbol (lib_id "Switch:SW_SPDT") (at 90.17 88.9 0) (unit 1)
     (in_bom yes) (on_board yes) (dnp no)
-    (property "Reference" "SW2" (at 85.09 82.55 0)
+    (property "Reference" "SW1" (at 85.09 82.55 0)
       (effects (font (size 1.27 1.27)))
     )
@@
           (reference "SW2") (unit 1)
         )
-        (path "/e63e39d7-6ac0-4ffd-8aa3-1841a4541b55/48ec5c41-bdf1-45f7-9034-4defa6aa7296"
+        (path "/e63e39d7-6ac0-4ffd-8aa3-1841a4541b55/25fe9e03-a231-44dc-96d1-9307cff67739"
           (reference "SW3") (unit 1)
         )
@@
   (symbol (lib_id "power:GND") (at 81.28 91.44 0) (unit 1)
     (in_bom yes) (on_board yes) (dnp no) (fields_autoplaced)
-    (property "Reference" "#PWR0109" (at 81.28 97.79 0)
+    (property "Reference" "#PWR014" (at 81.28 97.79 0)
       (effects (font (size 1.27 1.27)) hide)
     )
@@
           (reference "#PWR05") (unit 1)
         )
-        (path "/e63e39d7-6ac0-4ffd-8aa3-1841a4541b55/48ec5c41-bdf1-45f7-9034-4defa6aa7296"
+        (path "/e63e39d7-6ac0-4ffd-8aa3-1841a4541b55/25fe9e03-a231-44dc-96d1-9307cff67739"
           (reference "#PWR015") (unit 1)
         )
@@
   (symbol (lib_id "Device:C") (at 143.51 71.12 0) (unit 1)
     (in_bom yes) (on_board yes) (dnp no) (fields_autoplaced)
-    (property "Reference" "C5" (at 147.32 69.85 0)
+    (property "Reference" "C1" (at 147.32 69.85 0)
       (effects (font (size 1.27 1.27)) (justify left))
     )
@@
           (reference "C5") (unit 1)
         )
-        (path "/e63e39d7-6ac0-4ffd-8aa3-1841a4541b55/48ec5c41-bdf1-45f7-9034-4defa6aa7296"
+        (path "/e63e39d7-6ac0-4ffd-8aa3-1841a4541b55/25fe9e03-a231-44dc-96d1-9307cff67739"
           (reference "C7") (unit 1)
         )
@@
   (symbol (lib_id "74xGxx:SN74LVC1G14DBV") (at 111.76 96.52 0) (unit 1)
     (in_bom yes) (on_board yes) (dnp no)
-    (property "Reference" "U5" (at 99.695 99.695 0)
+    (property "Reference" "U1" (at 99.695 99.695 0)
       (effects (font (size 1.27 1.27)))
     )
@@
           (reference "U4") (unit 1)
         )
-        (path "/e63e39d7-6ac0-4ffd-8aa3-1841a4541b55/48ec5c41-bdf1-45f7-9034-4defa6aa7296"
+        (path "/e63e39d7-6ac0-4ffd-8aa3-1841a4541b55/25fe9e03-a231-44dc-96d1-9307cff67739"
           (reference "U6") (unit 1)
+        )
+      )
+    )
+  )
+  (symbol (lib_name "GND_1") (lib_id "power:GND") (at 111.76 114.3 0) (unit 1)
+    (in_bom yes) (on_board yes) (dnp no) (fields_autoplaced)
+    (property "Reference" "#PWR018" (at 111.76 120.65 0)
+      (effects (font (size 1.27 1.27)) hide)
+    )
+    (property "Value" "GND" (at 111.76 119.38 0)
+      (effects (font (size 1.27 1.27)))
+    )
+    (property "Footprint" "" (at 111.76 114.3 0)
+      (effects (font (size 1.27 1.27)) hide)
+    )
+    (property "Datasheet" "" (at 111.76 114.3 0)
+      (effects (font (size 1.27 1.27)) hide)
+    )
+    (pin "1")
+    (instances
+      (project "pdp11_front_panel"
+        (path "/e63e39d7-6ac0-4ffd-8aa3-1841a4541b55/ee444592-02b9-4a6d-bd44-edb99a2cfe0b"
+          (reference "#PWR018") (unit 1)
+        )
+        (path "/e63e39d7-6ac0-4ffd-8aa3-1841a4541b55/25fe9e03-a231-44dc-96d1-9307cff67739"
+          (reference "#PWR019") (unit 1)
+        )
+        (path "/e63e39d7-6ac0-4ffd-8aa3-1841a4541b55/48854766-3438-4455-aaf3-36ea48f913cb"
+          (reference "#PWR020") (unit 1)
         )
       )
@@
   (symbol (lib_id "74xGxx:SN74LVC1G14DBV") (at 121.92 81.28 0) (unit 1)
     (in_bom yes) (on_board yes) (dnp no)
-    (property "Reference" "U4" (at 131.445 74.295 0)
+    (property "Reference" "U2" (at 131.445 74.295 0)
       (effects (font (size 1.27 1.27)))
     )
@@
           (reference "U5") (unit 1)
         )
-        (path "/e63e39d7-6ac0-4ffd-8aa3-1841a4541b55/48ec5c41-bdf1-45f7-9034-4defa6aa7296"
+        (path "/e63e39d7-6ac0-4ffd-8aa3-1841a4541b55/25fe9e03-a231-44dc-96d1-9307cff67739"
           (reference "U7") (unit 1)
         )
       )
+    )
+  )
+  (symbol (lib_name "GND_1") (lib_id "power:GND") (at 82.55 114.3 0) (unit 1)
+    (in_bom yes) (on_board yes) (dnp no) (fields_autoplaced)
+    (property "Reference" "#PWR021" (at 82.55 120.65 0)
+      (effects (font (size 1.27 1.27)) hide)
+    )
+    (property "Value" "GND" (at 82.55 119.38 0)
+      (effects (font (size 1.27 1.27)))
+    )
+    (property "Footprint" "" (at 82.55 114.3 0)
+      (effects (font (size 1.27 1.27)) hide)
+    )
+    (property "Datasheet" "" (at 82.55 114.3 0)
+      (effects (font (size 1.27 1.27)) hide)
+    )
+    (pin "1")
+    (instances
+      (project "pdp11_front_panel"
+        (path "/e63e39d7-6ac0-4ffd-8aa3-1841a4541b55/ee444592-02b9-4a6d-bd44-edb99a2cfe0b"
+          (reference "#PWR021") (unit 1)
+        )
+        (path "/e63e39d7-6ac0-4ffd-8aa3-1841a4541b55/25fe9e03-a231-44dc-96d1-9307cff67739"
+          (reference "#PWR022") (unit 1)
+        )
+        (path "/e63e39d7-6ac0-4ffd-8aa3-1841a4541b55/48854766-3438-4455-aaf3-36ea48f913cb"
+          (reference "#PWR023") (unit 1)
+        )
+      )
