File: projects/pdp11_front_panel/bus_driver_translator.kicad_sch (KiCad schematic)
At the start: 4 parts, among them U3 74LVC1G07

Commit message: WIP.
Parts:
- added C5: 0.1u, symbol Device:C
- added U2: SN74LV1T34DBV, Package_TO_SOT_SMD:SOT-23-5, symbol Logic_LevelTranslator:SN74LV1T34DBV
- renumbered C3 to C1, R13 to R14, R12 to R2
Connections:
- net BUS: now also U2.2 (A)
- net GND: now also C5.2, U2.3 (GND)
- net VDD_XLATED: now also C5.1, U2.5 (VCC)
- new net BUS_XLATED: U2.4 (Y)
