File: projects/pdp11_front_panel/bus_translator.kicad_sch (KiCad schematic)
At the start: 3 parts, among them U2 SN74LV1T34DBV

Commit message: WIP.
Parts:
- renumbered C2 to C4, R2 to R13
Changed lines of the file:
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@@
   (symbol (lib_id "Device:C") (at 119.38 95.25 0) (unit 1)
     (in_bom yes) (on_board yes) (dnp no) (fields_autoplaced)
-    (property "Reference" "C2" (at 123.19 93.98 0)
+    (property "Reference" "C4" (at 123.19 93.98 0)
       (effects (font (size 1.27 1.27)) (justify left))
     )
@@
   (symbol (lib_id "Device:R") (at 149.86 68.58 0) (unit 1)
     (in_bom yes) (on_board yes) (dnp no) (fields_autoplaced)
-    (property "Reference" "R2" (at 152.4 67.31 0)
+    (property "Reference" "R13" (at 152.4 67.31 0)
       (effects (font (size 1.27 1.27)) (justify left))
     )
