File: projects/pdp11_front_panel/pdp11_front_panel.kicad_sch (KiCad schematic)
At the start: 0 parts

Commit message: .
Other:
- sheet Backplane Connection ports: added H9XX_CONN; removed BDCOK_H, BEVNT_L, BHALT_L, BPOK_H, SRUN_L
Changed lines of the file:
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@@
   (junction (at 86.995 43.18) (diameter 0) (color 0 0 0 0)
   )
-  (wire (pts (xy 176.53 39.37) (xy 189.23 39.37))
-    (stroke (width 0) (type default) (color 0 0 0 0))
-  )
-  (wire (pts (xy 142.24 50.8) (xy 125.095 50.8))
-    (stroke (width 0) (type default) (color 0 0 0 0))
-  )
-  (wire (pts (xy 125.095 46.99) (xy 125.095 29.845))
-    (stroke (width 0) (type default) (color 0 0 0 0))
-  )
-  (wire (pts (xy 125.095 50.8) (xy 125.095 59.055))
-    (stroke (width 0) (type default) (color 0 0 0 0))
-  )
   (wire (pts (xy 86.995 29.845) (xy 86.995 43.18))
     (stroke (width 0) (type default) (color 0 0 0 0))
   )
-  (wire (pts (xy 132.715 43.18) (xy 132.715 73.025))
-    (stroke (width 0) (type default) (color 0 0 0 0))
-  )
-  (wire (pts (xy 135.89 39.37) (xy 135.89 28.575))
-    (stroke (width 0) (type default) (color 0 0 0 0))
-  )
-  (wire (pts (xy 142.24 39.37) (xy 135.89 39.37))
-    (stroke (width 0) (type default) (color 0 0 0 0))
-  )
-  (wire (pts (xy 91.44 59.055) (xy 91.44 72.39))
-    (stroke (width 0) (type default) (color 0 0 0 0))
-  )
-  (wire (pts (xy 91.44 72.39) (xy 86.36 72.39))
-    (stroke (width 0) (type default) (color 0 0 0 0))
-  )
   (wire (pts (xy 86.995 43.18) (xy 96.52 43.18))
     (stroke (width 0) (type default) (color 0 0 0 0))
   )
-  (wire (pts (xy 142.24 43.18) (xy 132.715 43.18))
-    (stroke (width 0) (type default) (color 0 0 0 0))
-  )
   (wire (pts (xy 77.47 43.18) (xy 86.995 43.18))
     (stroke (width 0) (type default) (color 0 0 0 0))
@@
     (stroke (width 0) (type default) (color 0 0 0 0))
   )
-  (wire (pts (xy 125.095 59.055) (xy 91.44 59.055))
-    (stroke (width 0) (type default) (color 0 0 0 0))
-  )
-  (wire (pts (xy 142.24 46.99) (xy 125.095 46.99))
-    (stroke (width 0) (type default) (color 0 0 0 0))
-  )
-  (wire (pts (xy 132.715 73.025) (xy 126.365 73.025))
+  (bus (pts (xy 132.715 43.18) (xy 144.145 43.18))
     (stroke (width 0) (type default) (color 0 0 0 0))
   )
@@
     (effects (font (size 1.27 1.27)) (justify left bottom))
   )
-  (symbol (lib_id "power:+5V") (at 135.89 28.575 0) (unit 1)
-    (in_bom yes) (on_board yes) (fields_autoplaced)
-    (property "Reference" "#PWR?" (id 0) (at 135.89 32.385 0)
-      (effects (font (size 1.27 1.27)) hide)
-    )
-    (property "Value" "+5V" (id 1) (at 135.89 22.86 0))
-    (property "Footprint" "" (id 2) (at 135.89 28.575 0)
-      (effects (font (size 1.27 1.27)) hide)
-    )
-    (property "Datasheet" "" (id 3) (at 135.89 28.575 0)
-      (effects (font (size 1.27 1.27)) hide)
-    )
-    (pin "1")
-  )
-  (sheet (at 189.23 36.195) (size 21.59 12.065) (fields_autoplaced)
+  (sheet (at 167.64 55.88) (size 21.59 12.065) (fields_autoplaced)
     (stroke (width 0.1524) (type solid) (color 0 0 0 0))
     (fill (color 0 0 0 0.0000))
-    (property "Sheet name" "SRUN Annunciator" (id 0) (at 189.23 35.4834 0)
+    (property "Sheet name" "SRUN Annunciator" (id 0) (at 167.64 55.1684 0)
       (effects (font (size 1.27 1.27)) (justify left bottom))
     )
-    (property "Sheet file" "srun_annunciator.kicad_sch" (id 1) (at 189.23 48.8446 0)
+    (property "Sheet file" "srun_annunciator.kicad_sch" (id 1) (at 167.64 68.5296 0)
       (effects (font (size 1.27 1.27)) (justify left top))
     )
-    (pin "SRUN_L" input (at 189.23 39.37 180)
+    (pin "SRUN_L" input (at 167.64 59.055 180)
       (effects (font (size 1.27 1.27)) (justify left))
     )
   )
-  (sheet (at 142.24 35.56) (size 35.56 19.05) (fields_autoplaced)
+  (sheet (at 144.145 39.37) (size 30.48 8.255) (fields_autoplaced)
     (stroke (width 0.1524) (type solid) (color 0 0 0 0))
     (fill (color 0 0 0 0.0000))
-    (property "Sheet name" "Backplane Connection" (id 0) (at 142.24 34.8484 0)
+    (property "Sheet name" "Backplane Connection" (id 0) (at 144.145 38.6584 0)
       (effects (font (size 1.27 1.27)) (justify left bottom))
     )
-    (property "Sheet file" "backplane_connection.kicad_sch" (id 1) (at 142.24 55.1946 0)
+    (property "Sheet file" "backplane_connection.kicad_sch" (id 1) (at 144.145 48.2096 0)
       (effects (font (size 1.27 1.27)) (justify left top))
     )
-    (pin "SRUN_L" output (at 177.8 39.37 0)
-      (effects (font (size 1.27 1.27)) (justify right))
-    )
-    (pin "BDCOK_H" input (at 142.24 39.37 180)
-      (effects (font (size 1.27 1.27)) (justify left))
-    )
-    (pin "BEVNT_L" input (at 142.24 43.18 180)
-      (effects (font (size 1.27 1.27)) (justify left))
-    )
-    (pin "BPOK_H" input (at 142.24 46.99 180)
-      (effects (font (size 1.27 1.27)) (justify left))
-    )
-    (pin "BHALT_L" input (at 142.24 50.8 180)
+    (pin "H9XX_CONN" bidirectional (at 144.145 43.18 180)
       (effects (font (size 1.27 1.27)) (justify left))
     )
@@
       (reference "#PWR?") (unit 1) (value "VCC") (footprint "")
     )
-    (path "/f19791a4-61c6-4121-a491-c7fb6c038267"
-      (reference "#PWR?") (unit 1) (value "+5V") (footprint "")
-    )
     (path "/847f4119-abc7-484f-b3c7-1ea238d60dea/6a93bd1d-665d-4667-86ac-14d92afa413f"

Commit message: .
Other:
- added sheet Backplane Power (backplane_power.kicad_sch)
- added sheet Power Button (power_button.kicad_sch)
- sheet ATX Power ports: added +12V, +3V3, +5V, +5VSB, -12V, GND; removed none
- sheet BHALT ports: added +5VA, GND; removed none
- sheet Backplane Connection ports: added GND; removed none
- sheet LTC ports: added +5VA, BEVNT_L, GND; removed BEVENT_L
- sheet Power LEDs ports: added +12V, +3V3, +5V, +5VSB, -12V, GND; removed none
- sheet SRUN Annunciator ports: added +5VA, GND; removed none

Commit message: wip
Connections:
- no-connect marks 0 -> 1
Other:
- removed sheet BHALT
- removed sheet LTC
- removed sheet Power Button
- added sheet Debounced Switch (debounced_switch.kicad_sch)
- added sheet Debounced Switch1 (debounced_switch.kicad_sch)
- added sheet Debounced Switch2 (debounced_switch.kicad_sch)

Commit message: wip
Other:
- added sheet LineClock (line_clock.kicad_sch)
- added sheet PowerSequence (power_sequence.kicad_sch)
- sheet ATX Power ports: added ATX_OUT; removed +12V, +3V3, +5V, +5VSB, -12V, ATX_PWR_OK
- sheet Power LEDs ports: added ATX_IN; removed +12V, +3V3, +5V, +5VSB, -12V, ATX_PWR_OK
- note removed: "Power reset via BPOK_H here."

Commit message: wip
Connections:
- no-connect marks 1 -> 0
Other:
- sheet ATX Power renamed ATX Power Connector
- removed sheet Debounced Switch
- removed sheet Debounced Switch1
- removed sheet Debounced Switch2
- removed sheet LineClock
- removed sheet PowerSequence
- removed sheet SRUN Annunciator
- added sheet Bus Interface (bus_interface.kicad_sch)
- added sheet Controller (controller.kicad_sch)
- added sheet Front Panel Connection (optional) (backplane_connection.kicad_sch)

Commit message: WIP.
Other:
- sheet Controller ports: added none; removed H9XX_CONN
Changed lines of the file:
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@@
 (kicad_sch (version 20230121) (generator eeschema)
   (paper "A4")
-  (junction (at 233.68 114.3) (diameter 0) (color 0 0 0 0)
+  (junction (at 233.68 133.35) (diameter 0) (color 0 0 0 0)
   )
   (bus_entry (at 107.95 34.29) (size 2.54 2.54)
@@
     (stroke (width 0) (type default))
   )
-  (bus (pts (xy 184.15 114.3) (xy 233.68 114.3))
+  (bus (pts (xy 219.71 118.11) (xy 219.71 114.3))
+    (stroke (width 0) (type default))
+  )
+  (bus (pts (xy 233.68 114.3) (xy 233.68 133.35))
+    (stroke (width 0) (type default))
+  )
+  (bus (pts (xy 172.72 133.35) (xy 233.68 133.35))
     (stroke (width 0) (type default))
   )
@@
     (stroke (width 0) (type default))
   )
+  (bus (pts (xy 147.32 118.11) (xy 219.71 118.11))
+    (stroke (width 0) (type default))
+  )
   (bus (pts (xy 82.55 34.29) (xy 107.95 34.29))
     (stroke (width 0) (type default))
@@
     (stroke (width 0) (type default))
   )
+  (bus (pts (xy 233.68 133.35) (xy 233.68 140.97))
+    (stroke (width 0) (type default))
+  )
   (bus (pts (xy 115.57 34.29) (xy 123.19 34.29))
     (stroke (width 0) (type default))
   )
+  (bus (pts (xy 107.5719 114.3) (xy 104.14 114.3))
+    (stroke (width 0) (type default))
+  )
   (wire (pts (xy 257.81 147.32) (xy 257.81 152.4))
     (stroke (width 0) (type default))
   )
-  (wire (pts (xy 257.81 120.65) (xy 257.81 125.73))
+  (bus (pts (xy 147.32 130.81) (xy 151.13 130.81))
     (stroke (width 0) (type default))
   )
-  (bus (pts (xy 233.68 114.3) (xy 233.68 140.97))
+  (wire (pts (xy 257.81 120.65) (xy 257.81 125.73))
     (stroke (width 0) (type default))
   )
@@
     (stroke (width 0) (type default))
   )
+  (bus (pts (xy 107.5719 114.308) (xy 107.5719 114.3))
+    (stroke (width 0) (type default))
+  )
   (wire (pts (xy 68.58 113.03) (xy 63.5 113.03))
     (stroke (width 0) (type default))
@@
     (stroke (width 0) (type default))
   )
+  (bus (pts (xy 147.32 130.81) (xy 147.32 118.11))
+    (stroke (width 0) (type default))
+  )
   (wire (pts (xy 118.11 64.77) (xy 149.86 64.77))
     (stroke (width 0) (type default))
@@
     (stroke (width 0) (type default))
   )
+  (bus (pts (xy 219.71 114.3) (xy 107.95 114.3))
+    (stroke (width 0) (type default))
+  )
   (image (at 243.205 67.31) (scale 0.283011)
     (data
@@
     (effects (font (size 1.27 1.27)) (justify left bottom))
   )
+  (label "{X_SRUN_L,X_BEVNT_L,X_BEVENT_L_DRIVE,X_BDCOK_H,X_BDCOK_H_DRIVE,X_BPOK_H_DRIVE,X_BHALT_L,X_BHALT_L_DRIVE}"
+    (at 107.95 114.3 0) (fields_autoplaced)
+    (effects (font (size 1.27 1.27)) (justify left bottom))
+  )
   (label "-12V" (at 110.49 36.83 0) (fields_autoplaced)
     (effects (font (size 1.27 1.27)) (justify left bottom))
   )
-  (label "{SRUN_L,BEVNT_L,BDCOK_H,BPOK_H,BHALT_L}" (at 187.96 114.3 0) (fields_autoplaced)
+  (label "{SRUN_L,BEVNT_L,BDCOK_H,BPOK_H,BHALT_L}" (at 175.26 133.35 0) (fields_autoplaced)
     (effects (font (size 1.27 1.27)) (justify left bottom))
   )
@@
       (effects (font (size 1.27 1.27)) (justify left))
     )
-    (pin "H9XX_CONN" bidirectional (at 104.14 114.3 0)
-      (effects (font (size 1.27 1.27)) (justify right))
-    )
     (pin "ATX_PS_ON#" output (at 104.14 119.38 0)
       (effects (font (size 1.27 1.27)) (justify right))
@@
     )
   )
-  (sheet (at 162.56 109.22) (size 21.59 10.16) (fields_autoplaced)
+  (sheet (at 151.13 128.27) (size 21.59 10.16) (fields_autoplaced)
     (stroke (width 0.1524) (type solid))
     (fill (color 0 0 0 0.0000))
-    (property "Sheetname" "Bus Interface" (at 162.56 108.5084 0)
+    (property "Sheetname" "Bus Interface" (at 151.13 127.5584 0)
       (effects (font (size 1.27 1.27)) (justify left bottom))
     )
-    (property "Sheetfile" "bus_interface.kicad_sch" (at 162.56 119.9646 0)
+    (property "Sheetfile" "bus_interface.kicad_sch" (at 151.13 139.0146 0)
       (effects (font (size 1.27 1.27)) (justify left top))
     )
-    (pin "H9XX_CONN" bidirectional (at 184.15 114.3 0)
+    (pin "H9XX_CONN" bidirectional (at 172.72 133.35 0)
       (effects (font (size 1.27 1.27)) (justify right))
     )
-    (pin "BUS_XLATED" passive (at 162.56 111.76 180)
+    (pin "BUS_XLATED" passive (at 151.13 130.81 180)
       (effects (font (size 1.27 1.27)) (justify left))
     )

Commit message: wip
Other:
- removed sheet Bus Interface
- added sheet Backplane Pullups (backplane_pullups.kicad_sch)
- sheet Controller ports: added H9XX_CONN; removed none
