File: projects/pdp11_front_panel/backplane_connection.kicad_sch (KiCad schematic)
At the start: 1 part

Commit message: .
Connections:
- net BPOK_H: no longer J?.10 (Pin_10)
- net BEVNT_L renamed BEVENT_L
- no-connect marks 2 -> 5
Other:
- moved on the sheet: J?
Changed lines of the file:
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@@
 (kicad_sch (version 20211123) (generator eeschema)
   (paper "A4")
-  (no_connect (at 88.9 101.6))
-  (no_connect (at 104.14 109.22))
-  (wire (pts (xy 87.63 111.76) (xy 91.44 111.76))
+  (no_connect (at 123.19 106.68))
+  (no_connect (at 138.43 114.3))
+  (no_connect (at 138.43 116.84))
+  (no_connect (at 138.43 119.38))
+  (no_connect (at 125.73 119.38))
+  (bus_entry (at 50.8 86.36) (size 2.54 2.54)
     (stroke (width 0) (type default) (color 0 0 0 0))
   )
-  (wire (pts (xy 66.04 116.84) (xy 91.44 116.84))
+  (bus_entry (at 86.995 86.36) (size 2.54 2.54)
     (stroke (width 0) (type default) (color 0 0 0 0))
   )
-  (wire (pts (xy 107.95 116.84) (xy 104.14 116.84))
+  (bus_entry (at 59.69 85.725) (size 2.54 2.54)
     (stroke (width 0) (type default) (color 0 0 0 0))
   )
-  (wire (pts (xy 104.14 106.68) (xy 107.95 106.68))
+  (bus_entry (at 40.005 86.36) (size 2.54 2.54)
     (stroke (width 0) (type default) (color 0 0 0 0))
   )
-  (wire (pts (xy 107.95 106.68) (xy 107.95 99.06))
+  (bus_entry (at 72.39 86.36) (size 2.54 2.54)
     (stroke (width 0) (type default) (color 0 0 0 0))
   )
-  (wire (pts (xy 87.63 109.22) (xy 91.44 109.22))
+  (wire (pts (xy 52.705 88.9) (xy 53.34 88.9))
     (stroke (width 0) (type default) (color 0 0 0 0))
   )
-  (wire (pts (xy 107.95 120.65) (xy 107.95 116.84))
+  (wire (pts (xy 121.92 116.84) (xy 125.73 116.84))
     (stroke (width 0) (type default) (color 0 0 0 0))
   )
-  (wire (pts (xy 107.95 99.06) (xy 66.04 99.06))
+  (wire (pts (xy 53.34 121.92) (xy 125.73 121.92))
     (stroke (width 0) (type default) (color 0 0 0 0))
   )
-  (wire (pts (xy 87.63 95.25) (xy 87.63 109.22))
+  (wire (pts (xy 142.24 121.92) (xy 138.43 121.92))
     (stroke (width 0) (type default) (color 0 0 0 0))
   )
-  (wire (pts (xy 87.63 111.76) (xy 87.63 123.19))
+  (wire (pts (xy 138.43 111.76) (xy 142.24 111.76))
     (stroke (width 0) (type default) (color 0 0 0 0))
   )
-  (wire (pts (xy 66.04 120.65) (xy 107.95 120.65))
+  (wire (pts (xy 142.24 111.76) (xy 142.24 104.14))
     (stroke (width 0) (type default) (color 0 0 0 0))
   )
-  (wire (pts (xy 135.89 95.25) (xy 87.63 95.25))
+  (wire (pts (xy 74.93 104.14) (xy 142.24 104.14))
     (stroke (width 0) (type default) (color 0 0 0 0))
   )
-  (wire (pts (xy 66.04 106.68) (xy 91.44 106.68))
+  (wire (pts (xy 53.34 121.92) (xy 53.34 88.9))
+    (stroke (width 0) (type default) (color 0 0 0 0))
+  )
+  (bus (pts (xy 28.575 86.36) (xy 40.005 86.36))
+    (stroke (width 0) (type default) (color 0 0 0 0))
+  )
+  (bus (pts (xy 40.005 86.36) (xy 50.8 86.36))
+    (stroke (width 0) (type default) (color 0 0 0 0))
+  )
+  (wire (pts (xy 121.92 114.3) (xy 125.73 114.3))
+    (stroke (width 0) (type default) (color 0 0 0 0))
+  )
+  (wire (pts (xy 89.535 88.9) (xy 89.535 100.33))
+    (stroke (width 0) (type default) (color 0 0 0 0))
+  )
+  (wire (pts (xy 142.24 125.73) (xy 142.24 121.92))
+    (stroke (width 0) (type default) (color 0 0 0 0))
+  )
+  (wire (pts (xy 42.545 125.73) (xy 42.545 88.9))
+    (stroke (width 0) (type default) (color 0 0 0 0))
+  )
+  (wire (pts (xy 62.23 88.265) (xy 62.23 111.76))
+    (stroke (width 0) (type default) (color 0 0 0 0))
+  )
+  (wire (pts (xy 42.545 125.73) (xy 99.695 125.73))
+    (stroke (width 0) (type default) (color 0 0 0 0))
+  )
+  (wire (pts (xy 121.92 100.33) (xy 121.92 114.3))
+    (stroke (width 0) (type default) (color 0 0 0 0))
+  )
+  (wire (pts (xy 89.535 100.33) (xy 121.92 100.33))
+    (stroke (width 0) (type default) (color 0 0 0 0))
+  )
+  (bus (pts (xy 72.39 86.36) (xy 86.995 86.36))
+    (stroke (width 0) (type default) (color 0 0 0 0))
+  )
+  (wire (pts (xy 121.92 116.84) (xy 121.92 128.27))
+    (stroke (width 0) (type default) (color 0 0 0 0))
+  )
+  (wire (pts (xy 41.91 88.9) (xy 42.545 88.9))
+    (stroke (width 0) (type default) (color 0 0 0 0))
+  )
+  (wire (pts (xy 100.33 125.73) (xy 142.24 125.73))
+    (stroke (width 0) (type default) (color 0 0 0 0))
+  )
+  (bus (pts (xy 86.995 86.36) (xy 88.265 86.36))
+    (stroke (width 0) (type default) (color 0 0 0 0))
+  )
+  (bus (pts (xy 50.8 86.36) (xy 72.39 86.36))
+    (stroke (width 0) (type default) (color 0 0 0 0))
+  )
+  (wire (pts (xy 74.93 88.9) (xy 74.93 104.14))
+    (stroke (width 0) (type default) (color 0 0 0 0))
+  )
+  (wire (pts (xy 62.23 111.76) (xy 125.73 111.76))
     (stroke (width 0) (type default) (color 0 0 0 0))
   )
@@
     )
   )
-  (hierarchical_label "BDCOK_H" (shape input) (at 66.04 106.68 180)
-    (effects (font (size 1.27 1.27)) (justify right))
+  (label "SRUN_L" (at 89.535 88.9 0)
+    (effects (font (size 1.27 1.27)) (justify left bottom))
   )
-  (hierarchical_label "SRUN_L" (shape output) (at 135.89 95.25 0)
-    (effects (font (size 1.27 1.27)) (justify left))
+  (label "{SRUN_L,BEVENT_L,BDCOK_H,BPOK_H,BHALT_L}" (at 29.21 86.36 0)
+    (effects (font (size 1.27 1.27)) (justify left bottom))
   )
-  (hierarchical_label "BHALT_L" (shape input) (at 66.04 116.84 180)
-    (effects (font (size 1.27 1.27)) (justify right))
+  (label "BDCOK_H" (at 62.23 88.9 0)
+    (effects (font (size 1.27 1.27)) (justify left bottom))
   )
-  (hierarchical_label "BPOK_H" (shape input) (at 66.04 120.65 180)
-    (effects (font (size 1.27 1.27)) (justify right))
+  (label "BHALT_L" (at 52.705 88.9 0)
+    (effects (font (size 1.27 1.27)) (justify left bottom))
+  )
+  (label "BEVENT_L" (at 74.93 88.9 0)
+    (effects (font (size 1.27 1.27)) (justify left bottom))
+  )
+  (label "BPOK_H" (at 41.91 88.9 0)
+    (effects (font (size 1.27 1.27)) (justify left bottom))
   )
-  (hierarchical_label "BEVNT_L" (shape input) (at 66.04 99.06 180)
+  (hierarchical_label "H9XX_CONN" (shape bidirectional) (at 28.575 86.36 180)
     (effects (font (size 1.27 1.27)) (justify right))
   )
-  (symbol (lib_id "power:GND") (at 87.63 123.19 0) (unit 1)
+  (symbol (lib_id "power:GND") (at 121.92 128.27 0) (unit 1)
     (in_bom yes) (on_board yes) (fields_autoplaced)
-    (property "Reference" "#PWR?" (id 0) (at 87.63 129.54 0)
+    (property "Reference" "#PWR?" (id 0) (at 121.92 134.62 0)
       (effects (font (size 1.27 1.27)) hide)
     )
-    (property "Value" "GND" (id 1) (at 87.63 128.27 0))
-    (property "Footprint" "" (id 2) (at 87.63 123.19 0)
+    (property "Value" "GND" (id 1) (at 121.92 133.35 0))
+    (property "Footprint" "" (id 2) (at 121.92 128.27 0)
       (effects (font (size 1.27 1.27)) hide)
     )
-    (property "Datasheet" "" (id 3) (at 87.63 123.19 0)
+    (property "Datasheet" "" (id 3) (at 121.92 128.27 0)
       (effects (font (size 1.27 1.27)) hide)
     )
     (pin "1")
   )
-  (symbol (lib_id "Connector_Generic:Conn_02x05_Odd_Even") (at 96.52 111.76 0) (unit 1)
+  (symbol (lib_id "Connector_Generic:Conn_02x05_Odd_Even") (at 130.81 116.84 0) (unit 1)
     (in_bom yes) (on_board yes) (fields_autoplaced)
-    (property "Reference" "J?" (id 0) (at 97.79 100.33 0))
-    (property "Value" "Conn_02x05_Odd_Even" (id 1) (at 97.79 102.87 0))
-    (property "Footprint" "" (id 2) (at 96.52 111.76 0)
+    (property "Reference" "J?" (id 0) (at 132.08 105.41 0))
+    (property "Value" "Conn_02x05_Odd_Even" (id 1) (at 132.08 107.95 0))
+    (property "Footprint" "" (id 2) (at 130.81 116.84 0)
       (effects (font (size 1.27 1.27)) hide)
     )
-    (property "Datasheet" "~" (id 3) (at 96.52 111.76 0)
+    (property "Datasheet" "~" (id 3) (at 130.81 116.84 0)
       (effects (font (size 1.27 1.27)) hide)
     )

Commit message: .
Parts:
- gave numbers to parts that had none: 1
Connections:
- net BEVENT_L renamed BEVNT_L
- no-connect marks 5 -> 4
Changed lines of the file:
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@@
-(kicad_sch (version 20211123) (generator eeschema)
+(kicad_sch (version 20230121) (generator eeschema)
   (paper "A4")
-  (no_connect (at 123.19 106.68))
+  (junction (at 53.975 121.92) (diameter 0) (color 0 0 0 0)
+  )
   (no_connect (at 138.43 114.3))
   (no_connect (at 138.43 116.84))
   (no_connect (at 138.43 119.38))
   (no_connect (at 125.73 119.38))
-  (bus_entry (at 50.8 86.36) (size 2.54 2.54)
-    (stroke (width 0) (type default) (color 0 0 0 0))
-  )
-  (bus_entry (at 86.995 86.36) (size 2.54 2.54)
-    (stroke (width 0) (type default) (color 0 0 0 0))
+  (bus_entry (at 84.455 86.36) (size 2.54 2.54)
+    (stroke (width 0) (type default))
   )
-  (bus_entry (at 59.69 85.725) (size 2.54 2.54)
-    (stroke (width 0) (type default) (color 0 0 0 0))
+  (bus_entry (at 75.565 86.36) (size 2.54 2.54)
+    (stroke (width 0) (type default))
   )
-  (bus_entry (at 40.005 86.36) (size 2.54 2.54)
-    (stroke (width 0) (type default) (color 0 0 0 0))
+  (bus_entry (at 51.435 86.36) (size 2.54 2.54)
+    (stroke (width 0) (type default))
   )
-  (bus_entry (at 72.39 86.36) (size 2.54 2.54)
-    (stroke (width 0) (type default) (color 0 0 0 0))
+  (bus_entry (at 41.275 86.36) (size 2.54 2.54)
+    (stroke (width 0) (type default))
   )
-  (wire (pts (xy 52.705 88.9) (xy 53.34 88.9))
-    (stroke (width 0) (type default) (color 0 0 0 0))
+  (bus_entry (at 62.23 86.36) (size 2.54 2.54)
+    (stroke (width 0) (type default))
   )
   (wire (pts (xy 121.92 116.84) (xy 125.73 116.84))
-    (stroke (width 0) (type default) (color 0 0 0 0))
+    (stroke (width 0) (type default))
   )
-  (wire (pts (xy 53.34 121.92) (xy 125.73 121.92))
-    (stroke (width 0) (type default) (color 0 0 0 0))
+  (wire (pts (xy 53.975 88.9) (xy 53.975 121.92))
+    (stroke (width 0) (type default))
   )
   (wire (pts (xy 142.24 121.92) (xy 138.43 121.92))
-    (stroke (width 0) (type default) (color 0 0 0 0))
+    (stroke (width 0) (type default))
   )
   (wire (pts (xy 138.43 111.76) (xy 142.24 111.76))
-    (stroke (width 0) (type default) (color 0 0 0 0))
+    (stroke (width 0) (type default))
   )
   (wire (pts (xy 142.24 111.76) (xy 142.24 104.14))
-    (stroke (width 0) (type default) (color 0 0 0 0))
+    (stroke (width 0) (type default))
   )
-  (wire (pts (xy 74.93 104.14) (xy 142.24 104.14))
-    (stroke (width 0) (type default) (color 0 0 0 0))
+  (bus (pts (xy 27.94 86.36) (xy 41.275 86.36))
+    (stroke (width 0) (type default))
   )
-  (wire (pts (xy 53.34 121.92) (xy 53.34 88.9))
-    (stroke (width 0) (type default) (color 0 0 0 0))
+  (wire (pts (xy 53.975 121.92) (xy 125.73 121.92))
+    (stroke (width 0) (type default))
   )
-  (bus (pts (xy 28.575 86.36) (xy 40.005 86.36))
-    (stroke (width 0) (type default) (color 0 0 0 0))
+  (wire (pts (xy 78.105 104.14) (xy 142.24 104.14))
+    (stroke (width 0) (type default))
   )
-  (bus (pts (xy 40.005 86.36) (xy 50.8 86.36))
-    (stroke (width 0) (type default) (color 0 0 0 0))
+  (wire (pts (xy 78.105 88.9) (xy 78.105 104.14))
+    (stroke (width 0) (type default))
   )
   (wire (pts (xy 121.92 114.3) (xy 125.73 114.3))
-    (stroke (width 0) (type default) (color 0 0 0 0))
+    (stroke (width 0) (type default))
   )
-  (wire (pts (xy 89.535 88.9) (xy 89.535 100.33))
-    (stroke (width 0) (type default) (color 0 0 0 0))
+  (wire (pts (xy 86.995 88.9) (xy 86.995 100.33))
+    (stroke (width 0) (type default))
   )
   (wire (pts (xy 142.24 125.73) (xy 142.24 121.92))
-    (stroke (width 0) (type default) (color 0 0 0 0))
+    (stroke (width 0) (type default))
   )
-  (wire (pts (xy 42.545 125.73) (xy 42.545 88.9))
-    (stroke (width 0) (type default) (color 0 0 0 0))
+  (wire (pts (xy 64.77 88.9) (xy 64.77 111.76))
+    (stroke (width 0) (type default))
   )
-  (wire (pts (xy 62.23 88.265) (xy 62.23 111.76))
-    (stroke (width 0) (type default) (color 0 0 0 0))
+  (wire (pts (xy 43.815 125.73) (xy 99.695 125.73))
+    (stroke (width 0) (type default))
   )
-  (wire (pts (xy 42.545 125.73) (xy 99.695 125.73))
-    (stroke (width 0) (type default) (color 0 0 0 0))
+  (bus (pts (xy 75.565 86.36) (xy 84.455 86.36))
+    (stroke (width 0) (type default))
   )
   (wire (pts (xy 121.92 100.33) (xy 121.92 114.3))
-    (stroke (width 0) (type default) (color 0 0 0 0))
+    (stroke (width 0) (type default))
   )
-  (wire (pts (xy 89.535 100.33) (xy 121.92 100.33))
-    (stroke (width 0) (type default) (color 0 0 0 0))
+  (wire (pts (xy 86.995 100.33) (xy 121.92 100.33))
+    (stroke (width 0) (type default))
   )
-  (bus (pts (xy 72.39 86.36) (xy 86.995 86.36))
-    (stroke (width 0) (type default) (color 0 0 0 0))
+  (bus (pts (xy 51.435 86.36) (xy 62.23 86.36))
+    (stroke (width 0) (type default))
   )
-  (wire (pts (xy 121.92 116.84) (xy 121.92 128.27))
-    (stroke (width 0) (type default) (color 0 0 0 0))
-  )
-  (wire (pts (xy 41.91 88.9) (xy 42.545 88.9))
-    (stroke (width 0) (type default) (color 0 0 0 0))
+  (wire (pts (xy 121.92 116.84) (xy 121.92 132.08))
+    (stroke (width 0) (type default))
   )
   (wire (pts (xy 100.33 125.73) (xy 142.24 125.73))
-    (stroke (width 0) (type default) (color 0 0 0 0))
+    (stroke (width 0) (type default))
+  )
+  (bus (pts (xy 62.23 86.36) (xy 75.565 86.36))
+    (stroke (width 0) (type default))
   )
-  (bus (pts (xy 86.995 86.36) (xy 88.265 86.36))
-    (stroke (width 0) (type default) (color 0 0 0 0))
+  (wire (pts (xy 53.975 123.19) (xy 53.975 121.92))
+    (stroke (width 0) (type default))
   )
-  (bus (pts (xy 50.8 86.36) (xy 72.39 86.36))
-    (stroke (width 0) (type default) (color 0 0 0 0))
+  (bus (pts (xy 41.275 86.36) (xy 51.435 86.36))
+    (stroke (width 0) (type default))
   )
-  (wire (pts (xy 74.93 88.9) (xy 74.93 104.14))
-    (stroke (width 0) (type default) (color 0 0 0 0))
+  (wire (pts (xy 43.815 88.9) (xy 43.815 125.73))
+    (stroke (width 0) (type default))
   )
-  (wire (pts (xy 62.23 111.76) (xy 125.73 111.76))
-    (stroke (width 0) (type default) (color 0 0 0 0))
+  (wire (pts (xy 64.77 111.76) (xy 125.73 111.76))
+    (stroke (width 0) (type default))
   )
   (image (at 71.12 45.72) (scale 0.848095)
@@
     )
   )
-  (label "SRUN_L" (at 89.535 88.9 0)
+  (label "BEVNT_L" (at 78.105 90.17 0)
     (effects (font (size 1.27 1.27)) (justify left bottom))
   )
-  (label "{SRUN_L,BEVENT_L,BDCOK_H,BPOK_H,BHALT_L}" (at 29.21 86.36 0)
+  (label "BDCOK_H" (at 64.77 90.17 0)
     (effects (font (size 1.27 1.27)) (justify left bottom))
   )
-  (label "BDCOK_H" (at 62.23 88.9 0)
+  (label "BHALT_L" (at 53.975 90.17 0)
     (effects (font (size 1.27 1.27)) (justify left bottom))
   )
-  (label "BHALT_L" (at 52.705 88.9 0)
+  (label "{SRUN_L,BEVNT_L,BDCOK_H,BPOK_H,BHALT_L}" (at 29.21 86.36 0) (fields_autoplaced)
     (effects (font (size 1.27 1.27)) (justify left bottom))
   )
-  (label "BEVENT_L" (at 74.93 88.9 0)
+  (label "BPOK_H" (at 43.815 90.17 0)
     (effects (font (size 1.27 1.27)) (justify left bottom))
   )
-  (label "BPOK_H" (at 41.91 88.9 0)
+  (label "SRUN_L" (at 86.995 90.17 0)
     (effects (font (size 1.27 1.27)) (justify left bottom))
   )
-  (hierarchical_label "H9XX_CONN" (shape bidirectional) (at 28.575 86.36 180)
+  (hierarchical_label "GND" (shape passive) (at 121.92 132.08 270) (fields_autoplaced)
     (effects (font (size 1.27 1.27)) (justify right))
   )
-  (symbol (lib_id "power:GND") (at 121.92 128.27 0) (unit 1)
-    (in_bom yes) (on_board yes) (fields_autoplaced)
-    (property "Reference" "#PWR?" (id 0) (at 121.92 134.62 0)
-      (effects (font (size 1.27 1.27)) hide)
-    )
-    (property "Value" "GND" (id 1) (at 121.92 133.35 0))
-    (property "Footprint" "" (id 2) (at 121.92 128.27 0)
-      (effects (font (size 1.27 1.27)) hide)
-    )
-    (property "Datasheet" "" (id 3) (at 121.92 128.27 0)
-      (effects (font (size 1.27 1.27)) hide)
-    )
-    (pin "1")
+  (hierarchical_label "H9XX_CONN" (shape bidirectional) (at 27.94 86.36 180) (fields_autoplaced)
+    (effects (font (size 1.27 1.27)) (justify right))
   )
   (symbol (lib_id "Connector_Generic:Conn_02x05_Odd_Even") (at 130.81 116.84 0) (unit 1)
-    (in_bom yes) (on_board yes) (fields_autoplaced)
-    (property "Reference" "J?" (id 0) (at 132.08 105.41 0))
-    (property "Value" "Conn_02x05_Odd_Even" (id 1) (at 132.08 107.95 0))
-    (property "Footprint" "" (id 2) (at 130.81 116.84 0)
+    (in_bom yes) (on_board yes) (dnp no) (fields_autoplaced)
+    (property "Reference" "J3" (at 132.08 105.41 0)
+      (effects (font (size 1.27 1.27)))
+    )
+    (property "Value" "Conn_02x05_Odd_Even" (at 132.08 107.95 0)
+      (effects (font (size 1.27 1.27)))
+    )
+    (property "Footprint" "" (at 130.81 116.84 0)
       (effects (font (size 1.27 1.27)) hide)
     )
-    (property "Datasheet" "~" (id 3) (at 130.81 116.84 0)
+    (property "Datasheet" "~" (at 130.81 116.84 0)
       (effects (font (size 1.27 1.27)) hide)
     )
@@
     (pin "8")
     (pin "9")
+    (instances
+      (project "pdp11_front_panel"
+        (path "/e63e39d7-6ac0-4ffd-8aa3-1841a4541b55/a264bf2f-3de9-43eb-af67-5739949c50d9"
+          (reference "J3") (unit 1)
+        )
+      )
+    )
   )
 )

Commit message: wip
Connections:
- net BDCOK_H: now also J3.10 (Pin_10); no longer J3.1 (Pin_1)
- net BPOK_H: now also J3.1 (Pin_1)
Other:
- note added: "1"
- note added: "10"
- note added: "2"
- note added: "3"
- note added: "4"
- note added: "5"
- note added: "6"
- note added: "7"
- note added: "8"
- note added: "9"
