File: projects/pdp11_front_panel/backplane_connection.kicad_sch (KiCad schematic)
At the start: 1 part, among them J3 Conn_02x05_Odd_Even

Commit message: wip
Other:
- moved on the sheet: J3
Changed lines of the file:
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@@
 (kicad_sch (version 20230121) (generator eeschema)
   (paper "A4")
-  (no_connect (at 138.43 114.3))
-  (no_connect (at 138.43 116.84))
-  (no_connect (at 138.43 119.38))
-  (no_connect (at 125.73 119.38))
-  (bus_entry (at 85.09 86.36) (size 2.54 2.54)
+  (no_connect (at 152.4 113.03))
+  (no_connect (at 152.4 115.57))
+  (no_connect (at 152.4 118.11))
+  (no_connect (at 139.7 118.11))
+  (bus_entry (at 119.38 86.36) (size 2.54 2.54)
     (stroke (width 0) (type default))
   )
-  (bus_entry (at 76.2 86.36) (size 2.54 2.54)
+  (bus_entry (at 109.22 86.36) (size 2.54 2.54)
     (stroke (width 0) (type default))
   )
-  (bus_entry (at 52.07 86.36) (size 2.54 2.54)
+  (bus_entry (at 86.36 86.36) (size 2.54 2.54)
     (stroke (width 0) (type default))
   )
-  (bus_entry (at 41.91 86.36) (size 2.54 2.54)
+  (bus_entry (at 76.2 86.36) (size 2.54 2.54)
     (stroke (width 0) (type default))
   )
-  (bus_entry (at 62.23 86.36) (size 2.54 2.54)
+  (bus_entry (at 96.52 86.36) (size 2.54 2.54)
     (stroke (width 0) (type default))
   )
-  (wire (pts (xy 121.92 116.84) (xy 125.73 116.84))
+  (wire (pts (xy 135.89 115.57) (xy 139.7 115.57))
     (stroke (width 0) (type default))
   )
-  (wire (pts (xy 54.61 88.9) (xy 54.61 121.92))
+  (wire (pts (xy 88.9 88.9) (xy 88.9 120.65))
     (stroke (width 0) (type default))
   )
-  (wire (pts (xy 147.32 121.92) (xy 138.43 121.92))
+  (wire (pts (xy 161.29 120.65) (xy 152.4 120.65))
     (stroke (width 0) (type default))
   )
-  (bus (pts (xy 27.94 86.36) (xy 41.91 86.36))
+  (bus (pts (xy 27.94 86.36) (xy 76.2 86.36))
     (stroke (width 0) (type default))
   )
@@
     (stroke (width 0) (type default))
   )
-  (wire (pts (xy 54.61 121.92) (xy 125.73 121.92))
+  (wire (pts (xy 88.9 120.65) (xy 139.7 120.65))
     (stroke (width 0) (type default))
   )
-  (wire (pts (xy 78.74 88.9) (xy 78.74 100.33))
+  (wire (pts (xy 111.76 88.9) (xy 111.76 99.06))
     (stroke (width 0) (type default))
   )
-  (wire (pts (xy 147.32 100.33) (xy 78.74 100.33))
+  (wire (pts (xy 161.29 99.06) (xy 111.76 99.06))
     (stroke (width 0) (type default))
   )
-  (wire (pts (xy 87.63 88.9) (xy 87.63 114.3))
+  (wire (pts (xy 78.74 88.9) (xy 78.74 110.49))
     (stroke (width 0) (type default))
   )
-  (wire (pts (xy 121.92 116.84) (xy 121.92 129.54))
+  (wire (pts (xy 121.92 88.9) (xy 121.92 113.03))
     (stroke (width 0) (type default))
   )
-  (wire (pts (xy 147.32 125.73) (xy 147.32 121.92))
+  (wire (pts (xy 135.89 115.57) (xy 135.89 128.27))
     (stroke (width 0) (type default))
   )
-  (wire (pts (xy 64.77 88.9) (xy 64.77 125.73))
+  (wire (pts (xy 161.29 124.46) (xy 161.29 120.65))
     (stroke (width 0) (type default))
   )
-  (wire (pts (xy 125.73 111.76) (xy 44.45 111.76))
+  (wire (pts (xy 99.06 88.9) (xy 99.06 124.46))
     (stroke (width 0) (type default))
   )
-  (bus (pts (xy 76.2 86.36) (xy 85.09 86.36))
+  (wire (pts (xy 139.7 110.49) (xy 78.74 110.49))
     (stroke (width 0) (type default))
   )
-  (bus (pts (xy 52.07 86.36) (xy 62.23 86.36))
+  (bus (pts (xy 109.22 86.36) (xy 119.38 86.36))
     (stroke (width 0) (type default))
   )
-  (wire (pts (xy 147.32 111.76) (xy 147.32 100.33))
+  (bus (pts (xy 86.36 86.36) (xy 96.52 86.36))
     (stroke (width 0) (type default))
   )
-  (wire (pts (xy 64.77 125.73) (xy 147.32 125.73))
+  (wire (pts (xy 161.29 110.49) (xy 161.29 99.06))
     (stroke (width 0) (type default))
   )
-  (bus (pts (xy 62.23 86.36) (xy 76.2 86.36))
+  (wire (pts (xy 99.06 124.46) (xy 161.29 124.46))
     (stroke (width 0) (type default))
   )
-  (bus (pts (xy 41.91 86.36) (xy 52.07 86.36))
+  (bus (pts (xy 96.52 86.36) (xy 109.22 86.36))
     (stroke (width 0) (type default))
   )
-  (wire (pts (xy 34.29 138.43) (xy 34.29 132.08))
+  (bus (pts (xy 76.2 86.36) (xy 86.36 86.36))
     (stroke (width 0) (type default))
   )
-  (wire (pts (xy 138.43 111.76) (xy 147.32 111.76))
+  (wire (pts (xy 34.29 138.43) (xy 34.29 132.08))
     (stroke (width 0) (type default))
   )
-  (wire (pts (xy 87.63 114.3) (xy 125.73 114.3))
+  (wire (pts (xy 152.4 110.49) (xy 161.29 110.49))
     (stroke (width 0) (type default))
   )
-  (wire (pts (xy 44.45 111.76) (xy 44.45 88.9))
+  (wire (pts (xy 121.92 113.03) (xy 139.7 113.03))
     (stroke (width 0) (type default))
   )
@@
     (effects (font (size 1.27 1.27)) (justify left bottom))
   )
-  (label "BEVNT_L" (at 78.74 90.17 0) (fields_autoplaced)
+  (label "BEVNT_L" (at 111.76 88.9 0) (fields_autoplaced)
     (effects (font (size 1.27 1.27)) (justify left bottom))
   )
-  (label "BDCOK_H" (at 64.77 90.17 0) (fields_autoplaced)
+  (label "BDCOK_H" (at 99.06 88.9 0) (fields_autoplaced)
     (effects (font (size 1.27 1.27)) (justify left bottom))
   )
-  (label "BHALT_L" (at 54.61 90.17 0) (fields_autoplaced)
+  (label "BHALT_L" (at 88.9 88.9 0) (fields_autoplaced)
     (effects (font (size 1.27 1.27)) (justify left bottom))
   )
@@
     (effects (font (size 1.27 1.27)) (justify left bottom))
   )
-  (label "BPOK_H" (at 44.45 90.17 0) (fields_autoplaced)
+  (label "BPOK_H" (at 78.74 88.9 0) (fields_autoplaced)
     (effects (font (size 1.27 1.27)) (justify left bottom))
   )
-  (label "SRUN_L" (at 87.63 90.17 0) (fields_autoplaced)
+  (label "SRUN_L" (at 121.92 88.9 0) (fields_autoplaced)
     (effects (font (size 1.27 1.27)) (justify left bottom))
   )
@@
           (reference "#PWR032") (unit 1)
         )
+        (path "/e63e39d7-6ac0-4ffd-8aa3-1841a4541b55/1c6a9b45-e815-4074-9c99-ea8fbb825eb2"
+          (reference "#PWR044") (unit 1)
+        )
       )
     )
   )
-  (symbol (lib_id "power:GND") (at 121.92 129.54 0) (unit 1)
+  (symbol (lib_id "power:GND") (at 135.89 128.27 0) (unit 1)
     (in_bom yes) (on_board yes) (dnp no) (fields_autoplaced)
-    (property "Reference" "#PWR026" (at 121.92 135.89 0)
+    (property "Reference" "#PWR026" (at 135.89 134.62 0)
       (effects (font (size 1.27 1.27)) hide)
     )
-    (property "Value" "GND" (at 121.92 134.62 0)
+    (property "Value" "GND" (at 135.89 133.35 0)
       (effects (font (size 1.27 1.27)))
     )
-    (property "Footprint" "" (at 121.92 129.54 0)
+    (property "Footprint" "" (at 135.89 128.27 0)
       (effects (font (size 1.27 1.27)) hide)
     )
-    (property "Datasheet" "" (at 121.92 129.54 0)
+    (property "Datasheet" "" (at 135.89 128.27 0)
       (effects (font (size 1.27 1.27)) hide)
     )
@@
           (reference "#PWR033") (unit 1)
         )
+        (path "/e63e39d7-6ac0-4ffd-8aa3-1841a4541b55/1c6a9b45-e815-4074-9c99-ea8fbb825eb2"
+          (reference "#PWR045") (unit 1)
+        )
       )
     )
   )
-  (symbol (lib_id "Connector_Generic:Conn_02x05_Odd_Even") (at 130.81 116.84 0) (unit 1)
+  (symbol (lib_id "Connector_Generic:Conn_02x05_Odd_Even") (at 144.78 115.57 0) (unit 1)
     (in_bom yes) (on_board yes) (dnp no) (fields_autoplaced)
-    (property "Reference" "J3" (at 132.08 105.41 0)
+    (property "Reference" "J3" (at 146.05 104.14 0)
       (effects (font (size 1.27 1.27)))
     )
-    (property "Value" "Conn_02x05_Odd_Even" (at 132.08 107.95 0)
+    (property "Value" "Conn_02x05_Odd_Even" (at 146.05 106.68 0)
       (effects (font (size 1.27 1.27)))
     )
-    (property "Footprint" "" (at 130.81 116.84 0)
+    (property "Footprint" "" (at 144.78 115.57 0)
       (effects (font (size 1.27 1.27)) hide)
     )
-    (property "Datasheet" "~" (at 130.81 116.84 0)
+    (property "Datasheet" "~" (at 144.78 115.57 0)
       (effects (font (size 1.27 1.27)) hide)
     )
@@
           (reference "J3") (unit 1)
         )
+        (path "/e63e39d7-6ac0-4ffd-8aa3-1841a4541b55/1c6a9b45-e815-4074-9c99-ea8fbb825eb2"
+          (reference "J6") (unit 1)
+        )
       )

Commit message: wip
Parts:
- renumbered J3 to J2
Changed lines of the file:
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@@
     (effects (font (size 1.27 1.27)) (justify left bottom))
   )
-  (label "{SRUN_L,BEVNT_L,BDCOK_H,BPOK_H,BHALT_L}" (at 29.21 86.36 0) (fields_autoplaced)
+  (label "{H9XX}" (at 34.29 86.36 0) (fields_autoplaced)
     (effects (font (size 1.27 1.27)) (justify left bottom))
   )
@@
     (effects (font (size 1.27 1.27)) (justify left bottom))
   )
-  (hierarchical_label "H9XX_CONN" (shape bidirectional) (at 27.94 86.36 180) (fields_autoplaced)
+  (hierarchical_label "{H9XX}" (shape bidirectional) (at 27.94 86.36 180) (fields_autoplaced)
     (effects (font (size 1.27 1.27)) (justify right))
   )
@@
         )
         (path "/e63e39d7-6ac0-4ffd-8aa3-1841a4541b55/a264bf2f-3de9-43eb-af67-5739949c50d9"
-          (reference "#PWR032") (unit 1)
+          (reference "#PWR018") (unit 1)
         )
         (path "/e63e39d7-6ac0-4ffd-8aa3-1841a4541b55/1c6a9b45-e815-4074-9c99-ea8fbb825eb2"
-          (reference "#PWR044") (unit 1)
+          (reference "#PWR039") (unit 1)
         )
       )
@@
         )
         (path "/e63e39d7-6ac0-4ffd-8aa3-1841a4541b55/a264bf2f-3de9-43eb-af67-5739949c50d9"
-          (reference "#PWR033") (unit 1)
+          (reference "#PWR019") (unit 1)
         )
         (path "/e63e39d7-6ac0-4ffd-8aa3-1841a4541b55/1c6a9b45-e815-4074-9c99-ea8fbb825eb2"
-          (reference "#PWR045") (unit 1)
+          (reference "#PWR040") (unit 1)
         )
       )
@@
   (symbol (lib_id "Connector_Generic:Conn_02x05_Odd_Even") (at 144.78 115.57 0) (unit 1)
     (in_bom yes) (on_board yes) (dnp no) (fields_autoplaced)
-    (property "Reference" "J3" (at 146.05 104.14 0)
+    (property "Reference" "J2" (at 146.05 104.14 0)
       (effects (font (size 1.27 1.27)))
     )
@@
       (project "pdp11_front_panel"
         (path "/e63e39d7-6ac0-4ffd-8aa3-1841a4541b55/a264bf2f-3de9-43eb-af67-5739949c50d9"
-          (reference "J3") (unit 1)
+          (reference "J2") (unit 1)
         )
         (path "/e63e39d7-6ac0-4ffd-8aa3-1841a4541b55/1c6a9b45-e815-4074-9c99-ea8fbb825eb2"
-          (reference "J6") (unit 1)
+          (reference "J5") (unit 1)
         )
       )

Commit message: wip
Parts:
- J2: footprint (none) -> Connector_PinSocket_2.54mm:PinSocket_2x05_P2.54mm_Vertical_SMD
Changed lines of the file:
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@@
         )
         (path "/e63e39d7-6ac0-4ffd-8aa3-1841a4541b55/1c6a9b45-e815-4074-9c99-ea8fbb825eb2"
-          (reference "#PWR039") (unit 1)
+          (reference "#PWR041") (unit 1)
         )
       )
@@
         )
         (path "/e63e39d7-6ac0-4ffd-8aa3-1841a4541b55/1c6a9b45-e815-4074-9c99-ea8fbb825eb2"
-          (reference "#PWR040") (unit 1)
+          (reference "#PWR042") (unit 1)
         )
       )
@@
       (effects (font (size 1.27 1.27)))
     )
-    (property "Footprint" "" (at 144.78 115.57 0)
+    (property "Footprint" "Connector_PinSocket_2.54mm:PinSocket_2x05_P2.54mm_Vertical_SMD" (at 144.78 115.57 0)
       (effects (font (size 1.27 1.27)) hide)
     )
@@
         )
         (path "/e63e39d7-6ac0-4ffd-8aa3-1841a4541b55/1c6a9b45-e815-4074-9c99-ea8fbb825eb2"
-          (reference "J5") (unit 1)
+          (reference "J6") (unit 1)
         )
       )

Commit message: wip
Parts:
- J2: footprint Connector_PinSocket_2.54mm:PinSocket_2x05_P2.54mm_Vertical_SMD -> Connector_PinHeader_2.54mm:PinHeader_2x05_P2.54mm_Vertical_SMD
Changed lines of the file:
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@@
       (effects (font (size 1.27 1.27)))
     )
-    (property "Footprint" "Connector_PinSocket_2.54mm:PinSocket_2x05_P2.54mm_Vertical_SMD" (at 144.78 115.57 0)
+    (property "Footprint" "Connector_PinHeader_2.54mm:PinHeader_2x05_P2.54mm_Vertical_SMD" (at 144.78 115.57 0)
       (effects (font (size 1.27 1.27)) hide)
     )
