File: projects/pdp11_front_panel/atx_power.kicad_sch (KiCad schematic)
At the start: 1 part

Commit message: .
Parts:
- gave numbers to parts that had none: 1
Connections:
- net +3V3: now reaches J2.1 (+3.3V), J2.12 (+3.3V), J2.13 (+3.3V), J2.2 (+3.3V)
- net VCC renamed +5VSB
- no-connect marks 1 -> 0
Changed lines of the file:
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@@
-(kicad_sch (version 20211123) (generator eeschema)
+(kicad_sch (version 20230121) (generator eeschema)
   (paper "A4")
-  (no_connect (at 154.94 80.01))
-  (wire (pts (xy 154.94 77.47) (xy 170.18 77.47))
-    (stroke (width 0) (type default) (color 0 0 0 0))
-  )
-  (wire (pts (xy 165.1 74.93) (xy 165.1 63.5))
-    (stroke (width 0) (type default) (color 0 0 0 0))
-  )
-  (wire (pts (xy 160.02 72.39) (xy 154.94 72.39))
-    (stroke (width 0) (type default) (color 0 0 0 0))
+  (wire (pts (xy 154.94 77.47) (xy 165.1 77.47))
+    (stroke (width 0) (type default))
   )
   (wire (pts (xy 154.94 74.93) (xy 165.1 74.93))
-    (stroke (width 0) (type default) (color 0 0 0 0))
+    (stroke (width 0) (type default))
   )
-  (wire (pts (xy 154.94 67.31) (xy 220.98 67.31))
-    (stroke (width 0) (type default) (color 0 0 0 0))
+  (wire (pts (xy 154.94 80.01) (xy 165.1 80.01))
+    (stroke (width 0) (type default))
+  )
+  (wire (pts (xy 154.94 67.31) (xy 165.1 67.31))
+    (stroke (width 0) (type default))
   )
   (wire (pts (xy 115.57 67.31) (xy 129.54 67.31))
-    (stroke (width 0) (type default) (color 0 0 0 0))
+    (stroke (width 0) (type default))
   )
-  (wire (pts (xy 175.26 63.5) (xy 175.26 87.63))
-    (stroke (width 0) (type default) (color 0 0 0 0))
+  (wire (pts (xy 142.24 92.71) (xy 142.24 97.79))
+    (stroke (width 0) (type default))
   )
-  (wire (pts (xy 154.94 87.63) (xy 175.26 87.63))
-    (stroke (width 0) (type default) (color 0 0 0 0))
+  (wire (pts (xy 154.94 87.63) (xy 165.1 87.63))
+    (stroke (width 0) (type default))
   )
-  (wire (pts (xy 170.18 77.47) (xy 170.18 63.5))
-    (stroke (width 0) (type default) (color 0 0 0 0))
+  (wire (pts (xy 154.94 72.39) (xy 165.1 72.39))
+    (stroke (width 0) (type default))
   )
-  (wire (pts (xy 142.24 92.71) (xy 142.24 93.98))
-    (stroke (width 0) (type default) (color 0 0 0 0))
-  )
-  (wire (pts (xy 160.02 63.5) (xy 160.02 72.39))
-    (stroke (width 0) (type default) (color 0 0 0 0))
-  )
-  (hierarchical_label "ATX_PS_ON#" (shape input) (at 115.57 67.31 180)
+  (hierarchical_label "GND" (shape passive) (at 142.24 97.79 270) (fields_autoplaced)
     (effects (font (size 1.27 1.27)) (justify right))
   )
-  (hierarchical_label "ATX_PWR_OK" (shape output) (at 220.98 67.31 0)
+  (hierarchical_label "+5VSB" (shape output) (at 165.1 77.47 0) (fields_autoplaced)
+    (effects (font (size 1.27 1.27)) (justify left))
+  )
+  (hierarchical_label "+12V" (shape output) (at 165.1 72.39 0) (fields_autoplaced)
+    (effects (font (size 1.27 1.27)) (justify left))
+  )
+  (hierarchical_label "ATX_PS_ON#" (shape input) (at 115.57 67.31 180) (fields_autoplaced)
+    (effects (font (size 1.27 1.27)) (justify right))
+  )
+  (hierarchical_label "+5V" (shape output) (at 165.1 74.93 0) (fields_autoplaced)
+    (effects (font (size 1.27 1.27)) (justify left))
+  )
+  (hierarchical_label "ATX_PWR_OK" (shape output) (at 165.1 67.31 0) (fields_autoplaced)
+    (effects (font (size 1.27 1.27)) (justify left))
+  )
+  (hierarchical_label "-12V" (shape output) (at 165.1 87.63 0) (fields_autoplaced)
+    (effects (font (size 1.27 1.27)) (justify left))
+  )
+  (hierarchical_label "+3V3" (shape output) (at 165.1 80.01 0) (fields_autoplaced)
     (effects (font (size 1.27 1.27)) (justify left))
   )
   (symbol (lib_id "Connector:ATX-24") (at 142.24 77.47 0) (unit 1)
-    (in_bom yes) (on_board yes) (fields_autoplaced)
-    (property "Reference" "J?" (id 0) (at 142.24 59.69 0))
-    (property "Value" "ATX-24" (id 1) (at 142.24 62.23 0))
-    (property "Footprint" "" (id 2) (at 142.24 80.01 0)
+    (in_bom yes) (on_board yes) (dnp no) (fields_autoplaced)
+    (property "Reference" "J2" (at 142.24 59.69 0)
+      (effects (font (size 1.27 1.27)))
+    )
+    (property "Value" "ATX-24" (at 142.24 62.23 0)
+      (effects (font (size 1.27 1.27)))
+    )
+    (property "Footprint" "" (at 142.24 80.01 0)
       (effects (font (size 1.27 1.27)) hide)
     )
-    (property "Datasheet" "https://www.intel.com/content/dam/www/public/us/en/documents/guides/power-supply-design-guide-june.pdf#page=33" (id 3) (at 203.2 91.44 0)
+    (property "Datasheet" "https://www.intel.com/content/dam/www/public/us/en/documents/guides/power-supply-design-guide-june.pdf#page=33" (at 203.2 91.44 0)
       (effects (font (size 1.27 1.27)) hide)
     )
@@
     (pin "8")
     (pin "9")
-  )
-  (symbol (lib_id "power:-12V") (at 175.26 63.5 0) (unit 1)
-    (in_bom yes) (on_board yes) (fields_autoplaced)
-    (property "Reference" "#PWR?" (id 0) (at 175.26 60.96 0)
-      (effects (font (size 1.27 1.27)) hide)
+    (instances
+      (project "pdp11_front_panel"
+        (path "/e63e39d7-6ac0-4ffd-8aa3-1841a4541b55/d4d8f7cc-faea-4935-ab3d-bc61af3c0a31"
+          (reference "J2") (unit 1)
+        )
+      )
     )
-    (property "Value" "-12V" (id 1) (at 175.26 58.42 0))
-    (property "Footprint" "" (id 2) (at 175.26 63.5 0)
-      (effects (font (size 1.27 1.27)) hide)
-    )
-    (property "Datasheet" "" (id 3) (at 175.26 63.5 0)
-      (effects (font (size 1.27 1.27)) hide)
-    )
-    (pin "1")
-  )
-  (symbol (lib_id "power:+12V") (at 160.02 63.5 0) (unit 1)
-    (in_bom yes) (on_board yes) (fields_autoplaced)
-    (property "Reference" "#PWR?" (id 0) (at 160.02 67.31 0)
-      (effects (font (size 1.27 1.27)) hide)
-    )
-    (property "Value" "+12V" (id 1) (at 160.02 58.42 0))
-    (property "Footprint" "" (id 2) (at 160.02 63.5 0)
-      (effects (font (size 1.27 1.27)) hide)
-    )
-    (property "Datasheet" "" (id 3) (at 160.02 63.5 0)
-      (effects (font (size 1.27 1.27)) hide)
-    )
-    (pin "1")
-  )
-  (symbol (lib_id "power:+5V") (at 165.1 63.5 0) (unit 1)
-    (in_bom yes) (on_board yes) (fields_autoplaced)
-    (property "Reference" "#PWR?" (id 0) (at 165.1 67.31 0)
-      (effects (font (size 1.27 1.27)) hide)
-    )
-    (property "Value" "+5V" (id 1) (at 165.1 58.42 0))
-    (property "Footprint" "" (id 2) (at 165.1 63.5 0)
-      (effects (font (size 1.27 1.27)) hide)
-    )
-    (property "Datasheet" "" (id 3) (at 165.1 63.5 0)
-      (effects (font (size 1.27 1.27)) hide)
-    )
-    (pin "1")
-  )
-  (symbol (lib_id "power:GND") (at 142.24 93.98 0) (unit 1)
-    (in_bom yes) (on_board yes) (fields_autoplaced)
-    (property "Reference" "#PWR?" (id 0) (at 142.24 100.33 0)
-      (effects (font (size 1.27 1.27)) hide)
-    )
-    (property "Value" "GND" (id 1) (at 142.24 99.06 0))
-    (property "Footprint" "" (id 2) (at 142.24 93.98 0)
-      (effects (font (size 1.27 1.27)) hide)
-    )
-    (property "Datasheet" "" (id 3) (at 142.24 93.98 0)
-      (effects (font (size 1.27 1.27)) hide)
-    )
-    (pin "1")
-  )
-  (symbol (lib_id "power:VCC") (at 170.18 63.5 0) (unit 1)
-    (in_bom yes) (on_board yes) (fields_autoplaced)
-    (property "Reference" "#PWR?" (id 0) (at 170.18 67.31 0)
-      (effects (font (size 1.27 1.27)) hide)
-    )
-    (property "Value" "VCC" (id 1) (at 170.18 58.42 0))
-    (property "Footprint" "" (id 2) (at 170.18 63.5 0)
-      (effects (font (size 1.27 1.27)) hide)
-    )
-    (property "Datasheet" "" (id 3) (at 170.18 63.5 0)
-      (effects (font (size 1.27 1.27)) hide)
-    )
-    (pin "1")
   )
 )

Commit message: wip
Changed lines of the file:
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@@
 (kicad_sch (version 20230121) (generator eeschema)
   (paper "A4")
-  (wire (pts (xy 154.94 77.47) (xy 165.1 77.47))
+  (bus_entry (at 196.85 55.88) (size -2.54 2.54)
     (stroke (width 0) (type default))
   )
-  (wire (pts (xy 154.94 74.93) (xy 165.1 74.93))
+  (bus_entry (at 190.5 55.88) (size -2.54 2.54)
     (stroke (width 0) (type default))
   )
-  (wire (pts (xy 154.94 80.01) (xy 165.1 80.01))
+  (bus_entry (at 209.55 55.88) (size -2.54 2.54)
     (stroke (width 0) (type default))
   )
-  (wire (pts (xy 154.94 67.31) (xy 165.1 67.31))
+  (bus_entry (at 201.93 55.88) (size -2.54 2.54)
+    (stroke (width 0) (type default))
+  )
+  (bus_entry (at 214.63 55.88) (size -2.54 2.54)
+    (stroke (width 0) (type default))
+  )
+  (bus_entry (at 176.53 55.88) (size -2.54 2.54)
+    (stroke (width 0) (type default))
+  )
+  (wire (pts (xy 154.94 77.47) (xy 199.39 77.47))
+    (stroke (width 0) (type default))
+  )
+  (bus (pts (xy 214.63 55.88) (xy 259.08 55.88))
+    (stroke (width 0) (type default))
+  )
+  (bus (pts (xy 196.85 55.88) (xy 201.93 55.88))
+    (stroke (width 0) (type default))
+  )
+  (wire (pts (xy 154.94 74.93) (xy 194.31 74.93))
+    (stroke (width 0) (type default))
+  )
+  (bus (pts (xy 176.53 55.88) (xy 190.5 55.88))
+    (stroke (width 0) (type default))
+  )
+  (bus (pts (xy 201.93 55.88) (xy 209.55 55.88))
+    (stroke (width 0) (type default))
+  )
+  (wire (pts (xy 154.94 80.01) (xy 207.01 80.01))
+    (stroke (width 0) (type default))
+  )
+  (wire (pts (xy 173.99 58.42) (xy 173.99 67.31))
     (stroke (width 0) (type default))
   )
@@
     (stroke (width 0) (type default))
   )
+  (bus (pts (xy 190.5 55.88) (xy 196.85 55.88))
+    (stroke (width 0) (type default))
+  )
+  (wire (pts (xy 207.01 80.01) (xy 207.01 58.42))
+    (stroke (width 0) (type default))
+  )
+  (wire (pts (xy 173.99 67.31) (xy 154.94 67.31))
+    (stroke (width 0) (type default))
+  )
+  (wire (pts (xy 212.09 58.42) (xy 212.09 87.63))
+    (stroke (width 0) (type default))
+  )
+  (bus (pts (xy 172.72 55.88) (xy 176.53 55.88))
+    (stroke (width 0) (type default))
+  )
+  (bus (pts (xy 209.55 55.88) (xy 214.63 55.88))
+    (stroke (width 0) (type default))
+  )
+  (wire (pts (xy 194.31 58.42) (xy 194.31 74.93))
+    (stroke (width 0) (type default))
+  )
+  (wire (pts (xy 199.39 77.47) (xy 199.39 58.42))
+    (stroke (width 0) (type default))
+  )
   (wire (pts (xy 142.24 92.71) (xy 142.24 97.79))
     (stroke (width 0) (type default))
   )
-  (wire (pts (xy 154.94 87.63) (xy 165.1 87.63))
+  (wire (pts (xy 154.94 87.63) (xy 212.09 87.63))
     (stroke (width 0) (type default))
   )
-  (wire (pts (xy 154.94 72.39) (xy 165.1 72.39))
+  (wire (pts (xy 154.94 72.39) (xy 187.96 72.39))
     (stroke (width 0) (type default))
+  )
+  (wire (pts (xy 187.96 58.42) (xy 187.96 72.39))
+    (stroke (width 0) (type default))
+  )
+  (label "{ATX_PWR_OK,+12V,+5V,+5VSB,+3V3,-12V}" (at 215.9 55.88 0) (fields_autoplaced)
+    (effects (font (size 1.27 1.27)) (justify left bottom))
+  )
+  (label "-12V" (at 212.09 58.42 0)
+    (effects (font (size 1.27 1.27)) (justify left bottom))
+  )
+  (label "+12V" (at 187.96 58.42 0)
+    (effects (font (size 1.27 1.27)) (justify left bottom))
+  )
+  (label "ATX_PWR_OK" (at 173.99 58.42 0)
+    (effects (font (size 1.27 1.27)) (justify left bottom))
+  )
+  (label "+5V" (at 194.31 58.42 0)
+    (effects (font (size 1.27 1.27)) (justify left bottom))
+  )
+  (label "+3V3" (at 207.01 58.42 0)
+    (effects (font (size 1.27 1.27)) (justify left bottom))
+  )
+  (label "+5VSB" (at 199.39 58.42 0)
+    (effects (font (size 1.27 1.27)) (justify left bottom))
+  )
+  (hierarchical_label "ATX_OUT" (shape input) (at 259.08 55.88 0) (fields_autoplaced)
+    (effects (font (size 1.27 1.27)) (justify left))
   )
   (hierarchical_label "GND" (shape passive) (at 142.24 97.79 270) (fields_autoplaced)
     (effects (font (size 1.27 1.27)) (justify right))
   )
-  (hierarchical_label "+5VSB" (shape output) (at 165.1 77.47 0) (fields_autoplaced)
-    (effects (font (size 1.27 1.27)) (justify left))
-  )
-  (hierarchical_label "+12V" (shape output) (at 165.1 72.39 0) (fields_autoplaced)
-    (effects (font (size 1.27 1.27)) (justify left))
-  )
   (hierarchical_label "ATX_PS_ON#" (shape input) (at 115.57 67.31 180) (fields_autoplaced)
     (effects (font (size 1.27 1.27)) (justify right))
   )
-  (hierarchical_label "+5V" (shape output) (at 165.1 74.93 0) (fields_autoplaced)
-    (effects (font (size 1.27 1.27)) (justify left))
-  )
-  (hierarchical_label "ATX_PWR_OK" (shape output) (at 165.1 67.31 0) (fields_autoplaced)
-    (effects (font (size 1.27 1.27)) (justify left))
-  )
-  (hierarchical_label "-12V" (shape output) (at 165.1 87.63 0) (fields_autoplaced)
-    (effects (font (size 1.27 1.27)) (justify left))
-  )
-  (hierarchical_label "+3V3" (shape output) (at 165.1 80.01 0) (fields_autoplaced)
-    (effects (font (size 1.27 1.27)) (justify left))
-  )
   (symbol (lib_id "Connector:ATX-24") (at 142.24 77.47 0) (unit 1)

Commit message: wip
Other:
- moved on the sheet: J2
Changed lines of the file:
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@@
 (kicad_sch (version 20230121) (generator eeschema)
   (paper "A4")
-  (bus_entry (at 196.85 55.88) (size -2.54 2.54)
+  (bus_entry (at 182.88 55.88) (size -2.54 2.54)
     (stroke (width 0) (type default))
   )
-  (bus_entry (at 190.5 55.88) (size -2.54 2.54)
+  (bus_entry (at 176.53 55.88) (size -2.54 2.54)
     (stroke (width 0) (type default))
   )
-  (bus_entry (at 209.55 55.88) (size -2.54 2.54)
+  (bus_entry (at 195.58 55.88) (size -2.54 2.54)
+    (stroke (width 0) (type default))
+  )
+  (bus_entry (at 187.96 55.88) (size -2.54 2.54)
     (stroke (width 0) (type default))
   )
@@
     (stroke (width 0) (type default))
   )
-  (bus_entry (at 214.63 55.88) (size -2.54 2.54)
+  (bus_entry (at 162.56 55.88) (size -2.54 2.54)
     (stroke (width 0) (type default))
   )
-  (bus_entry (at 176.53 55.88) (size -2.54 2.54)
+  (wire (pts (xy 140.97 77.47) (xy 185.42 77.47))
     (stroke (width 0) (type default))
   )
-  (wire (pts (xy 154.94 77.47) (xy 199.39 77.47))
+  (bus (pts (xy 182.88 55.88) (xy 187.96 55.88))
     (stroke (width 0) (type default))
   )
-  (bus (pts (xy 214.63 55.88) (xy 259.08 55.88))
+  (wire (pts (xy 140.97 74.93) (xy 180.34 74.93))
     (stroke (width 0) (type default))
   )
-  (bus (pts (xy 196.85 55.88) (xy 201.93 55.88))
+  (bus (pts (xy 162.56 55.88) (xy 176.53 55.88))
     (stroke (width 0) (type default))
   )
-  (wire (pts (xy 154.94 74.93) (xy 194.31 74.93))
+  (bus (pts (xy 187.96 55.88) (xy 195.58 55.88))
     (stroke (width 0) (type default))
   )
-  (bus (pts (xy 176.53 55.88) (xy 190.5 55.88))
+  (wire (pts (xy 140.97 80.01) (xy 193.04 80.01))
     (stroke (width 0) (type default))
   )
-  (bus (pts (xy 201.93 55.88) (xy 209.55 55.88))
+  (wire (pts (xy 160.02 58.42) (xy 160.02 67.31))
     (stroke (width 0) (type default))
   )
-  (wire (pts (xy 154.94 80.01) (xy 207.01 80.01))
+  (bus (pts (xy 201.93 55.88) (xy 259.08 55.88))
     (stroke (width 0) (type default))
   )
-  (wire (pts (xy 173.99 58.42) (xy 173.99 67.31))
+  (wire (pts (xy 101.6 67.31) (xy 115.57 67.31))
     (stroke (width 0) (type default))
   )
-  (wire (pts (xy 115.57 67.31) (xy 129.54 67.31))
+  (bus (pts (xy 176.53 55.88) (xy 182.88 55.88))
     (stroke (width 0) (type default))
   )
-  (bus (pts (xy 190.5 55.88) (xy 196.85 55.88))
+  (wire (pts (xy 193.04 80.01) (xy 193.04 58.42))
     (stroke (width 0) (type default))
   )
-  (wire (pts (xy 207.01 80.01) (xy 207.01 58.42))
+  (wire (pts (xy 160.02 67.31) (xy 140.97 67.31))
     (stroke (width 0) (type default))
   )
-  (wire (pts (xy 173.99 67.31) (xy 154.94 67.31))
+  (wire (pts (xy 199.39 58.42) (xy 199.39 87.63))
     (stroke (width 0) (type default))
   )
-  (wire (pts (xy 212.09 58.42) (xy 212.09 87.63))
+  (bus (pts (xy 158.75 55.88) (xy 162.56 55.88))
     (stroke (width 0) (type default))
   )
-  (bus (pts (xy 172.72 55.88) (xy 176.53 55.88))
+  (bus (pts (xy 195.58 55.88) (xy 201.93 55.88))
     (stroke (width 0) (type default))
   )
-  (bus (pts (xy 209.55 55.88) (xy 214.63 55.88))
+  (wire (pts (xy 180.34 58.42) (xy 180.34 74.93))
     (stroke (width 0) (type default))
   )
-  (wire (pts (xy 194.31 58.42) (xy 194.31 74.93))
+  (wire (pts (xy 185.42 77.47) (xy 185.42 58.42))
     (stroke (width 0) (type default))
   )
-  (wire (pts (xy 199.39 77.47) (xy 199.39 58.42))
+  (wire (pts (xy 128.27 92.71) (xy 128.27 97.79))
     (stroke (width 0) (type default))
   )
-  (wire (pts (xy 142.24 92.71) (xy 142.24 97.79))
+  (wire (pts (xy 140.97 87.63) (xy 199.39 87.63))
     (stroke (width 0) (type default))
   )
-  (wire (pts (xy 154.94 87.63) (xy 212.09 87.63))
+  (wire (pts (xy 140.97 72.39) (xy 173.99 72.39))
     (stroke (width 0) (type default))
   )
-  (wire (pts (xy 154.94 72.39) (xy 187.96 72.39))
+  (wire (pts (xy 173.99 58.42) (xy 173.99 72.39))
     (stroke (width 0) (type default))
   )
-  (wire (pts (xy 187.96 58.42) (xy 187.96 72.39))
-    (stroke (width 0) (type default))
-  )
-  (label "{ATX_PWR_OK,+12V,+5V,+5VSB,+3V3,-12V}" (at 215.9 55.88 0) (fields_autoplaced)
+  (label "{ATX_PWR_OK,+12V,+5V,+5VSB,+3V3,-12V}" (at 212.09 55.88 0) (fields_autoplaced)
     (effects (font (size 1.27 1.27)) (justify left bottom))
   )
-  (label "-12V" (at 212.09 58.42 0) (fields_autoplaced)
+  (label "-12V" (at 199.39 58.42 0) (fields_autoplaced)
     (effects (font (size 1.27 1.27)) (justify left bottom))
   )
-  (label "+12V" (at 187.96 58.42 0) (fields_autoplaced)
+  (label "+12V" (at 173.99 58.42 0) (fields_autoplaced)
     (effects (font (size 1.27 1.27)) (justify left bottom))
   )
-  (label "ATX_PWR_OK" (at 173.99 58.42 0) (fields_autoplaced)
+  (label "ATX_PWR_OK" (at 160.02 58.42 0) (fields_autoplaced)
     (effects (font (size 1.27 1.27)) (justify left bottom))
   )
-  (label "+5V" (at 194.31 58.42 0) (fields_autoplaced)
+  (label "+5V" (at 180.34 58.42 0) (fields_autoplaced)
     (effects (font (size 1.27 1.27)) (justify left bottom))
   )
-  (label "+3V3" (at 207.01 58.42 0) (fields_autoplaced)
+  (label "+3V3" (at 193.04 58.42 0) (fields_autoplaced)
     (effects (font (size 1.27 1.27)) (justify left bottom))
   )
-  (label "+5VSB" (at 199.39 58.42 0) (fields_autoplaced)
+  (label "+5VSB" (at 185.42 58.42 0) (fields_autoplaced)
     (effects (font (size 1.27 1.27)) (justify left bottom))
   )
@@
     (effects (font (size 1.27 1.27)) (justify left))
   )
-  (hierarchical_label "GND" (shape passive) (at 142.24 97.79 270) (fields_autoplaced)
+  (hierarchical_label "GND" (shape passive) (at 128.27 97.79 270) (fields_autoplaced)
     (effects (font (size 1.27 1.27)) (justify right))
   )
-  (hierarchical_label "ATX_PS_ON#" (shape input) (at 115.57 67.31 180) (fields_autoplaced)
+  (hierarchical_label "ATX_PS_ON#" (shape input) (at 101.6 67.31 180) (fields_autoplaced)
     (effects (font (size 1.27 1.27)) (justify right))
   )
-  (symbol (lib_id "Connector:ATX-24") (at 142.24 77.47 0) (unit 1)
+  (symbol (lib_id "Connector:ATX-24") (at 128.27 77.47 0) (unit 1)
     (in_bom yes) (on_board yes) (dnp no) (fields_autoplaced)
-    (property "Reference" "J2" (at 142.24 59.69 0)
+    (property "Reference" "J2" (at 128.27 59.69 0)
       (effects (font (size 1.27 1.27)))
     )
-    (property "Value" "ATX-24" (at 142.24 62.23 0)
+    (property "Value" "ATX-24" (at 128.27 62.23 0)
       (effects (font (size 1.27 1.27)))
     )
-    (property "Footprint" "" (at 142.24 80.01 0)
+    (property "Footprint" "" (at 128.27 80.01 0)
       (effects (font (size 1.27 1.27)) hide)
     )
-    (property "Datasheet" "https://www.intel.com/content/dam/www/public/us/en/documents/guides/power-supply-design-guide-june.pdf#page=33" (at 203.2 91.44 0)
+    (property "Datasheet" "https://www.intel.com/content/dam/www/public/us/en/documents/guides/power-supply-design-guide-june.pdf#page=33" (at 189.23 91.44 0)
       (effects (font (size 1.27 1.27)) hide)
     )
