File: projects/pdp11_front_panel/backplane_pullups.kicad_sch (KiCad schematic)
At the start: 10 parts

Commit message: wip
Parts:
- renumbered R2 to R16, R3 to R17, R4 to R18, R12 to R19, R13 to R20
Changed lines of the file:
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@@
     (stroke (width 0) (type default))
   )
-  (wire (pts (xy 46.99 179.07) (xy 46.99 181.61))
+  (wire (pts (xy 57.15 111.76) (xy 57.15 114.3))
     (stroke (width 0) (type default))
   )
@@
     (stroke (width 0) (type default))
   )
-  (wire (pts (xy 36.83 177.8) (xy 40.64 177.8))
+  (wire (pts (xy 46.99 110.49) (xy 50.8 110.49))
     (stroke (width 0) (type default))
   )
@@
     (stroke (width 0) (type default))
   )
-  (wire (pts (xy 40.64 177.8) (xy 40.64 170.18))
+  (wire (pts (xy 50.8 110.49) (xy 50.8 102.87))
     (stroke (width 0) (type default))
   )
@@
     (effects (font (size 1.27 1.27)) (justify left bottom))
   )
-  (label "{SRUN_L,BEVNT_L,BDCOK_H,BPOK_H,BHALT_L}" (at 48.26 39.37 0) (fields_autoplaced)
+  (label "{H9XX}" (at 52.07 39.37 0) (fields_autoplaced)
     (effects (font (size 1.27 1.27)) (justify left bottom))
   )
@@
     (effects (font (size 1.27 1.27)) (justify left bottom))
   )
-  (hierarchical_label "H9XX_CONN" (shape bidirectional) (at 46.99 39.37 180) (fields_autoplaced)
+  (hierarchical_label "{H9XX}" (shape bidirectional) (at 46.99 39.37 180) (fields_autoplaced)
     (effects (font (size 1.27 1.27)) (justify right))
   )
-  (hierarchical_label "GND" (shape passive) (at 46.99 179.07 90) (fields_autoplaced)
+  (hierarchical_label "GND" (shape passive) (at 57.15 111.76 90) (fields_autoplaced)
     (effects (font (size 1.27 1.27)) (justify left))
   )
-  (hierarchical_label "+5VA" (shape passive) (at 36.83 177.8 180) (fields_autoplaced)
+  (hierarchical_label "+5VA" (shape passive) (at 46.99 110.49 180) (fields_autoplaced)
     (effects (font (size 1.27 1.27)) (justify right))
   )
   (symbol (lib_id "Device:R") (at 130.81 69.85 0) (unit 1)
     (in_bom yes) (on_board yes) (dnp no) (fields_autoplaced)
-    (property "Reference" "R12" (at 133.35 68.58 0)
+    (property "Reference" "R19" (at 133.35 68.58 0)
       (effects (font (size 1.27 1.27)) (justify left))
     )
@@
       (project "pdp11_front_panel"
         (path "/e63e39d7-6ac0-4ffd-8aa3-1841a4541b55/6921a5ea-b943-4dc1-8acb-8a754944c3ee"
-          (reference "R12") (unit 1)
+          (reference "R19") (unit 1)
         )
       )
@@
         )
         (path "/e63e39d7-6ac0-4ffd-8aa3-1841a4541b55/6921a5ea-b943-4dc1-8acb-8a754944c3ee"
-          (reference "#PWR011") (unit 1)
+          (reference "#PWR038") (unit 1)
         )
       )
@@
     )
   )
-  (symbol (lib_id "power:GND") (at 46.99 181.61 0) (unit 1)
-    (in_bom yes) (on_board yes) (dnp no) (fields_autoplaced)
-    (property "Reference" "#PWR04" (at 46.99 187.96 0)
-      (effects (font (size 1.27 1.27)) hide)
-    )
-    (property "Value" "GND" (at 46.99 186.69 0)
+  (symbol (lib_id "power:GND") (at 57.15 114.3 0) (unit 1)
+    (in_bom yes) (on_board yes) (dnp no) (fields_autoplaced)
+    (property "Reference" "#PWR04" (at 57.15 120.65 0)
+      (effects (font (size 1.27 1.27)) hide)
+    )
+    (property "Value" "GND" (at 57.15 119.38 0)
       (effects (font (size 1.27 1.27)))
     )
-    (property "Footprint" "" (at 46.99 181.61 0)
-      (effects (font (size 1.27 1.27)) hide)
-    )
-    (property "Datasheet" "" (at 46.99 181.61 0)
+    (property "Footprint" "" (at 57.15 114.3 0)
+      (effects (font (size 1.27 1.27)) hide)
+    )
+    (property "Datasheet" "" (at 57.15 114.3 0)
       (effects (font (size 1.27 1.27)) hide)
     )
@@
         )
         (path "/e63e39d7-6ac0-4ffd-8aa3-1841a4541b55/6921a5ea-b943-4dc1-8acb-8a754944c3ee"
-          (reference "#PWR010") (unit 1)
+          (reference "#PWR037") (unit 1)
         )
       )
@@
   (symbol (lib_id "Device:R") (at 97.79 69.85 0) (unit 1)
     (in_bom yes) (on_board yes) (dnp no) (fields_autoplaced)
-    (property "Reference" "R2" (at 100.33 68.58 0)
+    (property "Reference" "R16" (at 100.33 68.58 0)
       (effects (font (size 1.27 1.27)) (justify left))
     )
@@
       (project "pdp11_front_panel"
         (path "/e63e39d7-6ac0-4ffd-8aa3-1841a4541b55/6921a5ea-b943-4dc1-8acb-8a754944c3ee"
-          (reference "R2") (unit 1)
+          (reference "R16") (unit 1)
         )
       )
@@
   (symbol (lib_id "Device:R") (at 140.97 69.85 0) (unit 1)
     (in_bom yes) (on_board yes) (dnp no) (fields_autoplaced)
-    (property "Reference" "R13" (at 143.51 68.58 0)
+    (property "Reference" "R20" (at 143.51 68.58 0)
       (effects (font (size 1.27 1.27)) (justify left))
     )
@@
       (project "pdp11_front_panel"
         (path "/e63e39d7-6ac0-4ffd-8aa3-1841a4541b55/6921a5ea-b943-4dc1-8acb-8a754944c3ee"
-          (reference "R13") (unit 1)
-        )
-      )
-    )
-  )
-  (symbol (lib_id "power:+5VA") (at 40.64 170.18 0) (unit 1)
-    (in_bom yes) (on_board yes) (dnp no) (fields_autoplaced)
-    (property "Reference" "#PWR05" (at 40.64 173.99 0)
-      (effects (font (size 1.27 1.27)) hide)
-    )
-    (property "Value" "+5VA" (at 40.64 165.1 0)
+          (reference "R20") (unit 1)
+        )
+      )
+    )
+  )
+  (symbol (lib_id "power:+5VA") (at 50.8 102.87 0) (unit 1)
+    (in_bom yes) (on_board yes) (dnp no) (fields_autoplaced)
+    (property "Reference" "#PWR05" (at 50.8 106.68 0)
+      (effects (font (size 1.27 1.27)) hide)
+    )
+    (property "Value" "+5VA" (at 50.8 97.79 0)
       (effects (font (size 1.27 1.27)))
     )
-    (property "Footprint" "" (at 40.64 170.18 0)
-      (effects (font (size 1.27 1.27)) hide)
-    )
-    (property "Datasheet" "" (at 40.64 170.18 0)
+    (property "Footprint" "" (at 50.8 102.87 0)
+      (effects (font (size 1.27 1.27)) hide)
+    )
+    (property "Datasheet" "" (at 50.8 102.87 0)
       (effects (font (size 1.27 1.27)) hide)
     )
@@
         )
         (path "/e63e39d7-6ac0-4ffd-8aa3-1841a4541b55/6921a5ea-b943-4dc1-8acb-8a754944c3ee"
-          (reference "#PWR09") (unit 1)
+          (reference "#PWR036") (unit 1)
         )
       )
@@
   (symbol (lib_id "Device:R") (at 107.95 69.85 0) (unit 1)
     (in_bom yes) (on_board yes) (dnp no) (fields_autoplaced)
-    (property "Reference" "R3" (at 110.49 68.58 0)
+    (property "Reference" "R17" (at 110.49 68.58 0)
       (effects (font (size 1.27 1.27)) (justify left))
     )
@@
       (project "pdp11_front_panel"
         (path "/e63e39d7-6ac0-4ffd-8aa3-1841a4541b55/6921a5ea-b943-4dc1-8acb-8a754944c3ee"
-          (reference "R3") (unit 1)
+          (reference "R17") (unit 1)
         )
       )
@@
   (symbol (lib_id "Device:R") (at 118.11 69.85 0) (unit 1)
     (in_bom yes) (on_board yes) (dnp no) (fields_autoplaced)
-    (property "Reference" "R4" (at 120.65 68.58 0)
+    (property "Reference" "R18" (at 120.65 68.58 0)
       (effects (font (size 1.27 1.27)) (justify left))
     )
@@
       (project "pdp11_front_panel"
         (path "/e63e39d7-6ac0-4ffd-8aa3-1841a4541b55/6921a5ea-b943-4dc1-8acb-8a754944c3ee"
-          (reference "R4") (unit 1)
-        )
-      )
+          (reference "R18") (unit 1)
+        )
+      )

Commit message: wip
Parts:
- JP1, JP2, JP3, JP4, JP5: footprint (none) -> Jumper:SolderJumper-2_P1.3mm_Bridged_RoundedPad1.0x1.5mm
- R16, R17, R18, R19, R20: footprint (none) -> Resistor_SMD:R_1206_3216Metric_Pad1.30x1.75mm_HandSolder
Changed lines of the file:
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@@
       (effects (font (size 1.27 1.27)) (justify left))
     )
-    (property "Footprint" "" (at 129.032 69.85 90)
+    (property "Footprint" "Resistor_SMD:R_1206_3216Metric_Pad1.30x1.75mm_HandSolder" (at 129.032 69.85 90)
       (effects (font (size 1.27 1.27)) hide)
     )
@@
       (effects (font (size 1.27 1.27)) (justify right))
     )
-    (property "Footprint" "" (at 97.79 52.07 0)
+    (property "Footprint" "Jumper:SolderJumper-2_P1.3mm_Bridged_RoundedPad1.0x1.5mm" (at 97.79 52.07 0)
       (effects (font (size 1.27 1.27)) hide)
     )
@@
       (effects (font (size 1.27 1.27)) (justify right))
     )
-    (property "Footprint" "" (at 118.11 52.07 0)
+    (property "Footprint" "Jumper:SolderJumper-2_P1.3mm_Bridged_RoundedPad1.0x1.5mm" (at 118.11 52.07 0)
       (effects (font (size 1.27 1.27)) hide)
     )
@@
       (effects (font (size 1.27 1.27)) (justify right))
     )
-    (property "Footprint" "" (at 140.97 52.07 0)
+    (property "Footprint" "Jumper:SolderJumper-2_P1.3mm_Bridged_RoundedPad1.0x1.5mm" (at 140.97 52.07 0)
       (effects (font (size 1.27 1.27)) hide)
     )
@@
         )
         (path "/e63e39d7-6ac0-4ffd-8aa3-1841a4541b55/6921a5ea-b943-4dc1-8acb-8a754944c3ee"
-          (reference "#PWR038") (unit 1)
+          (reference "#PWR040") (unit 1)
         )
       )
@@
       (effects (font (size 1.27 1.27)) (justify right))
     )
-    (property "Footprint" "" (at 130.81 52.07 0)
+    (property "Footprint" "Jumper:SolderJumper-2_P1.3mm_Bridged_RoundedPad1.0x1.5mm" (at 130.81 52.07 0)
       (effects (font (size 1.27 1.27)) hide)
     )
@@
         )
         (path "/e63e39d7-6ac0-4ffd-8aa3-1841a4541b55/6921a5ea-b943-4dc1-8acb-8a754944c3ee"
-          (reference "#PWR037") (unit 1)
+          (reference "#PWR039") (unit 1)
         )
       )
@@
       (effects (font (size 1.27 1.27)) (justify left))
     )
-    (property "Footprint" "" (at 96.012 69.85 90)
+    (property "Footprint" "Resistor_SMD:R_1206_3216Metric_Pad1.30x1.75mm_HandSolder" (at 96.012 69.85 90)
       (effects (font (size 1.27 1.27)) hide)
     )
@@
       (effects (font (size 1.27 1.27)) (justify left))
     )
-    (property "Footprint" "" (at 139.192 69.85 90)
+    (property "Footprint" "Resistor_SMD:R_1206_3216Metric_Pad1.30x1.75mm_HandSolder" (at 139.192 69.85 90)
       (effects (font (size 1.27 1.27)) hide)
     )
@@
         )
         (path "/e63e39d7-6ac0-4ffd-8aa3-1841a4541b55/6921a5ea-b943-4dc1-8acb-8a754944c3ee"
-          (reference "#PWR036") (unit 1)
+          (reference "#PWR038") (unit 1)
         )
       )
@@
       (effects (font (size 1.27 1.27)) (justify left))
     )
-    (property "Footprint" "" (at 106.172 69.85 90)
+    (property "Footprint" "Resistor_SMD:R_1206_3216Metric_Pad1.30x1.75mm_HandSolder" (at 106.172 69.85 90)
       (effects (font (size 1.27 1.27)) hide)
     )
@@
       (effects (font (size 1.27 1.27)) (justify left))
     )
-    (property "Footprint" "" (at 116.332 69.85 90)
+    (property "Footprint" "Resistor_SMD:R_1206_3216Metric_Pad1.30x1.75mm_HandSolder" (at 116.332 69.85 90)
       (effects (font (size 1.27 1.27)) hide)
     )
@@
       (effects (font (size 1.27 1.27)) (justify right))
     )
-    (property "Footprint" "" (at 107.95 52.07 0)
-      (effects (font (size 1.27 1.27)) hide)
-    )
+    (property "Footprint" "Jumper:SolderJumper-2_P1.3mm_Bridged_RoundedPad1.0x1.5mm" (at 107.95 52.07 0)
+      (effects (font (size 1.27 1.27)) hide)
+    )
