File: projects/pdp11_front_panel/controller.kicad_sch (KiCad schematic)
At the start: 10 parts, among them J3 Conn_01x05_Pin, Q1 2N7000, U1 Arduino_Micro, U2 AM26S10CDRG4

Commit message: wip
Parts:
- added J6: Conn_01x02_Pin, symbol Connector:Conn_01x02_Pin
- added R10: 10K, symbol Device:R
Connections:
- net ANN_SPARE0 is gone; now on net SW_AUX: U1.8 (~D3/SCL)
- net +5VA: now also R10.1
- net GND: now also J6.2 (Pin_2)
- net SW_AUX: no longer U1.17 (D12/A11)
- new net 60HZ/50HZ#: J6.1 (Pin_1), R10.2, U1.17 (D12/A11)
Other:
- sheet Power Switch2 renamed Aux Switch
- removed sheet Spare 0 Annunciator
- note added: "Install jumper for 50Hz"
- note added: "Placce near U1."
- note added: "Place near U2."
- moved on the sheet: C2, C3, R12, U1

Commit message: wip
Parts:
- removed J6: Conn_01x02_Pin, symbol Connector:Conn_01x02_Pin
- added J3: Conn_01x02, symbol Connector_Generic:Conn_01x02
- C2: footprint (none) -> Capacitor_SMD:C_0603_1608Metric_Pad1.08x0.95mm_HandSolder
- C3: value C -> 1u; footprint (none) -> Capacitor_SMD:C_0603_1608Metric_Pad1.08x0.95mm_HandSolder
- J4: renamed from J3; footprint (none) -> Connector_PinHeader_2.54mm:PinHeader_1x05_P2.54mm_Vertical
- R11: renamed from R10; footprint (none) -> Resistor_SMD:R_1206_3216Metric_Pad1.30x1.75mm_HandSolder
- R12, R13, R5, R6: footprint (none) -> Resistor_SMD:R_1206_3216Metric_Pad1.30x1.75mm_HandSolder
- U2: footprint AM26S10CDRG4:SOIC127P600X175-16N -> ch:SOIC127P600X175-16N
Connections:
- net 60HZ/50HZ#: now also J3.2 (Pin_2)
- net GND: now also J3.1 (Pin_1)

Commit message: wip
Parts:
- removed Q1: 2N7000, Package_TO_SOT_THT:TO-92_Inline, symbol Transistor_FET:2N7000
- added Q2: 2N7002, Package_TO_SOT_SMD:SOT-23, symbol Transistor_FET:2N7002
- J3: footprint (none) -> Connector_PinHeader_2.54mm:PinHeader_1x02_P2.54mm_Vertical
Connections:
- net ATX_PS_ON#: now also Q2.3 (D)
- net GND: now also Q2.2 (S)
- net at R5.2, R6.1: now also Q2.1 (G)
Changed lines of the file:
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@@
       (effects (font (size 1.27 1.27)))
     )
-    (property "Footprint" "" (at 29.21 156.21 0)
+    (property "Footprint" "Connector_PinHeader_2.54mm:PinHeader_1x02_P2.54mm_Vertical" (at 29.21 156.21 0)
       (effects (font (size 1.27 1.27)) hide)
     )
@@
     )
   )
+  (symbol (lib_id "Transistor_FET:2N7002") (at 219.71 135.89 0) (unit 1)
+    (in_bom yes) (on_board yes) (dnp no) (fields_autoplaced)
+    (property "Reference" "Q2" (at 226.06 134.62 0)
+      (effects (font (size 1.27 1.27)) (justify left))
+    )
+    (property "Value" "2N7002" (at 226.06 137.16 0)
+      (effects (font (size 1.27 1.27)) (justify left))
+    )
+    (property "Footprint" "Package_TO_SOT_SMD:SOT-23" (at 224.79 137.795 0)
+      (effects (font (size 1.27 1.27) italic) (justify left) hide)
+    )
+    (property "Datasheet" "https://www.onsemi.com/pub/Collateral/NDS7002A-D.PDF" (at 219.71 135.89 0)
+      (effects (font (size 1.27 1.27)) (justify left) hide)
+    )
+    (pin "1")
+    (pin "2")
+    (pin "3")
+    (instances
+      (project "pdp11_front_panel"
+        (path "/e63e39d7-6ac0-4ffd-8aa3-1841a4541b55/9c91720a-c48c-49a5-8459-4bb13d4bbf8a"
+          (reference "Q2") (unit 1)
+        )
+      )
+    )
+  )
   (symbol (lib_id "power:+5VA") (at 31.75 175.26 0) (unit 1)
     (in_bom yes) (on_board yes) (dnp no) (fields_autoplaced)
@@
         )
       )
-    )
-  )
-  (symbol (lib_id "Transistor_FET:2N7000") (at 219.71 135.89 0) (unit 1)
-    (in_bom yes) (on_board yes) (dnp no) (fields_autoplaced)
-    (property "Reference" "Q1" (at 226.06 134.62 0)
-      (effects (font (size 1.27 1.27)) (justify left))
-    )
-    (property "Value" "2N7000" (at 226.06 137.16 0)
-      (effects (font (size 1.27 1.27)) (justify left))
-    )
-    (property "Footprint" "Package_TO_SOT_THT:TO-92_Inline" (at 224.79 137.795 0)
-      (effects (font (size 1.27 1.27) italic) (justify left) hide)
-    )
-    (property "Datasheet" "https://www.vishay.com/docs/70226/70226.pdf" (at 219.71 135.89 0)
-      (effects (font (size 1.27 1.27)) (justify left) hide)
-    )
-    (pin "1")
-    (pin "2")
-    (pin "3")
-    (instances
-      (project "pdp11_front_panel"
-        (path "/e63e39d7-6ac0-4ffd-8aa3-1841a4541b55/ac18ea73-065c-46aa-ad52-732cc0cb5b05"
-          (reference "Q1") (unit 1)
-        )
-        (path "/e63e39d7-6ac0-4ffd-8aa3-1841a4541b55/9c91720a-c48c-49a5-8459-4bb13d4bbf8a"
-          (reference "Q2") (unit 1)
-        )
-      )

Commit message: .
Parts:
- removed U1: Arduino_Micro, Arduino:Arduino_Micro, symbol arduino:Arduino_Micro
- renumbered R5 to R14, R6 to R15
Other:
- moved on the sheet: R12
