File: projects/pdp11_front_panel/switch.kicad_sch (KiCad schematic)
At the start: 3 parts, among them SW2 SW_SPDT

Commit message: wip
Parts:
- C3: footprint (none) -> Capacitor_SMD:C_0603_1608Metric_Pad1.08x0.95mm_HandSolder
- R21: footprint (none) -> Resistor_SMD:R_1206_3216Metric_Pad1.30x1.75mm_HandSolder
Changed lines of the file:
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@@
     (effects (font (size 1.27 1.27)) (justify right))
   )
-  (hierarchical_label "VCC" (shape passive) (at 88.9 41.91 90) (fields_autoplaced)
+  (hierarchical_label "SW" (shape output) (at 132.08 49.53 0) (fields_autoplaced)
     (effects (font (size 1.27 1.27)) (justify left))
   )
-  (hierarchical_label "SW" (shape output) (at 132.08 49.53 0) (fields_autoplaced)
+  (hierarchical_label "VCC" (shape passive) (at 88.9 41.91 90) (fields_autoplaced)
     (effects (font (size 1.27 1.27)) (justify left))
   )
@@
     )
   )
+  (symbol (lib_id "Device:R") (at 110.49 49.53 90) (unit 1)
+    (in_bom yes) (on_board yes) (dnp no) (fields_autoplaced)
+    (property "Reference" "R21" (at 110.49 43.18 90)
+      (effects (font (size 1.27 1.27)))
+    )
+    (property "Value" "10K" (at 110.49 45.72 90)
+      (effects (font (size 1.27 1.27)))
+    )
+    (property "Footprint" "Resistor_SMD:R_1206_3216Metric_Pad1.30x1.75mm_HandSolder" (at 110.49 51.308 90)
+      (effects (font (size 1.27 1.27)) hide)
+    )
+    (property "Datasheet" "~" (at 110.49 49.53 0)
+      (effects (font (size 1.27 1.27)) hide)
+    )
+    (pin "1")
+    (pin "2")
+    (instances
+      (project "pdp11_front_panel"
+        (path "/e63e39d7-6ac0-4ffd-8aa3-1841a4541b55/9c91720a-c48c-49a5-8459-4bb13d4bbf8a"
+          (reference "R21") (unit 1)
+        )
+        (path "/e63e39d7-6ac0-4ffd-8aa3-1841a4541b55/9c91720a-c48c-49a5-8459-4bb13d4bbf8a/f2405389-79c5-45c7-90a8-7b3da2b876ad"
+          (reference "R24") (unit 1)
+        )
+        (path "/e63e39d7-6ac0-4ffd-8aa3-1841a4541b55/9c91720a-c48c-49a5-8459-4bb13d4bbf8a/b89f43e1-0f50-478b-ba15-0cf7977e6432"
+          (reference "R10") (unit 1)
+        )
+        (path "/e63e39d7-6ac0-4ffd-8aa3-1841a4541b55/9c91720a-c48c-49a5-8459-4bb13d4bbf8a/b9a90149-907d-418a-99b6-1b0dfcd047ff"
+          (reference "R22") (unit 1)
+        )
+        (path "/e63e39d7-6ac0-4ffd-8aa3-1841a4541b55/9c91720a-c48c-49a5-8459-4bb13d4bbf8a/9ff020da-711e-42e7-aa10-8ef407e2bd65"
+          (reference "R23") (unit 1)
+        )
+      )
+    )
+  )
   (symbol (lib_id "Device:C") (at 116.84 54.61 0) (unit 1)
     (in_bom yes) (on_board yes) (dnp no) (fields_autoplaced)
@@
       (effects (font (size 1.27 1.27)) (justify left))
     )
-    (property "Footprint" "" (at 117.8052 58.42 0)
+    (property "Footprint" "Capacitor_SMD:C_0603_1608Metric_Pad1.08x0.95mm_HandSolder" (at 117.8052 58.42 0)
       (effects (font (size 1.27 1.27)) hide)
     )
@@
         )
       )
-    )
-  )
-  (symbol (lib_id "Device:R") (at 110.49 49.53 90) (unit 1)
-    (in_bom yes) (on_board yes) (dnp no) (fields_autoplaced)
-    (property "Reference" "R21" (at 110.49 43.18 90)
-      (effects (font (size 1.27 1.27)))
-    )
-    (property "Value" "10K" (at 110.49 45.72 90)
-      (effects (font (size 1.27 1.27)))
-    )
-    (property "Footprint" "" (at 110.49 51.308 90)
-      (effects (font (size 1.27 1.27)) hide)
-    )
-    (property "Datasheet" "~" (at 110.49 49.53 0)
-      (effects (font (size 1.27 1.27)) hide)
-    )
-    (pin "1")
-    (pin "2")
-    (instances
-      (project "pdp11_front_panel"
-        (path "/e63e39d7-6ac0-4ffd-8aa3-1841a4541b55/9c91720a-c48c-49a5-8459-4bb13d4bbf8a"
-          (reference "R21") (unit 1)
-        )
-        (path "/e63e39d7-6ac0-4ffd-8aa3-1841a4541b55/9c91720a-c48c-49a5-8459-4bb13d4bbf8a/f2405389-79c5-45c7-90a8-7b3da2b876ad"
-          (reference "R24") (unit 1)
-        )
-        (path "/e63e39d7-6ac0-4ffd-8aa3-1841a4541b55/9c91720a-c48c-49a5-8459-4bb13d4bbf8a/b89f43e1-0f50-478b-ba15-0cf7977e6432"
-          (reference "R11") (unit 1)
-        )
-        (path "/e63e39d7-6ac0-4ffd-8aa3-1841a4541b55/9c91720a-c48c-49a5-8459-4bb13d4bbf8a/b9a90149-907d-418a-99b6-1b0dfcd047ff"
-          (reference "R22") (unit 1)
-        )
-        (path "/e63e39d7-6ac0-4ffd-8aa3-1841a4541b55/9c91720a-c48c-49a5-8459-4bb13d4bbf8a/9ff020da-711e-42e7-aa10-8ef407e2bd65"
-          (reference "R23") (unit 1)
-        )
-      )

Commit message: .
Parts:
- renumbered C3 to C6, R21 to R24
Changed lines of the file:
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@@
       )
       (project "pdp11_front_panel"
-        (path "/e63e39d7-6ac0-4ffd-8aa3-1841a4541b55/9c91720a-c48c-49a5-8459-4bb13d4bbf8a"
-          (reference "SW1") (unit 1)
-        )
         (path "/e63e39d7-6ac0-4ffd-8aa3-1841a4541b55/9c91720a-c48c-49a5-8459-4bb13d4bbf8a/f2405389-79c5-45c7-90a8-7b3da2b876ad"
           (reference "SW4") (unit 1)
@@
         (path "/e63e39d7-6ac0-4ffd-8aa3-1841a4541b55/9c91720a-c48c-49a5-8459-4bb13d4bbf8a/b89f43e1-0f50-478b-ba15-0cf7977e6432"
           (reference "SW1") (unit 1)
-        )
-        (path "/e63e39d7-6ac0-4ffd-8aa3-1841a4541b55/9c91720a-c48c-49a5-8459-4bb13d4bbf8a/b9a90149-907d-418a-99b6-1b0dfcd047ff"
-          (reference "SW2") (unit 1)
         )
         (path "/e63e39d7-6ac0-4ffd-8aa3-1841a4541b55/9c91720a-c48c-49a5-8459-4bb13d4bbf8a/9ff020da-711e-42e7-aa10-8ef407e2bd65"
@@
   (symbol (lib_id "Device:R") (at 110.49 49.53 90) (unit 1)
     (in_bom yes) (on_board yes) (dnp no) (fields_autoplaced)
-    (property "Reference" "R21" (at 110.49 43.18 90)
+    (property "Reference" "R24" (at 110.49 43.18 90)
       (effects (font (size 1.27 1.27)))
     )
@@
     (instances
       (project "pdp11_front_panel"
-        (path "/e63e39d7-6ac0-4ffd-8aa3-1841a4541b55/9c91720a-c48c-49a5-8459-4bb13d4bbf8a"
-          (reference "R21") (unit 1)
-        )
         (path "/e63e39d7-6ac0-4ffd-8aa3-1841a4541b55/9c91720a-c48c-49a5-8459-4bb13d4bbf8a/f2405389-79c5-45c7-90a8-7b3da2b876ad"
           (reference "R24") (unit 1)
@@
         (path "/e63e39d7-6ac0-4ffd-8aa3-1841a4541b55/9c91720a-c48c-49a5-8459-4bb13d4bbf8a/b89f43e1-0f50-478b-ba15-0cf7977e6432"
           (reference "R10") (unit 1)
-        )
-        (path "/e63e39d7-6ac0-4ffd-8aa3-1841a4541b55/9c91720a-c48c-49a5-8459-4bb13d4bbf8a/b9a90149-907d-418a-99b6-1b0dfcd047ff"
-          (reference "R22") (unit 1)
         )
         (path "/e63e39d7-6ac0-4ffd-8aa3-1841a4541b55/9c91720a-c48c-49a5-8459-4bb13d4bbf8a/9ff020da-711e-42e7-aa10-8ef407e2bd65"
@@
   (symbol (lib_id "Device:C") (at 116.84 54.61 0) (unit 1)
     (in_bom yes) (on_board yes) (dnp no) (fields_autoplaced)
-    (property "Reference" "C3" (at 120.65 53.34 0)
+    (property "Reference" "C6" (at 120.65 53.34 0)
       (effects (font (size 1.27 1.27)) (justify left))
     )
@@
     (instances
       (project "pdp11_front_panel"
-        (path "/e63e39d7-6ac0-4ffd-8aa3-1841a4541b55/9c91720a-c48c-49a5-8459-4bb13d4bbf8a"
-          (reference "C3") (unit 1)
-        )
         (path "/e63e39d7-6ac0-4ffd-8aa3-1841a4541b55/9c91720a-c48c-49a5-8459-4bb13d4bbf8a/f2405389-79c5-45c7-90a8-7b3da2b876ad"
           (reference "C6") (unit 1)
@@
           (reference "C1") (unit 1)
         )
-        (path "/e63e39d7-6ac0-4ffd-8aa3-1841a4541b55/9c91720a-c48c-49a5-8459-4bb13d4bbf8a/b9a90149-907d-418a-99b6-1b0dfcd047ff"
-          (reference "C4") (unit 1)
-        )
         (path "/e63e39d7-6ac0-4ffd-8aa3-1841a4541b55/9c91720a-c48c-49a5-8459-4bb13d4bbf8a/9ff020da-711e-42e7-aa10-8ef407e2bd65"

Commit message: Clean up and push random stuff.
Parts:
- renumbered C6 to C1, R24 to R10, SW2 to SW1
