File: projects/stm32g0_usbc/stm32g0_usbc.kicad_sch (KiCad schematic)
At the start: 27 parts, among them J1 USB_C_Receptacle_USB2.0, J3 Conn_ARM_JTAG_SWD_10, U1 STM32G0B1CBT, U2 MCP1754S-3302xMB, U3 8MHz 20pF ±10ppm, Y2 NX3225GD 8 MHz

Commit message: .
Parts:
- removed U3: 8MHz 20pF ±10ppm, JLCPCB:OSC-SMD_L5.0-W3.2, symbol JLCPCB Chips, Crystals:8MHz 20pF ±10ppm
- removed Y2: NX3225GD 8 MHz, Crystal:Crystal_SMD_3215-2Pin_3.2x1.5mm, symbol Device:Crystal
- added C10, C4: 100n, Capacitor_SMD:C_0603_1608Metric, symbol Device:C
- added D4: NUP2105L, Package_TO_SOT_SMD:SOT-23, symbol Power_Protection:NUP2105L
- added D5: D_Schottky, Diode_SMD:D_SMA, symbol Device:D_Schottky
- added J2: DE9_Plug, Connector_Dsub:DSUB-9_Male_Horizontal_P2.77x2.84mm_EdgePinOffset4.94mm_Housed_MountingHolesOffset7.48mm, symbol Connector:DE9_Plug
- added J4: Conn_01x02, Connector_PinHeader_2.54mm:PinHeader_1x02_P2.54mm_Vertical, symbol Connector_Generic:Conn_01x02
- added J5: Screw_Terminal_01x03, TerminalBlock_Phoenix:TerminalBlock_Phoenix_MKDS-1,5-3_1x03_P5.00mm_Horizontal, symbol Connector:Screw_Terminal_01x03
- added J6: 5054481071, molex_microlock_plus:MOLEX_5054481071, symbol molex_microlock_plus:5054481071
- added J7: Conn_Coaxial_Power, Connector_BarrelJack:BarrelJack_CUI_PJ-063AH_Horizontal, symbol Connector:Conn_Coaxial_Power
- added J8: Screw_Terminal_01x02, TerminalBlock_Phoenix:TerminalBlock_Phoenix_MKDS-1,5-2-5.08_1x02_P5.08mm_Horizontal, symbol Connector:Screw_Terminal_01x02
- added R10, R9: 0, Resistor_SMD:R_1206_3216Metric, symbol Device:R
- added R7: DNI, Resistor_SMD:R_1206_3216Metric, symbol Device:R
- added R8: 120, Resistor_SMD:R_1206_3216Metric, symbol Device:R
- added U3: TJA1051T-3, Package_SO:SOIC-8_3.9x4.9mm_P1.27mm, symbol Interface_CAN_LIN:TJA1051T-3
- added Y1: Crystal_GND24_Small, Crystal:Crystal_SMD_3225-4Pin_3.2x2.5mm, symbol Device:Crystal_GND24_Small
Connections:
- net +3V3: now also C4.1, U3.5 (VIO)
- net +5V: now also C10.1, U3.3 (VCC)
- net GND: now also C10.2, C4.2, D4.3 (A), J2.6, J5.3 (Pin_3), J6.2, J6.4, J6.6, J6.S1 (SHIELD1), J6.S2 (SHIELD2), J7.2 (Ext), J8.2 (Pin_2), R10.2, R7.2, R9.2, U3.2 (GND), Y1.2, Y1.4
- net OSC_IN: now also Y1.1
- net OSC_OUT: now also Y1.3
- net CAN1_S: now reaches U1.37 (PA15)
- net CAN1_S: now also U3.8 (S)
- net CAN1_RX: now reaches U1.38 (PD0)
- net CAN1_RX: now also U3.4 (RXD)
- net CAN1_TX: now reaches U1.39 (PD1)
- net CAN1_TX: now also U3.1 (TXD)
- new net: J4.2 (Pin_2), R8.1
- new net +12V: D5.1 (K), J6.1, J6.3, J6.5
- new net +12V_IN: D5.2 (A), J7.1 (In), J8.1 (Pin_1)
- new net 12V_SHIELD: J6.7, R9.1
- new net CAN1_H: D4.1 (K), J2.7, J4.1 (Pin_1), J5.1 (Pin_1), J6.9, U3.7 (CANH)
- new net CAN1_L: D4.2 (K), J2.2, J5.2 (Pin_2), J6.10, R8.2, U3.6 (CANL)
- new net CAN1_SH: J2.5, R7.1
- new net SHIELD: J6.8, R10.1
- no-connect marks 39 -> 40
Other:
- moved on the sheet: C1, C3, C5, C6, C7, C8, C9, D1, D2, D3, J3, R1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

Commit message: 1v0
Parts:
- removed U2: MCP1754S-3302xMB, Package_TO_SOT_SMD:SOT-89-3, symbol Regulator_Linear:MCP1754S-3302xMB
- added U4: LP5907MFX-3.3, Package_TO_SOT_SMD:SOT-23-5, symbol Regulator_Linear:LP5907MFX-3.3
- J1: symbol Connector:USB_C_Receptacle_USB2.0 -> Connector:USB_C_Receptacle_USB2.0_16P
Connections:
- net +3V3: now also U4.5 (OUT)
- net +5V: now also U4.1 (IN), U4.3 (EN)
- net GND: now also U4.2 (GND)
- no-connect marks 40 -> 41
Other:
- note removed: "150 mA"
- moved on the sheet: C1, C3, C7, C8, C9, D4, D5, J2, J4, J6, J7, J8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

Commit message: .
Other:
- note added: "8 MHz 3225"
Changed lines of the file:
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@@
     (stroke (width 0) (type default))
+  )
+  (text "8 MHz 3225" (at 26.67 123.19 0)
+    (effects (font (size 1.27 1.27)) (justify left bottom))
   )
   (label "NRESET" (at 154.94 166.37 0) (fields_autoplaced)

Commit message: lcsc
Parts:
- C3, C4, C9: LCSC (none) -> C14663
- C7, C8: value 6p2 -> 6p2 C0G
- D5: LCSC (none) -> C2997264
- FB1: LCSC (none) -> C62708
- J3: LCSC (none) -> C5160761; now not fitted
- J5, J8: now not fitted
- R10, R9: LCSC (none) -> C473612
- R7: value DNI -> 0; LCSC (none) -> C473612; now not fitted
- U3: LCSC (none) -> C5342108
- U4: LCSC (none) -> C80670
- Y1: LCSC (none) -> C518135
Changed lines of the file:
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@@
+      (effects (font (size 1.27 1.27)) hide)
+    )
+    (property "LCSC" "C80670" (at 91.44 171.45 0)
       (effects (font (size 1.27 1.27)) hide)
     )
@@
   )
   (symbol (lib_id "Connector:Screw_Terminal_01x03") (at 261.62 93.98 0) (unit 1)
-    (in_bom yes) (on_board yes) (dnp no) (fields_autoplaced)
+    (in_bom yes) (on_board yes) (dnp yes) (fields_autoplaced)
     (property "Reference" "J5" (at 264.16 92.71 0)
       (effects (font (size 1.27 1.27)) (justify left))
@@
     )
     (property "Datasheet" "~" (at 30.48 132.08 0)
+      (effects (font (size 1.27 1.27)) hide)
+    )
+    (property "LCSC" "C518135" (at 30.48 132.08 0)
       (effects (font (size 1.27 1.27)) hide)
     )
@@
   )
   (symbol (lib_id "Device:R") (at 248.92 139.7 0) (unit 1)
-    (in_bom yes) (on_board yes) (dnp no) (fields_autoplaced)
+    (in_bom yes) (on_board yes) (dnp yes) (fields_autoplaced)
     (property "Reference" "R7" (at 251.46 138.43 0)
       (effects (font (size 1.27 1.27)) (justify left))
     )
-    (property "Value" "DNI" (at 251.46 140.97 0)
+    (property "Value" "0" (at 251.46 140.97 0)
       (effects (font (size 1.27 1.27)) (justify left))
     )
@@
     )
     (property "Datasheet" "~" (at 248.92 139.7 0)
+      (effects (font (size 1.27 1.27)) hide)
+    )
+    (property "LCSC" "C473612" (at 248.92 139.7 0)
       (effects (font (size 1.27 1.27)) hide)
     )
@@
   (symbol (lib_id "Device:C") (at 22.86 135.89 0) (unit 1)
     (in_bom yes) (on_board yes) (dnp no)
-    (property "Reference" "C7" (at 15.875 134.62 0)
-      (effects (font (size 1.27 1.27)) (justify left))
-    )
-    (property "Value" "6p2" (at 15.875 137.16 0)
+    (property "Reference" "C7" (at 16.51 135.89 0)
+      (effects (font (size 1.27 1.27)) (justify left))
+    )
+    (property "Value" "6p2 C0G" (at 15.24 138.43 0)
       (effects (font (size 1.27 1.27)) (justify left))
     )
@@
       (effects (font (size 1.27 1.27)) hide)
     )
+    (property "LCSC" "C62708" (at 73.66 29.21 90)
+      (effects (font (size 1.27 1.27)) hide)
+    )
     (pin "2")
     (pin "1")
@@
     )
     (property "Datasheet" "~" (at 270.51 41.91 0)
+      (effects (font (size 1.27 1.27)) hide)
+    )
+    (property "LCSC" "C473612" (at 270.51 41.91 0)
       (effects (font (size 1.27 1.27)) hide)
     )
@@
       (effects (font (size 1.27 1.27)) hide)
     )
+    (property "LCSC" "C473612" (at 227.33 40.64 0)
+      (effects (font (size 1.27 1.27)) hide)
+    )
     (pin "1")
     (pin "2")
@@
       (effects (font (size 1.27 1.27)) hide)
     )
+    (property "LCSC" "C14663" (at 54.61 135.89 0)
+      (effects (font (size 1.27 1.27)) hide)
+    )
     (pin "2")
     (pin "1")
@@
       (effects (font (size 1.27 1.27)) (justify left))
     )
-    (property "Value" "6p2" (at 41.275 137.16 0)
+    (property "Value" "6p2 C0G" (at 41.275 137.16 0)
       (effects (font (size 1.27 1.27)) (justify left))
     )
@@
       (effects (font (size 1.27 1.27)) hide)
     )
+    (property "LCSC" "C14663" (at 34.29 104.14 0)
+      (effects (font (size 1.27 1.27)) hide)
+    )
     (pin "1")
     (pin "2")
@@
   )
   (symbol (lib_id "Connector:Screw_Terminal_01x02") (at 177.8 38.1 0) (unit 1)
-    (in_bom yes) (on_board yes) (dnp no) (fields_autoplaced)
+    (in_bom yes) (on_board yes) (dnp yes) (fields_autoplaced)
     (property "Reference" "J8" (at 180.975 38.1 0)
       (effects (font (size 1.27 1.27)) (justify left))
@@
     )
     (property "Datasheet" "~" (at 153.67 100.33 0)
+      (effects (font (size 1.27 1.27)) hide)
+    )
+    (property "LCSC" "C14663" (at 153.67 100.33 0)
       (effects (font (size 1.27 1.27)) hide)
     )
@@
       (effects (font (size 1.27 1.27)) hide)
     )
+    (property "LCSC" "C5342108" (at 185.42 92.71 0)
+      (effects (font (size 1.27 1.27)) hide)
+    )
     (pin "8")
     (pin "1")
@@
     )
     (property "Datasheet" "~" (at 179.07 30.48 0)
+      (effects (font (size 1.27 1.27)) hide)
+    )
+    (property "LCSC" "C2997264" (at 179.07 30.48 0)
       (effects (font (size 1.27 1.27)) hide)
     )
@@
   )
   (symbol (lib_id "Connector:Conn_ARM_JTAG_SWD_10") (at 140.97 173.99 0) (unit 1)
-    (in_bom yes) (on_board yes) (dnp no)
+    (in_bom yes) (on_board yes) (dnp yes)
     (property "Reference" "J3" (at 154.305 186.055 0)
       (effects (font (size 1.27 1.27)) (justify right))
@@
       (effects (font (size 1.27 1.27)) hide)
     )
+    (property "LCSC" "C5160761" (at 140.97 173.99 0)
+      (effects (font (size 1.27 1.27)) hide)
+    )

Commit message: small tweaks
Parts:
- J4: footprint Connector_PinHeader_2.54mm:PinHeader_1x02_P2.54mm_Vertical -> Connector_PinHeader_2.54mm:PinHeader_1x03_P2.54mm_Vertical; symbol Connector_Generic:Conn_01x02 -> Connector_Generic:Conn_01x03
Connections:
- net CAN1_H: now also J4.2 (Pin_2); no longer J4.1 (Pin_1)
- net at R8.1: now also J4.3 (Pin_3); no longer J4.2 (Pin_2)
- no-connect marks 41 -> 42

Commit message: .
Parts:
- C7, C8: value 6p2 C0G -> 6.2p C0G
- D1: LCSC (none) -> C9900012286
- D2: LCSC (none) -> C3030991
- D3: LCSC (none) -> C5252984
- D4: LCSC (none) -> C284104
- J2: LCSC (none) -> C3134122
- J6: LCSC (none) -> C17610436
- J7: LCSC (none) -> C2928097
Changed lines of the file:
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@@
+      (effects (font (size 1.27 1.27)) hide)
+    )
+    (property "LCSC" "C5252984" (at 58.42 180.34 90)
+      (effects (font (size 1.27 1.27)) hide)
+    )
+    (property "Field5" "" (at 58.42 180.34 90)
       (effects (font (size 1.27 1.27)) hide)
     )
@@
     )
     (property "Datasheet" " ~" (at 265.43 127 0)
+      (effects (font (size 1.27 1.27)) hide)
+    )
+    (property "LCSC" "C3134122" (at 265.43 127 0)
       (effects (font (size 1.27 1.27)) hide)
     )
@@
       (effects (font (size 1.27 1.27)) (justify left))
     )
-    (property "Value" "6p2 C0G" (at 15.24 138.43 0)
+    (property "Value" "6.2p C0G" (at 15.24 138.43 0)
       (effects (font (size 1.27 1.27)) (justify left))
     )
@@
       (effects (font (size 1.27 1.27)) hide)
     )
+    (property "LCSC" "C284104" (at 242.57 139.7 0)
+      (effects (font (size 1.27 1.27)) hide)
+    )
     (pin "3")
     (pin "2")
@@
       (effects (font (size 1.27 1.27)) (justify left))
     )
-    (property "Value" "6p2 C0G" (at 41.275 137.16 0)
+    (property "Value" "6.2p C0G" (at 41.275 137.16 0)
       (effects (font (size 1.27 1.27)) (justify left))
     )
@@
       (effects (font (size 1.27 1.27)) hide)
     )
+    (property "LCSC" "C9900012286" (at 31.75 180.34 90)
+      (effects (font (size 1.27 1.27)) hide)
+    )
     (pin "2")
     (pin "1")
@@
     )
     (property "Datasheet" "~" (at 45.72 180.34 0)
+      (effects (font (size 1.27 1.27)) hide)
+    )
+    (property "LCSC" "C3030991" (at 45.72 180.34 90)
       (effects (font (size 1.27 1.27)) hide)
     )
@@
       (effects (font (size 1.27 1.27)) (justify bottom) hide)
     )
+    (property "LCSC" "C17610436" (at 248.92 34.29 0)
+      (effects (font (size 1.27 1.27)) hide)
+    )
     (pin "6")
     (pin "S2")
@@
       (effects (font (size 1.27 1.27)) hide)
     )
+    (property "LCSC" "C2928097" (at 165.1 30.48 90)
+      (effects (font (size 1.27 1.27)) hide)
+    )

Commit message: .
Parts:
- D1: MPN (none) -> 150060YS75000
- D2: MPN (none) -> 150060RS75000
- D3: MPN (none) -> 150060GS75000
- J6: MPN (none) -> 5054481071
- J7: Digikey (none) -> CP-063AH-ND; MPN (none) -> PJ-063AH
Changed lines of the file:
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@@
       (effects (font (size 1.27 1.27)) hide)
     )
-    (property "Field5" "" (at 58.42 180.34 90)
+    (property "MPN" "150060GS75000" (at 58.42 180.34 90)
       (effects (font (size 1.27 1.27)) hide)
     )
@@
       (effects (font (size 1.27 1.27)) hide)
     )
+    (property "MPN" "150060YS75000" (at 31.75 180.34 90)
+      (effects (font (size 1.27 1.27)) hide)
+    )
     (pin "2")
     (pin "1")
@@
     )
     (property "LCSC" "C3030991" (at 45.72 180.34 90)
+      (effects (font (size 1.27 1.27)) hide)
+    )
+    (property "MPN" "150060RS75000" (at 45.72 180.34 90)
       (effects (font (size 1.27 1.27)) hide)
     )
@@
       (effects (font (size 1.27 1.27)) hide)
     )
+    (property "MPN" "5054481071" (at 248.92 34.29 0)
+      (effects (font (size 1.27 1.27)) hide)
+    )
     (pin "6")
     (pin "S2")
@@
       (effects (font (size 1.27 1.27)) hide)
     )
+    (property "Digikey" "CP-063AH-ND" (at 165.1 30.48 90)
+      (effects (font (size 1.27 1.27)) hide)
+    )
+    (property "MPN" "PJ-063AH" (at 165.1 30.48 90)
+      (effects (font (size 1.27 1.27)) hide)
+    )
