File: projects/rpi_sa8x8hat/rpi_sa8x8hat.kicad_sch (KiCad schematic)
At the start: 5 parts, among them J1 RPi_GPIO

Commit message: .
Parts:
- removed H1, H2, H3, H4: MountingHole, RPi_Hat:RPi_Hat_Mounting_Hole, symbol Mechanical:MountingHole
- added H1, H2, H3, H4: MountingHole_Pad, rpi_sa8x8hat:RPi_Hat_Mounting_Hole, symbol Mechanical:MountingHole_Pad
- J1: footprint RPi_Hat:Samtec_HLE-120-02-XXX-DV-BE-XX-XX -> rpi_sa8x8hat:Samtec_HLE-120-02-XXX-DV-BE-XX-XX; symbol RPi_Hat:RPi_GPIO -> rpi_sa8x8hat:RPi_GPIO
Connections:
- net 3V3: now reaches J1.1 (3.3V)
- net 3V3: now also J1.17 (3.3V)
- net GND: now reaches J1.14 (GND)
- net GND: now also J1.20 (GND), J1.25 (GND), J1.30 (GND), J1.34 (GND), J1.39 (GND), J1.6 (GND), J1.9 (GND), H1.1, H2.1, H3.1, H4.1
- net 5V: now reaches J1.2 (5V)
- net 5V: now also J1.4 (5V)
- net BCM_ID_SDA: now reaches J1.27 (BCM0_ID_SD)
- net BCM_ID_SCL: now reaches J1.28 (BCM1_ID_SC)
- net BCM_I2S_WCLK: now reaches J1.35 (BCM19_MISO_PCM_FS)
- net BCM_I2S_IN: now reaches J1.38 (BCM20_MOSI_PCM_DI)
- net BCM_I2S_OUT: now reaches J1.40 (BCM21_SCLK_PCM_DO)

Commit message: WIP
Parts:
- added FL1: LPF, rpi_sa8x8hat:0500LP15A500, symbol rpi_s8x8hat:LPF
- added U1: SA818, rpi_sa8x8hat:SA818, symbol rpi_s8x8hat:SA818
Connections:
- net GND: now also FL1.1 (GND), FL1.3 (GND), FL1.5 (GND), FL1.7 (GND)
- new net: FL1.8 (IN), U1.12 (ANT)
Changed lines of the file:
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@@
   (junction (at 100.965 35.56) (diameter 0) (color 0 0 0 0)
   )
+  (junction (at 209.55 67.31) (diameter 0) (color 0 0 0 0)
+  )
+  (junction (at 212.09 67.31) (diameter 0) (color 0 0 0 0)
+  )
   (junction (at 49.53 35.56) (diameter 0) (color 0 0 0 0)
   )
@@
   (junction (at 16.51 176.53) (diameter 0) (color 0 0 0 0)
   )
+  (junction (at 214.63 67.31) (diameter 0) (color 0 0 0 0)
+  )
   (junction (at 16.51 186.69) (diameter 0) (color 0 0 0 0)
   )
@@
     (stroke (width 0) (type default))
   )
+  (wire (pts (xy 212.09 67.31) (xy 209.55 67.31))
+    (stroke (width 0) (type default))
+  )
   (wire (pts (xy 47.625 66.04) (xy 50.8 66.04))
     (stroke (width 0) (type default))
@@
     (stroke (width 0) (type default))
   )
+  (wire (pts (xy 212.09 65.405) (xy 212.09 67.31))
+    (stroke (width 0) (type default))
+  )
+  (wire (pts (xy 214.63 65.405) (xy 214.63 67.31))
+    (stroke (width 0) (type default))
+  )
   (wire (pts (xy 16.51 189.23) (xy 16.51 186.69))
     (stroke (width 0) (type default))
   )
+  (wire (pts (xy 209.55 65.405) (xy 209.55 67.31))
+    (stroke (width 0) (type default))
+  )
+  (wire (pts (xy 214.63 67.31) (xy 212.09 67.31))
+    (stroke (width 0) (type default))
+  )
   (wire (pts (xy 17.78 171.45) (xy 16.51 171.45))
     (stroke (width 0) (type default))
@@
     (stroke (width 0) (type default))
   )
+  (wire (pts (xy 187.325 56.515) (xy 201.93 56.515))
+    (stroke (width 0) (type default))
+  )
+  (wire (pts (xy 209.55 67.31) (xy 209.55 68.58))
+    (stroke (width 0) (type default))
+  )
+  (wire (pts (xy 217.17 65.405) (xy 217.17 67.31))
+    (stroke (width 0) (type default))
+  )
   (wire (pts (xy 31.75 78.74) (xy 50.8 78.74))
+    (stroke (width 0) (type default))
+  )
+  (wire (pts (xy 217.17 67.31) (xy 214.63 67.31))
     (stroke (width 0) (type default))
   )
@@
     )
   )
+  (symbol (lib_id "rpi_s8x8hat:LPF") (at 222.25 70.485 0) (unit 1)
+    (in_bom yes) (on_board yes) (dnp no)
+    (property "Reference" "FL1" (at 224.79 52.8671 0)
+      (effects (font (size 1.27 1.27)))
+    )
+    (property "Value" "LPF" (at 224.79 61.595 0)
+      (effects (font (size 1.27 1.27)) hide)
+    )
+    (property "Footprint" "rpi_sa8x8hat:0500LP15A500" (at 217.17 31.115 0)
+      (effects (font (size 2.54 2.54)) hide)
+    )
+    (property "Datasheet" "" (at 217.17 31.115 0)
+      (effects (font (size 2.54 2.54)) hide)
+    )
+    (pin "8")
+    (pin "6")
+    (pin "5")
+    (pin "7")
+    (pin "2")
+    (pin "3")
+    (pin "4")
+    (pin "1")
+    (instances
+      (project "rpi_sa8x8hat"
+        (path "/2209fe87-8924-4afe-ae44-30084e3bc758"
+          (reference "FL1") (unit 1)
+        )
+      )
+    )
+  )
   (symbol (lib_id "Mechanical:MountingHole_Pad") (at 20.32 186.69 270) (unit 1)
     (in_bom yes) (on_board yes) (dnp no) (fields_autoplaced)
@@
         )
       )
+    )
+  )
+  (symbol (lib_id "power:GND") (at 209.55 68.58 0) (unit 1)
+    (in_bom yes) (on_board yes) (dnp no) (fields_autoplaced)
+    (property "Reference" "#PWR04" (at 209.55 74.93 0)
+      (effects (font (size 1.27 1.27)) hide)
+    )
+    (property "Value" "GND" (at 209.55 73.66 0)
+      (effects (font (size 1.27 1.27)))
+    )
+    (property "Footprint" "" (at 209.55 68.58 0)
+      (effects (font (size 1.27 1.27)) hide)
+    )
+    (property "Datasheet" "" (at 209.55 68.58 0)
+      (effects (font (size 1.27 1.27)) hide)
+    )
+    (pin "1")
+    (instances
+      (project "rpi_sa8x8hat"
+        (path "/2209fe87-8924-4afe-ae44-30084e3bc758"
+          (reference "#PWR04") (unit 1)
+        )
+      )
+    )
+  )
+  (symbol (lib_id "rpi_s8x8hat:SA818") (at 175.895 60.325 0) (unit 1)
+    (in_bom yes) (on_board yes) (dnp no) (fields_autoplaced)
+    (property "Reference" "U1" (at 175.26 76.2 0)
+      (effects (font (size 1.27 1.27)))
+    )
+    (property "Value" "SA818" (at 175.26 78.74 0)
+      (effects (font (size 1.27 1.27)))
+    )
+    (property "Footprint" "rpi_sa8x8hat:SA818" (at 175.895 40.005 0)
+      (effects (font (size 1.27 1.27)) hide)
+    )
+    (property "Datasheet" "" (at 175.895 40.005 0)
+      (effects (font (size 1.27 1.27)) hide)
+    )
+    (pin "1")
+    (pin "16")
+    (pin "17")
+    (pin "19")
+    (pin "7")
+    (pin "6")
+    (pin "5")
+    (pin "8")
+    (pin "3")
+    (pin "12")
+    (pin "18")
+    (pin "10")
+    (pin "9")
+    (instances
+      (project "rpi_sa8x8hat"
+        (path "/2209fe87-8924-4afe-ae44-30084e3bc758"
+          (reference "U1") (unit 1)
+        )
+      )

Commit message: wip
Parts:
- removed FL1: LPF, rpi_sa8x8hat:0500LP15A500, symbol rpi_s8x8hat:LPF
- added C1, C10, C11, C13, C14, C15, C7: 100n, symbol Device:C
- added C12, C2, C3, C4, C5, C6, C9: 10u, symbol Device:C
- added C8: 1u, symbol Device:C
- added JP1: SolderJumper_2_Open, Jumper:SolderJumper-2_P1.3mm_Open_TrianglePad1.0x1.5mm, symbol Jumper:SolderJumper_2_Open
- added R1, R13, R2, R4: 0, symbol Device:R
- added R10, R11, R12, R5, R6, R7, R8, R9: 10K, symbol Device:R
- added R3: 27, symbol Device:R
- added U2: TLV320AIC3204, Package_DFN_QFN:QFN-32-1EP_5x5mm_P0.5mm_EP3.7x3.7mm, symbol rpi_s8x8hat:TLV320AIC3204
- added U3: AT24CS32-STUM, Package_TO_SOT_SMD:SOT-23-5, symbol Memory_EEPROM:AT24CS32-STUM
Connections:
- net 5V is gone; now on net +5V: J1.2 (5V), J1.4 (5V)
- net BCM_I2S_IN: now also R3.1
- net BCM_I2S_OUT: now also R2.1
- net BCM_I2S_WCLK: now also R4.1
- net GND: now also U1.10 (GND), U1.9 (GND), C1.2, C10.2, C11.2, C12.2, C13.2, C14.2, C15.2, C2.2, C5.2, C6.2, C7.2, C8.2, C9.2, JP1.1 (A), R13.2, U2.12 (SPI_SELECT), U2.17 (AVss), U2.28 (DVss), U2.33 (PAD), U2.7 (IOVss), U3.2 (GND)
- net BCM_SDA: now reaches J1.3 (BCM2_SDA)
- net BCM_SDA: now also R8.2, U2.10 (SDA/MOSI)
- net BCM_GPIO13: now reaches J1.33 (BCM13_PWM1)
- net BCM_GPIO13: now also R10.2, U2.31 (~{RESET})
- net BCM_SCL: now reaches J1.5 (BCM3_SCL)
- net BCM_SCL: now also R9.2, U2.9 (SCL/~{SS})
- net BCM_CLK_25MHZ: now reaches J1.7 (BCM4_GPCLK0)
- net BCM_CLK_25MHZ: now also R1.1
- net at U1.6 (~{PD}): now also R11.2
- net at U1.7 (HI/~{LOW}): now also R12.2, R13.1
- net +5V: now reaches U1.8 (VBAT)
- net +5V: now also C12.1, C13.1, R11.1, R12.1
- net 3V3 renamed +3V3
- net +3V3: now also C1.1, C10.1, C7.1, C8.1, C9.1, R10.1, R5.1, R6.1, R7.1, R8.1, R9.1, U2.26 (LDOIN/HPVdd), U2.30 (DLDO_SELECT), U2.6 (IOVdd), U3.4 (VCC)
- net BCM_ID_SCL renamed BCM1_ID_SCL
- net BCM1_ID_SCL: now also R5.2, U3.1 (SCL)
- net BCM_ID_SDA renamed BCM1_ID_SDA
- net BCM1_ID_SDA: now also R6.2, U3.3 (SDA)
- new net: C14.1, C6.1, U2.29 (DVdd_OUT)
- new net: C3.1, U2.22 (LOL)
- new net: C4.1, U2.23 (LOR)
- new net: R1.2, U2.1 (MCLK)
- new net: C11.1, C2.1, U2.18 (REF)
- new net: C15.1, C5.1, U2.24 (AVdd_OUT)
- new net: R4.2, U2.3 (WCLK)
- new net: R2.2, U2.4 (DIN/MFP1)
- new net: R3.2, U2.5 (DOUT/MFP2)
- new net: JP1.2 (B), R7.2, U3.5 (WP)
- no-connect marks 0 -> 25
Other:
- note added: "HAT ID"
- note added: "Place near the source. Starting point: 10 for MCLK, 27 for others"
- note added: "TODO: Add filter"
- note added: "TODO: Add level translator"
- note added: "Whenever any of the analog input terminals IN1_L, IN2_L, IN3_L, IN1_R, IN2_R or IN3_R are not used in an application, it is recommended to short the unused input terminals together (if convenient) and connect them to ground using a small capacitor (example 0.1 µF)."
- note added: "Whenever any of the analog output terminals LOL, LOR, HPL or HPR are not used in an application, they should be left open or not connected."

Commit message: wip
Parts:
- removed R12: 10K, symbol Device:R
- removed R13: 0, symbol Device:R
- added FID1, FID2, FID3: Fiducial, symbol Mechanical:Fiducial
- added JP1: SolderJumper_2_Bridged, symbol Jumper:SolderJumper_2_Bridged
- added R1: 10K, symbol Device:R
- added U2: FILTER, symbol rpi_s8x8hat:FILTER-3TERM
- J1: symbol rpi_sa8x8hat:RPi_GPIO -> rpi_s8x8hat:RPi_GPIO
- U1: footprint rpi_sa8x8hat:SA818 -> (none)
- renumbered C12 to C1, C6 to C10, C2 to C11, C3 to C12, C4 to C13, C15 to C14, C5 to C15, C13 to C2, C1 to C3, C10 to C4, C9 to C5, C8 to C6, C11 to C8, C14 to C9, JP1 to JP2, R3 to R10, R4 to R11, R1 to R12, R11 to R2, R8 to R3, R9 to R4, R10 to R8, R2 to R9, U2 to U4
Connections:
- net +5V: now also R1.1
- net GND: now also JP1.1 (A), U2.3 (GND)
- net at U1.7 (~{LOWPWR}): now also JP1.2 (B)
- net at U1.12 (ANT): now also U2.1 (IN)
- net at U1.5 (~{TXEN}): now also R1.2
Other:
- note removed: "TODO: Add filter"
- company: (none) -> Murgatroid Heavy Industries, LLC
- title: (none) -> RPi SA818 Hat
- moved on the sheet: C1, C10, C11, C12, C13, C14, C15, C2, C4, C5, C6, C7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

Commit message: wip
Parts:
- FID1, FID2, FID3: footprint (none) -> Fiducial:Fiducial_0.5mm_Mask1.5mm
Changed lines of the file:
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@@
       (effects (font (size 1.27 1.27)) (justify left))
     )
-    (property "Footprint" "" (at 34.925 192.405 0)
+    (property "Footprint" "Fiducial:Fiducial_0.5mm_Mask1.5mm" (at 34.925 192.405 0)
       (effects (font (size 1.27 1.27)) hide)
     )
@@
       (effects (font (size 1.27 1.27)) (justify left))
     )
-    (property "Footprint" "" (at 24.13 192.405 0)
+    (property "Footprint" "Fiducial:Fiducial_0.5mm_Mask1.5mm" (at 24.13 192.405 0)
       (effects (font (size 1.27 1.27)) hide)
     )
@@
       (effects (font (size 1.27 1.27)) (justify left))
     )
-    (property "Footprint" "" (at 29.21 192.405 0)
-      (effects (font (size 1.27 1.27)) hide)
-    )
+    (property "Footprint" "Fiducial:Fiducial_0.5mm_Mask1.5mm" (at 29.21 192.405 0)
+      (effects (font (size 1.27 1.27)) hide)
+    )

Commit message: V8
Parts:
- J1: symbol rpi_s8x8hat:RPi_GPIO -> rpi_sa8x8hat:RPi_GPIO
- U1: symbol rpi_s8x8hat:SA818 -> rpi_sa8x8hat:SA818
- U2: symbol rpi_s8x8hat:FILTER-3TERM -> rpi_sa8x8hat:FILTER-3TERM
- U4: symbol rpi_s8x8hat:TLV320AIC3204 -> rpi_sa8x8hat:TLV320AIC3204

Commit message: wip
Parts:
- U1: footprint (none) -> rpi_sa8x8hat:SA8x8
Changed lines of the file:
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@@
 			)
 		)
-		(property "Footprint" ""
+		(property "Footprint" "rpi_sa8x8hat:SA8x8"
 			(at 62.23 134.62 0)
 			(effects
@@
 		(pin "4"
 		)
+		(pin "PAD"
+		)
 		(instances
