File: projects/impulse_pluggy/impulse_pluggy.kicad_sch (KiCad schematic)
At the start: 14 parts, among them J1 Conn_01x02_Socket, J10 DNP, J11 DNP, J2 Conn_01x02_Socket, J3 Conn_01x02_Socket, J4 Conn_01x02_Socket, J5 Conn_01x02_Socket, J6 Conn_01x02_Socket, J7 Conn_01x05_Socket

Commit message: wip
Parts:
- removed J10: DNP, Connector_PinHeader_2.54mm:PinHeader_1x02_P2.54mm_Vertical, symbol Connector:Conn_01x02_Pin
- added JP1: SolderJumper_2_Open, Jumper:SolderJumper-2_P1.3mm_Open_TrianglePad1.0x1.5mm, symbol Jumper:SolderJumper_2_Open
- J6: value Conn_01x02_Socket -> DNP
- J7: value Conn_01x05_Socket -> DNP
Connections:
- net WD_1: now also JP1.2 (B)
- net WD_2: now also JP1.1 (A)
Other:
- moved on the sheet: J1, J11, J2, J3, J4, J5, J6, J7, R1, R2, R3, R4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

Commit message: wip
Parts:
- J1, J2, J3, J4, J5: footprint Connector_PinSocket_2.54mm:PinSocket_1x02_P2.54mm_Vertical -> Connector_PinSocket_2.54mm:PinSocket_1x02_P2.54mm_Vertical_SMD_Pin1Left
- J11: value DNP -> Conn_01x06_Pin; now not fitted
- J6: value DNP -> Conn_01x02_Socket; footprint Connector_PinSocket_2.54mm:PinSocket_1x02_P2.54mm_Vertical -> Connector_PinSocket_2.54mm:PinSocket_1x02_P2.54mm_Vertical_SMD_Pin1Left; now not fitted
- J7: value DNP -> Conn_01x06_Socket; footprint Connector_PinSocket_2.54mm:PinSocket_1x06_P2.54mm_Vertical -> Connector_PinSocket_2.54mm:PinSocket_1x06_P2.54mm_Vertical_SMD_Pin1Left; now not fitted
Changed lines of the file:
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@@
 		(in_bom yes)
 		(on_board yes)
-		(dnp no)
+		(dnp yes)
 		(property "Reference" "J6"
 			(at 66.04 82.804 0)
@@
 			)
 		)
-		(property "Value" "DNP"
-			(at 65.278 85.09 0)
-			(effects
-				(font
-					(size 1.27 1.27)
-				)
-			)
-		)
-		(property "Footprint" "Connector_PinSocket_2.54mm:PinSocket_1x02_P2.54mm_Vertical"
+		(property "Value" "Conn_01x02_Socket"
+			(at 57.912 84.836 0)
+			(effects
+				(font
+					(size 1.27 1.27)
+				)
+			)
+		)
+		(property "Footprint" "Connector_PinSocket_2.54mm:PinSocket_1x02_P2.54mm_Vertical_SMD_Pin1Left"
 			(at 68.58 82.55 0)
 			(effects
@@
 			)
 		)
-		(property "Footprint" "Connector_PinSocket_2.54mm:PinSocket_1x02_P2.54mm_Vertical"
+		(property "Footprint" "Connector_PinSocket_2.54mm:PinSocket_1x02_P2.54mm_Vertical_SMD_Pin1Left"
 			(at 68.58 71.12 0)
 			(effects
@@
 			)
 		)
-		(property "Footprint" "Connector_PinSocket_2.54mm:PinSocket_1x02_P2.54mm_Vertical"
+		(property "Footprint" "Connector_PinSocket_2.54mm:PinSocket_1x02_P2.54mm_Vertical_SMD_Pin1Left"
 			(at 68.58 58.42 0)
 			(effects
@@
 		(in_bom yes)
 		(on_board yes)
-		(dnp no)
+		(dnp yes)
 		(property "Reference" "J11"
 			(at 133.35 93.98 0)
@@
 			)
 		)
-		(property "Value" "DNP"
-			(at 133.35 96.52 0)
+		(property "Value" "Conn_01x06_Pin"
+			(at 138.938 96.52 0)
 			(effects
 				(font
@@
 			)
 		)
-		(property "Footprint" "Connector_PinSocket_2.54mm:PinSocket_1x02_P2.54mm_Vertical"
+		(property "Footprint" "Connector_PinSocket_2.54mm:PinSocket_1x02_P2.54mm_Vertical_SMD_Pin1Left"
 			(at 68.58 64.77 0)
 			(effects
@@
 		(in_bom yes)
 		(on_board yes)
-		(dnp no)
+		(dnp yes)
 		(property "Reference" "J7"
 			(at 67.056 95.25 0)
@@
 			)
 		)
-		(property "Value" "DNP"
+		(property "Value" "Conn_01x06_Socket"
 			(at 67.31 97.79 0)
 			(effects
@@
 			)
 		)
-		(property "Footprint" "Connector_PinSocket_2.54mm:PinSocket_1x06_P2.54mm_Vertical"
+		(property "Footprint" "Connector_PinSocket_2.54mm:PinSocket_1x06_P2.54mm_Vertical_SMD_Pin1Left"
 			(at 68.58 96.52 0)
 			(effects
@@
 			)
 		)
-		(property "Footprint" "Connector_PinSocket_2.54mm:PinSocket_1x02_P2.54mm_Vertical"
+		(property "Footprint" "Connector_PinSocket_2.54mm:PinSocket_1x02_P2.54mm_Vertical_SMD_Pin1Left"
 			(at 68.58 49.53 0)
 			(effects
@@
 			)
 		)
-		(property "Footprint" "Connector_PinSocket_2.54mm:PinSocket_1x02_P2.54mm_Vertical"
+		(property "Footprint" "Connector_PinSocket_2.54mm:PinSocket_1x02_P2.54mm_Vertical_SMD_Pin1Left"
 			(at 68.58 43.18 0)
 			(effects

Commit message: checkpoint
Parts:
- removed J11: Conn_01x06_Pin, Connector_PinHeader_2.54mm:PinHeader_1x06_P2.54mm_Vertical, symbol Connector:Conn_01x06_Pin
- removed JP1: SolderJumper_2_Open, Jumper:SolderJumper-2_P1.3mm_Open_TrianglePad1.0x1.5mm, symbol Jumper:SolderJumper_2_Open
- J1, J2, J3, J4, J5: footprint Connector_PinSocket_2.54mm:PinSocket_1x02_P2.54mm_Vertical_SMD_Pin1Left -> impulse_pluggy:SAMTEC_SSM-102-L-SV-BE
- J6: footprint Connector_PinSocket_2.54mm:PinSocket_1x02_P2.54mm_Vertical_SMD_Pin1Left -> impulse_pluggy:SAMTEC_SSM-102-L-SV-BE; now fitted
- J7: footprint Connector_PinSocket_2.54mm:PinSocket_1x06_P2.54mm_Vertical_SMD_Pin1Left -> impulse_pluggy:SAMTEC_SSM-106-L-SV-BE; now fitted
Connections:
- net CAN_H_1: now also R1.2; no longer R1.1
- net CAN_H_2: now also R1.1; no longer R1.2
- net CAN_L_1: now also R2.2; no longer R2.1
- net CAN_L_2: now also R2.1; no longer R2.2
- net ID_0_1: now also R3.2; no longer R3.1
- net ID_0_2: now also R3.1; no longer R3.2
- net ID_1_1: now also R4.2; no longer R4.1
- net ID_1_2: now also R4.1; no longer R4.2
- net ID_2_1: now also R5.2; no longer R5.1
- net ID_2_2: now also R5.1; no longer R5.2
- no-connect marks 0 -> 8
Other:
- moved on the sheet: R1, R2, R3, R4, R5
