File: projects/impulse_powercal/impulse_powercal.kicad_pcb (KiCad board)
At the start: 2 copper layers, 40 x 44.2 mm, 12 parts, among them J1 Conn_Coaxial, J2 Conn_01x02_Pin, J3 Conn_01x01_Pin, J4 Conn_01x01_Pin

Commit message: .
Parts:
- added C1: DNP, Capacitor_SMD:C_0805_2012Metric_Pad1.18x1.45mm_HandSolder, F.Cu at (111.5, 106.8)
- added J5: DC37_Plug, Connector_Dsub:DSUB-37_Male_Horizontal_P2.77x2.54mm_EdgePinOffset9.40mm, F.Cu at (124.9, 71.5)
- added R5: 100K, Resistor_SMD:R_1206_3216Metric_Pad1.30x1.75mm_HandSolder, F.Cu at (94.8, 76.0)
- added R6: DNP, Resistor_SMD:R_1206_3216Metric_Pad1.30x1.75mm_HandSolder, F.Cu at (112.0, 109.8)
- added R7: 0, Resistor_SMD:R_1206_3216Metric_Pad1.30x1.75mm_HandSolder, F.Cu at (96.3, 82.8)
- added R8: 0, Resistor_SMD:R_1206_3216Metric_Pad1.30x1.75mm_HandSolder, F.Cu at (96.2, 80.2)
- added R9: 0, Resistor_SMD:R_1206_3216Metric_Pad1.30x1.75mm_HandSolder, F.Cu at (105.8, 76.0)
- moved J1 27.6 mm to (126.9, 86.4), turned to -90 degrees
- moved H1 21.5 mm to (65.0, 65.0)
- moved H3 21.5 mm to (135.0, 65.0)
- moved H2 20.0 mm to (65.0, 108.5)
- moved H4 20.0 mm to (135.0, 108.5)
Connections:
- net /HI renamed /HEAT_P
- net /LO renamed /HEAT_N
Routing:
- net /AIN0/1_P: track 0.00 -> 27.1 mm
- net /AIN0/1_N: track 0.00 -> 26.8 mm
- net /HEAT_P: track 41.4 -> 67.5 mm, vias 0 -> 2
- net /HEAT_N: track 42.4 -> 67.2 mm, vias 0 -> 2
- net GND: vias 0 -> 9
- added copper zone on B.Cu, net GND
- added copper zone on F.Cu, net GND
- added copper zone on F.Cu, net GNDJ
- removed copper zone on B.Cu, net (none)
Other:
- board size 40 x 44.2 mm -> 80 x 53.5 mm

Commit message: ..
Parts:
- removed R9: 0, Resistor_SMD:R_1206_3216Metric_Pad1.30x1.75mm_HandSolder
- moved R5 2.30 mm to (96.2, 77.8), turned to 0 degrees
Connections:
- J5 pad 1: GNDJ -> GND
- J5 pad 10: GNDJ -> GND
- J5 pad 19: GNDJ -> GND
- J5 pad 30: GNDJ -> GND
- J5 pad 8: GNDJ -> GND
- R5 pad 2: GNDJ -> GND
Routing:
- net GND: track 0.00 -> 1.20 mm, vias 9 -> 7
- removed copper zone on F.Cu, net GNDJ
Other:
- board text added: "H+"
- board text added: "H-"
- board text added: "Impulse Labs HEB Power Cal v1.0 ch@"
- board text removed: "HI"
- board text removed: "Impulse HEB Power Cal v1.0"
- board text removed: "LO"

Commit message: .
Parts:
- J5: value DC37_Plug -> 7472524-SINGLE; footprint Connector_Dsub:DSUB-37_Male_Horizontal_P2.77x2.54mm_EdgePinOffset9.40mm -> impulse_powercal:7472524
- moved J5 27.4 mm to (100.0, 60.1)
- moved H1 5.00 mm to (60.0, 108.5)
- moved H2 5.00 mm to (60.0, 65.0)
- moved H3 4.75 mm to (139.8, 108.5)
- moved H4 4.75 mm to (139.8, 65.0)
- moved J4 4.25 mm to (131.2, 86.4)
- renumbered H2 to H1, H1 to H2, H4 to H3, H3 to H4, J4 to J1, J1 to J4, R6 to R5, R5 to R6, R8 to R7, R7 to R8
Routing:
- net /HEAT_P: track 67.5 -> 71.8 mm
- net /HEAT_N: track 67.2 -> 71.4 mm
- net /AIN0/1_P: track 27.1 -> 28.5 mm
- net /AIN0/1_N: track 26.6 -> 27.7 mm
Other:
- board size 80 x 53.5 mm -> 89.8 x 53.5 mm

Commit message: ship it
Other:
- board text added: "DATAMATRIX CODE DATAMATRIX CODE DATAMATRIX CODE DATAMATRIX CODE DATAMATRIX CODE ########"
Changed lines of the file:
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@@
 		(tags "Connector")
 		(property "Reference" "J5"
-			(at -33.5 -14.35 360)
+			(at -33.5 -14.35 0)
 			(layer "F.SilkS")
 			(effects
@@
 		)
 		(property "Value" "7472524-SINGLE"
-			(at 0 -3.56 360)
+			(at 0 -3.56 0)
 			(layer "F.SilkS")
 			(hide yes)
@@
 		)
 		(property "Footprint" "impulse_powercal:7472524"
-			(at 0 0 360)
+			(at 0 0 0)
 			(layer "F.Fab")
 			(hide yes)
@@
 		)
 		(property "Datasheet" ""
-			(at 0 0 360)
+			(at 0 0 0)
 			(layer "F.Fab")
 			(hide yes)
@@
 		)
 		(property "Description" "37-pin male plug pin D-SUB connector, Mounting Hole"
-			(at 0 0 360)
+			(at 0 0 0)
 			(layer "F.Fab")
 			(hide yes)
@@
 		)
 		(fp_text user "${REFERENCE}"
-			(at 0 -3.56 360)
+			(at 0 -3.56 0)
 			(layer "F.Fab")
 			(effects
@@
 	)
 	(gr_rect
-		(start 57.075 87.2)
-		(end 82.5 97.5)
+		(start 64.2875 102.25)
+		(end 89.7125 112.05)
 		(stroke
 			(width 0.1)
@@
 	)
 	(gr_line
+		(start 70 85)
+		(end 70 97.5)
+		(stroke
+			(width 0.1)
+			(type default)
+		)
+		(layer "Dwgs.User")
+	)
+	(gr_line
 		(start 55 108.5)
 		(end 158.5 108.5)
@@
 	)
 	(gr_line
+		(start 70 97.5)
+		(end 57.5 97.5)
+		(stroke
+			(width 0.1)
+			(type default)
+		)
+		(layer "Dwgs.User")
+	)
+	(gr_line
+		(start 57.5 97.5)
+		(end 57.5 85)
+		(stroke
+			(width 0.1)
+			(type default)
+		)
+		(layer "Dwgs.User")
+	)
+	(gr_line
+		(start 57.5 85)
+		(end 70 85)
+		(stroke
+			(width 0.1)
+			(type default)
+		)
+		(layer "Dwgs.User")
+	)
+	(gr_line
 		(start 139.75 60)
 		(end 60 60)
@@
 	)
 	(gr_text "Impulse Labs\nHEB Power Cal\nv1.0 ch@"
-		(at 56.75 85 0)
+		(at 57 83.5 0)
 		(layer "F.SilkS")
 		(effects
@@
 			)
 			(justify left bottom)
+		)
+	)
+	(gr_text "DATAMATRIX CODE\nDATAMATRIX CODE\nDATAMATRIX CODE\nDATAMATRIX CODE\nDATAMATRIX CODE\n########"
+		(at 57.75 94.75 0)
+		(layer "Dwgs.User")
+		(effects
+			(font
+				(size 0.9 0.9)
+				(thickness 0.15)
+			)
+			(justify left bottom)

Commit message: V1.1
Parts:
- removed C1: DNP, Capacitor_SMD:C_0805_2012Metric_Pad1.18x1.45mm_HandSolder
- added J6: Screw_Terminal_01x02, TerminalBlock_Phoenix:TerminalBlock_Phoenix_MPT-0,5-2-2.54_1x02_P2.54mm_Horizontal, F.Cu at (119.8, 109.8)
- J2: value Conn_01x02_Pin -> Screw_Terminal_01x02; footprint Connector_Wire:SolderWire-0.5sqmm_1x02_P4.6mm_D0.9mm_OD2.1mm -> TerminalBlock_Phoenix:TerminalBlock_Phoenix_MPT-0,5-2-2.54_1x02_P2.54mm_Horizontal
- R7: renamed from R5; value DNP -> 0
- moved R2 1.25 mm to (100.0, 88.8)
- moved R3 1.25 mm to (100.0, 93.8)
- moved R4 1.25 mm to (100.0, 98.8)
- moved R5 1.25 mm to (100.0, 103.8)
- moved J1 1.21 mm to (92.3, 96.3)
- moved J4 1.20 mm to (107.7, 96.3)
- moved J2 1.04 mm to (98.7, 109.8)
- moved R7 0.55 mm to (112.0, 109.2)
- renumbered H3 to H2, H2 to H3, J3 to J1, J4 to J3, J1 to J4, R8 to R1, R1 to R2, R2 to R3, R3 to R4, R4 to R5, R7 to R6, R6 to R8
Routing:
- net /HEAT_N: track 71.4 -> 70.2 mm
- net /HEAT_P: track 71.8 -> 70.6 mm
- net GND: vias 7 -> 6
Other:
- board text added: "..REPLACE WITH.. DATAMATRIX CODE DATAMATRIX CODE DATAMATRIX CODE DATAMATRIX CODE DATAMATRIX CODE ###SERIALNO###"
- board text added: "GND"
- board text added: "Impulse Labs HEB Power Cal v1.1 ch@"
- board text removed: "DATAMATRIX CODE DATAMATRIX CODE DATAMATRIX CODE DATAMATRIX CODE DATAMATRIX CODE ########"
- board text removed: "Impulse Labs HEB Power Cal v1.0 ch@"

Commit message: wip to v2
Parts:
- added C1: C, Capacitor_SMD:C_0603_1608Metric_Pad1.08x0.95mm_HandSolder, F.Cu at (85.1, 82.4)
- added C2: C, Capacitor_SMD:C_0603_1608Metric_Pad1.08x0.95mm_HandSolder, F.Cu at (85.1, 79.0)
- added C3: C, Capacitor_SMD:C_0603_1608Metric_Pad1.08x0.95mm_HandSolder, F.Cu at (83.5, 80.7)
- added J7: 5054481071, impulse_powercal:MOLEX_5054481071, F.Cu at (138.0, 95.3)
- added J8: Screw_Terminal_01x02, TerminalBlock_RND:TerminalBlock_RND_205-00287_1x02_P5.08mm_Horizontal, F.Cu at (138.7, 85.4)
- added J9: Conn_Coaxial, Connector_Coaxial:SMA_Amphenol_901-144_Vertical, F.Cu at (61.3, 92.4)
- added R10: 100K, Resistor_SMD:R_0805_2012Metric_Pad1.20x1.40mm_HandSolder, F.Cu at (87.8, 83.7)
- added R11: 0, Resistor_SMD:R_0805_2012Metric_Pad1.20x1.40mm_HandSolder, F.Cu at (130.4, 85.4)
- added R9: R, Resistor_SMD:R_0805_2012Metric_Pad1.20x1.40mm_HandSolder, F.Cu at (130.3, 100.4)
- J3: footprint Connector_Coaxial:BNC_Amphenol_B6252HB-NPP3G-50_Horizontal -> Connector_Coaxial:SMA_Amphenol_901-144_Vertical
- R1, R6, R8: footprint Resistor_SMD:R_1206_3216Metric_Pad1.30x1.75mm_HandSolder -> Resistor_SMD:R_0805_2012Metric_Pad1.20x1.40mm_HandSolder
- R7: value 0 -> R; footprint Resistor_SMD:R_1206_3216Metric_Pad1.30x1.75mm_HandSolder -> Resistor_SMD:R_0805_2012Metric_Pad1.20x1.40mm_HandSolder
- moved J3 55.6 mm to (75.9, 92.4), turned to 0 degrees
- moved R7 22.1 mm to (130.3, 96.8), turned to 180 degrees
- moved R1 8.56 mm to (87.8, 81.7)
- moved R6 8.47 mm to (87.8, 79.7)
- moved R8 8.45 mm to (87.8, 77.7)
Connections:
- R7 pad 1: /HEAT_N -> /12V_SHIELD
Routing:
- net /AIN2/3_P: track 0.00 -> 57.4 mm
- net /AIN0/1_P: track 28.5 -> 47.7 mm
- net +VDC: track 0.00 -> 17.0 mm
- net /AIN0/1_N: track 27.7 -> 42.9 mm, vias 0 -> 2
- net /SHIELD: track 0.00 -> 15.1 mm, vias 0 -> 2
- net GND: track 1.20 -> 6.28 mm, vias 6 -> 24
- net /12V_SHIELD: track 0.00 -> 4.01 mm
- net /HEAT_N: track 70.2 -> 68.9 mm, vias 2 -> 4
- added copper zone on F.Cu, net +VDC
- added copper zone on F.Cu, net /AIN0/1_N
Other:
- board text added: "Impulse Labs HEB Power Cal v1.2 ch@"
- board text removed: "Impulse Labs HEB Power Cal v1.1 ch@"

Commit message: v1.2
Parts:
- added J8: Screw_Terminal_01x02, TerminalBlock_Phoenix:TerminalBlock_Phoenix_MPT-0,5-2-2.54_1x02_P2.54mm_Horizontal, F.Cu at (129.9, 109.9)
- C1: renamed from C3; value C -> 500n
- C2: renamed from C1; value C -> 1u
- C3: renamed from C2; value C -> 1u
- J1: renamed from J9; footprint Connector_Coaxial:SMA_Amphenol_901-144_Vertical -> Connector_Coaxial:SMA_Amphenol_132291-12_Vertical
- J10: renamed from J8; footprint TerminalBlock_RND:TerminalBlock_RND_205-00287_1x02_P5.08mm_Horizontal -> TerminalBlock_Phoenix:TerminalBlock_Phoenix_MKDS-3-2-5.08_1x02_P5.08mm_Horizontal
- J2: renamed from J3; footprint Connector_Coaxial:SMA_Amphenol_901-144_Vertical -> Connector_Coaxial:SMA_Amphenol_132291-12_Vertical
- R2: renamed from R1; value 0 -> 2000
- R3: renamed from R6; value 0 -> 1u
- moved J10 1.45 mm to (138.9, 83.9)
- moved R11 1.44 mm to (130.5, 84.0)
- moved J9 1.17 mm to (138.6, 96.3)
- moved R9 1.17 mm to (130.9, 101.4)
- moved R10 0.92 mm to (130.9, 97.5)
- moved J7 0.05 mm to (119.8, 109.9)
- moved J4 0.05 mm to (98.7, 109.9)
- renumbered H3 to H2, H2 to H3, J1 to J3, J2 to J4, J4 to J6, J6 to J7, J7 to J9, R10 to R1, R7 to R10, R8 to R4, R4 to R6, R3 to R7, R2 to R8
Routing:
- net +VDC: track 17.0 -> 48.9 mm
- net /AIN2/3_P: track 57.4 -> 61.1 mm
- net /SHIELD: track 15.1 -> 12.0 mm
- net /12V_SHIELD: track 4.01 -> 2.96 mm
- net GND: vias 24 -> 25
- added copper zone on B.Cu, net /AIN0/1_N
- added copper zone on B.Cu, net /HEAT_N
- removed copper zone on F.Cu, net /AIN0/1_N
Other:
- board text added: "GND V+"
- board text added: "dV"
- board text added: "lpf(dV)"

Commit message: update
Parts:
- R10: value R -> 0
- R3: value 1u -> 2000
Changed lines of the file:
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@@
 		)
 		(property "Value" "Screw_Terminal_01x02"
-			(at 1.27 4.16 360)
+			(at 1.27 4.16 0)
 			(layer "F.Fab")
 			(effects
@@
 		)
 		(fp_text user "${REFERENCE}"
-			(at 1.27 2 360)
+			(at 1.27 2 0)
 			(layer "F.Fab")
 			(effects
@@
 			)
 		)
-		(property "Value" "R"
+		(property "Value" "0"
 			(at 0 1.65 0)
 			(layer "F.Fab")
@@
 			)
 		)
-		(property "Value" "1u"
+		(property "Value" "2000"
 			(at 0 1.65 180)
 			(layer "F.Fab")
