File: projects/impulse_drvbo/impulse_drvbo.kicad_pcb (KiCad board)
At the start: 2 copper layers, 89.8 x 53.5 mm, 5 parts, among them J5 7472524-SINGLE

Commit message: wip
Parts:
- added C1: C, Capacitor_SMD:C_0603_1608Metric_Pad1.08x0.95mm_HandSolder, F.Cu at (83.5, 78.5)
- added C2: C, Capacitor_SMD:C_0603_1608Metric_Pad1.08x0.95mm_HandSolder, F.Cu at (83.5, 82.5)
- added C3: C, Capacitor_SMD:C_0603_1608Metric_Pad1.08x0.95mm_HandSolder, F.Cu at (81.5, 80.5)
- added C4: C, Capacitor_SMD:C_0603_1608Metric_Pad1.08x0.95mm_HandSolder, F.Cu at (96.0, 77.5)
- added C5: C, Capacitor_SMD:C_0603_1608Metric_Pad1.08x0.95mm_HandSolder, F.Cu at (104.0, 77.5)
- added C6: C, Capacitor_SMD:C_0603_1608Metric_Pad1.08x0.95mm_HandSolder, F.Cu at (112.5, 77.5)
- added C7: C, Capacitor_SMD:C_0603_1608Metric_Pad1.08x0.95mm_HandSolder, F.Cu at (121.0, 77.5)
- added J1: 5054481671, impulse_drvbo:MOLEX_5054481671, F.Cu at (62.7, 88.1)
- added J10: Conn_Coaxial, Connector_Coaxial:SMA_Amphenol_132291-12_Vertical, F.Cu at (128.0, 106.5)
- added J2: 5054481671, impulse_drvbo:MOLEX_5054481671, F.Cu at (137.5, 88.0)
- added J3: Conn_Coaxial, Connector_Coaxial:SMA_Amphenol_132291-12_Vertical, F.Cu at (73.0, 106.5)
- added J4: Conn_Coaxial, Connector_Coaxial:SMA_Amphenol_132291-12_Vertical, F.Cu at (82.5, 106.5)
- added J6: Conn_Coaxial, Connector_Coaxial:SMA_Amphenol_132291-12_Vertical, F.Cu at (92.0, 106.5)
- added J7: Conn_Coaxial, Connector_Coaxial:SMA_Amphenol_132291-12_Vertical, F.Cu at (101.0, 106.5)
- added J8: Conn_Coaxial, Connector_Coaxial:SMA_Amphenol_132291-12_Vertical, F.Cu at (110.0, 106.5)
- added J9: Conn_Coaxial, Connector_Coaxial:SMA_Amphenol_132291-12_Vertical, F.Cu at (119.0, 106.5)
- added R1: 0, Resistor_SMD:R_0805_2012Metric_Pad1.20x1.40mm_HandSolder, F.Cu at (86.5, 79.0)
- added R2: 0, Resistor_SMD:R_0805_2012Metric_Pad1.20x1.40mm_HandSolder, F.Cu at (86.5, 82.0)
- added R3: 100K, Resistor_SMD:R_0805_2012Metric_Pad1.20x1.40mm_HandSolder, F.Cu at (86.5, 76.5)
- added R4: 100K, Resistor_SMD:R_0805_2012Metric_Pad1.20x1.40mm_HandSolder, F.Cu at (86.5, 84.5)
- added R5: 0, Resistor_SMD:R_0805_2012Metric_Pad1.20x1.40mm_HandSolder, F.Cu at (99.0, 76.5)
- added R6: 0, Resistor_SMD:R_0805_2012Metric_Pad1.20x1.40mm_HandSolder, F.Cu at (107.0, 76.5)
- added R7: 0, Resistor_SMD:R_0805_2012Metric_Pad1.20x1.40mm_HandSolder, F.Cu at (115.5, 76.5)
- added R8: 0, Resistor_SMD:R_0805_2012Metric_Pad1.20x1.40mm_HandSolder, F.Cu at (124.0, 76.5)
Other:
- copper layers 2 -> 4

Commit message: wip
Parts:
- moved J10 69.4 mm to (121.0, 37.5)
- moved J3 69.4 mm to (66.0, 37.5)
- moved J4 69.4 mm to (75.5, 37.5)
- moved J6 69.4 mm to (85.0, 37.5)
- moved J7 69.4 mm to (94.0, 37.5)
- moved J8 69.4 mm to (103.0, 37.5)
- moved J9 69.4 mm to (112.0, 37.5)
- moved J2 44.1 mm to (97.0, 105.5), turned to 0 degrees
- moved J1 23.8 mm to (79.0, 105.5), turned to 0 degrees
Routing:
- net /I_AC_COIL: track 0.00 -> 24.7 mm, vias 0 -> 2
- net /3V3: track 0.00 -> 24.2 mm, vias 0 -> 2
- net /SHIELD: track 0.00 -> 23.0 mm, vias 0 -> 2
- net /HS_NTC_1: track 0.00 -> 22.9 mm, vias 0 -> 3
- net /PWM_A_L: track 0.00 -> 22.8 mm, vias 0 -> 2
- net /PWM_B_L: track 0.00 -> 22.6 mm, vias 0 -> 2
- net /~{GATE_DRIVER_ENABLE}: track 0.00 -> 22.2 mm, vias 0 -> 2
- net /V_DC_BUS_P: track 0.00 -> 22.2 mm, vias 0 -> 2
- net /V_DC_BUS_N: track 0.00 -> 21.9 mm, vias 0 -> 2
- net /HS_NTC_2: track 0.00 -> 21.8 mm, vias 0 -> 2
- net GND: track 0.00 -> 11.7 mm, vias 0 -> 8
- net /PWM_B_H: track 0.00 -> 3.65 mm, vias 0 -> 2
- net /PWM_A_H: track 0.00 -> 3.65 mm, vias 0 -> 2
- net /5V0: track 0.00 -> 3.65 mm, vias 0 -> 2
- net /I_DC_BUS: track 0.00 -> 3.25 mm, vias 0 -> 2

Commit message: wip
Routing:
- net /5V0: track 3.65 -> 29.4 mm, vias 2 -> 4
- net /PWM_A_H: track 3.65 -> 25.1 mm
- net /PWM_B_H: track 3.65 -> 24.0 mm
- net /I_DC_BUS: track 3.25 -> 21.8 mm
- net GND: track 11.7 -> 8.75 mm
- net /3V3: track 24.2 -> 26.7 mm, vias 2 -> 4
- net /HS_NTC_1: vias 3 -> 2

Commit message: wip
Parts:
- moved J10 79.3 mm to (127.5, 116.5)
- moved J3 79.3 mm to (72.5, 116.5)
- moved J4 79.3 mm to (82.0, 116.5)
- moved J6 79.3 mm to (91.5, 116.5)
- moved J7 79.3 mm to (100.5, 116.5)
- moved J8 79.3 mm to (109.5, 116.5)
- moved J9 79.3 mm to (118.5, 116.5)
- moved J2 42.9 mm to (138.0, 93.0), turned to 90 degrees
- moved J1 21.1 mm to (62.0, 93.0), turned to -90 degrees
- moved H3 13.5 mm to (140.0, 122.0)
- moved H1 13.5 mm to (60.0, 122.0)
- moved H4 0.25 mm to (140.0, 65.0)
Connections:
- J6 pad 1: /I_DC_COIL -> /I_DC_BUS
- R6 pad 1: /I_DC_COIL -> /I_DC_BUS
Routing:
- net /V_DC_BUS_N: track 21.9 -> 140.2 mm, vias 2 -> 6
- net /I_DC_BUS: track 21.8 -> 139.4 mm, vias 2 -> 4
- net /I_AC_COIL: track 24.7 -> 129.1 mm, vias 2 -> 5
- net /HS_NTC_2: track 21.8 -> 126.1 mm, vias 2 -> 4
- net /V_DC_BUS_P: track 22.6 -> 122.4 mm, vias 2 -> 5
- net /PWM_B_L: track 22.6 -> 115.6 mm, vias 2 -> 4
- net /PWM_A_L: track 22.8 -> 115.6 mm, vias 2 -> 4
- net /PWM_A_H: track 25.1 -> 109.6 mm
- net /SHIELD: track 23.0 -> 101.2 mm, vias 2 -> 4
- net /HS_NTC_1: track 22.9 -> 98.3 mm, vias 2 -> 4
- net /PWM_B_H: track 24.0 -> 98.2 mm, vias 2 -> 4
- net /~{GATE_DRIVER_ENABLE}: track 22.2 -> 78.3 mm, vias 2 -> 4
- net /3V3: track 26.7 -> 71.5 mm
- net /5V0: track 29.4 -> 71.0 mm
- net /AIN8/9_P: track 0.00 -> 40.6 mm, vias 0 -> 1
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- added copper zone on B.Cu, net /V_DC_BUS_N
- added copper zone on F.Cu, net GND
Other:
- board size 89.8 x 53.5 mm -> 90 x 67 mm

Commit message: wip
Parts:
- added C8: C, Capacitor_SMD:C_0603_1608Metric_Pad1.08x0.95mm_HandSolder, F.Cu at (141.9, 105.0)
- added FID1: Fiducial, Fiducial:Fiducial_0.5mm_Mask1mm, B.Cu at (60.5, 79.0)
- added FID2: Fiducial, Fiducial:Fiducial_0.5mm_Mask1mm, B.Cu at (127.5, 122.0)
- added FID3: Fiducial, Fiducial:Fiducial_0.5mm_Mask1mm, F.Cu at (59.5, 74.0)
- added FID4: Fiducial, Fiducial:Fiducial_0.5mm_Mask1mm, F.Cu at (123.0, 124.0)
- added R9: 0, Resistor_SMD:R_0805_2012Metric_Pad1.20x1.40mm_HandSolder, F.Cu at (142.0, 103.0)
- moved R3 14.8 mm to (73.8, 84.0), turned to -90 degrees
- moved R8 13.8 mm to (111.0, 81.2)
- moved R7 13.4 mm to (103.0, 81.2)
- moved R5 12.9 mm to (87.0, 81.2)
- moved R6 12.9 mm to (95.0, 81.2)
- moved R1 11.9 mm to (75.8, 84.0), turned to 90 degrees
- moved J10 10.8 mm to (137.5, 112.5)
- moved J3 10.7 mm to (62.5, 112.5)
- moved C7 10.4 mm to (110.8, 79.2), turned to 0 degrees
- moved C6 9.91 mm to (102.8, 79.2), turned to 0 degrees
- moved C4 9.41 mm to (86.8, 79.2), turned to 0 degrees
- moved C5 9.41 mm to (94.8, 79.2), turned to 0 degrees
- moved C1 8.62 mm to (75.2, 81.0), turned to 180 degrees
- moved R2 8.49 mm to (78.2, 84.0), turned to 90 degrees
- moved J4 8.06 mm to (75.0, 112.5)
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Routing:
- net /I_AC_COIL: track 129.1 -> 99.6 mm
- net /PWM_A_H: track 109.6 -> 89.4 mm, vias 2 -> 3
- net /HS_NTC_1: track 98.3 -> 84.3 mm, vias 4 -> 5
- net /AIN6/7_P: track 35.1 -> 23.9 mm
- net /AIN8/9_P: track 40.6 -> 29.4 mm, vias 1 -> 0
- net /SHIELD: track 101.2 -> 111.1 mm
- net /I_DC_BUS: track 139.4 -> 129.8 mm
- net /PWM_B_L: track 115.6 -> 108.0 mm, vias 4 -> 5
- net /AIN4/5_P: track 27.0 -> 19.7 mm
- net /PWM_B_H: track 98.2 -> 93.1 mm, vias 4 -> 5
- net /AIN2/3_P: track 22.2 -> 17.4 mm
- net /HS_NTC_2: track 126.1 -> 122.0 mm
- net /PWM_A_L: track 115.6 -> 111.7 mm
- net /AIN0/1_N: track 18.4 -> 15.4 mm
- net /V_DC_BUS_N: track 140.2 -> 137.5 mm
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Other:
- board text added: "DATAMATRIX CODE DATAMATRIX CODE DATAMATRIX CODE DATAMATRIX CODE DATAMATRIX CODE DATAMATRIX CODE ###SERNUM##"
- board text added: "HS_NTC_1 AIN6"
- board text added: "HS_NTC_1 AIN8"
- board text added: "I_AC_COIL"
- board text added: "I_AC_COIL AIN2"
- board text added: "I_DC_BUS"
- board text added: "I_DC_BUS AIN4"
- board text added: "Impulse Labs Drvbo v1.0 ch@"
- board text added: "PWM_A_H"
- board text added: "PWM_A_L"
- board text added: "PWM_B_H"
- board text added: "PWM_B_L"
- board text added: "V_DC AIN0+/AIN1-"
- board text added: "V_DC diff"
- board text removed: "DATAMATRIX CODE DATAMATRIX CODE DATAMATRIX CODE DATAMATRIX CODE DATAMATRIX CODE ########"
- board text removed: "Impulse Labs HEB Drvbo v1.0 ch@"

Commit message: prod candidate
Parts:
- added J11: Screw_Terminal_01x02, TerminalBlock_Phoenix:TerminalBlock_Phoenix_MPT-0,5-2-2.54_1x02_P2.54mm_Horizontal, F.Cu at (58.8, 72.5)
- added J12: Screw_Terminal_01x02, TerminalBlock_Phoenix:TerminalBlock_Phoenix_MPT-0,5-2-2.54_1x02_P2.54mm_Horizontal, F.Cu at (141.2, 81.8)
- added J13: Screw_Terminal_01x02, TerminalBlock_Phoenix:TerminalBlock_Phoenix_MPT-0,5-2-2.54_1x02_P2.54mm_Horizontal, F.Cu at (141.2, 75.0)
- added J14: Screw_Terminal_01x02, TerminalBlock_Phoenix:TerminalBlock_Phoenix_MPT-0,5-2-2.54_1x02_P2.54mm_Horizontal, F.Cu at (58.8, 79.2)
- added TP1: TestPoint, TestPoint:TestPoint_Pad_D1.5mm, F.Cu at (106.0, 84.2)
- added TP2: TestPoint, TestPoint:TestPoint_Pad_D1.5mm, F.Cu at (113.8, 84.2)
- FID1, FID2, FID3, FID4: footprint Fiducial:Fiducial_0.5mm_Mask1mm -> Fiducial:Fiducial_0.5mm_Mask1.5mm
- moved FID3 11.5 mm to (69.8, 79.2)
- moved FID1 5.10 mm to (65.5, 80.0)
Routing:
- net /5V0: track 71.0 -> 94.5 mm
- net /3V3: track 71.5 -> 86.1 mm
- net /~{GATE_DRIVER_ENABLE}: track 78.3 -> 92.0 mm
- net /HS_NTC_1: track 84.3 -> 86.3 mm
- net /HS_NTC_2: track 122.0 -> 123.7 mm
- net /PWM_A_H: track 89.4 -> 90.5 mm
- net /AIN8/9_P: track 29.4 -> 28.6 mm
- net /AIN0/1_P: track 17.8 -> 17.2 mm
- net /AIN0/1_N: track 15.4 -> 14.7 mm
- net GND: vias 99 -> 143
Other:
- board text added: "3V3,GND"
- board text added: "5V0,GND"
- board text added: "GND,GND"
- board text added: "HS_NTC_2 AIN8"
- board text added: "Impulse Labs drvbo v1.0 ch@"
- board text added: "~{EN},GND"
- board text removed: "HS_NTC_1 AIN8"
- board text removed: "Impulse Labs Drvbo v1.0 ch@"
