File: projects/impulse_drvbo/impulse_drvbo.kicad_sch (KiCad schematic)
At the start: 5 parts, among them J5 7472524-SINGLE

Commit message: wip
Parts:
- added C1, C2, C3, C4, C5, C6, C7: C, Capacitor_SMD:C_0603_1608Metric_Pad1.08x0.95mm_HandSolder, symbol Device:C
- added J1, J2: 5054481671, impulse_drvbo:MOLEX_5054481671, symbol impulse_drvbo:5054481671
- added J10, J3, J4, J6, J7, J8, J9: Conn_Coaxial, Connector_Coaxial:SMA_Amphenol_132291-12_Vertical, symbol Connector:Conn_Coaxial
- added R1, R2, R5, R6, R7, R8: 0, Resistor_SMD:R_0805_2012Metric_Pad1.20x1.40mm_HandSolder, symbol Device:R
- added R3, R4: 100K, Resistor_SMD:R_0805_2012Metric_Pad1.20x1.40mm_HandSolder, symbol Device:R
Connections:
- net AIN0/1_N: now also C2.1, C3.2, R2.2, R4.1
- net AIN0/1_P: now also C1.1, C3.1, R1.2, R3.1
- net AIN2/3_P: now also C4.1, R5.2
- net AIN4/5_P: now also C5.1, R6.2
- net AIN6/7_P: now also C6.1, R7.2
- net AIN8/9_P: now also C7.1, R8.2
- net GND: now also C1.2, C2.2, C4.2, C5.2, C6.2, C7.2, J1.10, J1.6, J1.S1 (SHIELD1), J1.S2 (SHIELD2), J10.2 (Ext), J2.10, J2.6, J2.S1 (SHIELD1), J2.S2 (SHIELD2), J4.2 (Ext), J6.2 (Ext), J7.2 (Ext), J8.2 (Ext), J9.2 (Ext), R3.2, R4.2
- new net 3V3: J1.5, J2.5
- new net 5V0: J1.9, J2.9
- new net HS_NTC_1: J1.1, J2.1, R7.1
- new net HS_NTC_2: J1.2, J2.2, R8.1
- new net I_AC_COIL: J1.3, J2.3, J4.1 (In), R5.1
- new net I_DC_BUS: J1.4, J2.4
- new net I_DC_COIL: J6.1 (In), R6.1
- new net PWM_A_H: J1.7, J2.7, J8.1 (In)
- new net PWM_A_L: J1.8, J2.8, J7.1 (In)
- new net PWM_B_H: J1.11, J10.1 (In), J2.11
- new net PWM_B_L: J1.12, J2.12, J9.1 (In)
- new net SHIELD: J1.14, J2.14
- new net V_DC_BUS_N: J1.16, J2.16, J3.2 (Ext), R2.1
- new net V_DC_BUS_P: J1.15, J2.15, J3.1 (In), R1.1
- new net ~{GATE_DRIVER_ENABLE}: J1.13, J2.13
- no-connect marks 34 -> 30
Other:
- moved on the sheet: H1, H2, H3, H4, J5

Commit message: wip
Changed lines of the file:
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@@
 	(wire
 		(pts
+			(xy 30.48 36.83) (xy 55.88 36.83)
+		)
+		(stroke
+			(width 0)
+			(type default)
+		)
+	)
+	(wire
+		(pts
 			(xy 82.55 91.44) (xy 82.55 86.36)
 		)
@@
 	(wire
 		(pts
-			(xy 33.02 41.91) (xy 55.88 41.91)
-		)
-		(stroke
-			(width 0)
-			(type default)
-		)
-	)
-	(wire
-		(pts
 			(xy 33.02 31.75) (xy 55.88 31.75)
 		)
@@
 	(wire
 		(pts
-			(xy 33.02 36.83) (xy 55.88 36.83)
-		)
-		(stroke
-			(width 0)
-			(type default)
-		)
-	)
-	(wire
-		(pts
 			(xy 293.37 46.99) (xy 311.15 46.99)
 		)
@@
 	(wire
 		(pts
+			(xy 24.13 41.91) (xy 55.88 41.91)
+		)
+		(stroke
+			(width 0)
+			(type default)
+		)
+	)
+	(wire
+		(pts
 			(xy 201.93 49.53) (xy 201.93 58.42)
 		)
@@
 		)
 	)
+	(netclass_flag ""
+		(length 2.54)
+		(shape round)
+		(at 24.13 41.91 90)
+		(fields_autoplaced yes)
+		(effects
+			(font
+				(size 1.27 1.27)
+			)
+			(justify left bottom)
+		)
+		(property "Netclass" "Power"
+			(at 21.59 41.2115 90)
+			(show_name yes)
+			(effects
+				(font
+					(size 1.27 1.27)
+					(italic yes)
+				)
+				(justify left)
+			)
+		)
+	)
+	(netclass_flag ""
+		(length 2.54)
+		(shape round)
+		(at 30.48 36.83 90)
+		(fields_autoplaced yes)
+		(effects
+			(font
+				(size 1.27 1.27)
+			)
+			(justify left bottom)
+		)
+		(property "Netclass" "Power"
+			(at 27.94 36.1315 90)
+			(show_name yes)
+			(effects
+				(font
+					(size 1.27 1.27)
+					(italic yes)
+				)
+				(justify left)
+			)
+		)
+	)

Commit message: wip
Connections:
- net I_DC_COIL is gone; now on net I_DC_BUS: J6.1 (In), R6.1
Changed lines of the file:
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@@
 		)
 	)
-	(label "I_DC_COIL"
+	(label "I_DC_BUS"
 		(at 176.53 110.49 0)
 		(fields_autoplaced yes)

Commit message: wip
Parts:
- added C8: C, Capacitor_SMD:C_0603_1608Metric_Pad1.08x0.95mm_HandSolder, symbol Device:C
- added FID1, FID2, FID3, FID4: Fiducial, Fiducial:Fiducial_0.5mm_Mask1mm, symbol Mechanical:Fiducial
- added R9: 0, Resistor_SMD:R_0805_2012Metric_Pad1.20x1.40mm_HandSolder, symbol Device:R
- J10, J3, J4, J6, J7, J8, J9: now not fitted
Connections:
- net GND: now also C8.2, R9.1
- net SHIELD: now also C8.1, R9.2

Commit message: prod candidate
Parts:
- added J11, J12, J13, J14: Screw_Terminal_01x02, TerminalBlock_Phoenix:TerminalBlock_Phoenix_MPT-0,5-2-2.54_1x02_P2.54mm_Horizontal, symbol Connector:Screw_Terminal_01x02
- added TP1, TP2: TestPoint, TestPoint:TestPoint_Pad_D1.5mm, symbol Connector:TestPoint
- FID1, FID2, FID3, FID4: footprint Fiducial:Fiducial_0.5mm_Mask1mm -> Fiducial:Fiducial_0.5mm_Mask1.5mm
Connections:
- net 3V3: now also J12.1 (Pin_1)
- net 5V0: now also J13.1 (Pin_1)
- net GND: now also J11.1 (Pin_1), J11.2 (Pin_2), J12.2 (Pin_2), J13.2 (Pin_2), J14.2 (Pin_2)
- net HS_NTC_1: now also TP1.1
- net HS_NTC_2: now also TP2.1
- net ~{GATE_DRIVER_ENABLE}: now also J14.1 (Pin_1)
Other:
- moved on the sheet: C6, C7, FID1, FID2, FID3, FID4, R7, R8
