File: projects/lora_nicerf_hat/lora_nicerf_hat.kicad_sch (KiCad schematic)
At the start: 1 part, among them J1 GPIO

Commit message: wip
Parts:
- added C1, C2, C3: C, Capacitor_SMD:C_0805_2012Metric_Pad1.18x1.45mm_HandSolder, symbol Device:C
- added C4, C5: DNI, Resistor_SMD:R_0402_1005Metric, symbol Device:R
- added J2: Conn_Coaxial, ch:SMA_Molex-73391-0070_Vertical, symbol Connector:Conn_Coaxial
- added L1: 0R, Resistor_SMD:R_0402_1005Metric, symbol Device:R
- added TP1: TestPoint, TestPoint:TestPoint_THTPad_2.0x2.0mm_Drill1.0mm, symbol Connector:TestPoint
- added U1: TPS7A0533PDBZ, Package_TO_SOT_SMD:SOT-23, symbol Regulator_Linear:TPS7A0533PDBZ
- added U2: LoRa1262-915, ch:G-Nice_RF_LoRa1262-915, symbol ch:G-Nice_RF_LoRa1262-915
Connections:
- net ~{RESET}: now reaches J1.12 (BCM18_PCM_C)
- net ~{RESET}: now also U2.6 (~{RESET})
- net GND: now reaches J1.14 (GND)
- net GND: now also J1.20 (GND), J1.25 (GND), J1.30 (GND), J1.34 (GND), J1.39 (GND), J1.6 (GND), J1.9 (GND), C1.2, C2.2, C3.2, C4.2, C5.2, J2.2 (Ext), U1.1 (GND), U2.1 (GND), U2.10 (GND), U2.8 (GND)
- net MOSI: now reaches J1.19 (BCM10_MOSI)
- net MOSI: now also U2.3 (MOSI)
- net +5V: now reaches J1.2 (5V)
- net +5V: now also J1.4 (5V), C1.1, U1.3 (VI)
- net MISO: now reaches J1.21 (BCM9_MISO)
- net MISO: now also U2.2 (MISO)
- net SCLK: now reaches J1.23 (BCM11_SCLK)
- net SCLK: now also U2.4 (SCK)
- net DIO1: now reaches J1.36 (BCM16)
- net DIO1: now also U2.15 (DIO1)
- net BUSY: now reaches J1.38 (BCM20_MOSI_PCM_DI)
- net BUSY: now also U2.16 (BUSY)
- net ~{CS}: now reaches J1.40 (BCM21_SCLK_PCM_DO)
- net ~{CS}: now also U2.5 (~{CS})
- new net: TP1.1, U2.11 (DIO3)
- new net +3.3VP: C2.1, C3.1, U1.2 (VO), U2.13 (VCC)
- new net RF: C5.1, J2.1 (In), L1.2
- new net RF_APRES_PI: C4.1, L1.1, U2.9 (RF)
- no-connect marks 0 -> 23
Other:
- note added: "Place near U1"
- moved on the sheet: J1

Commit message: wip
Parts:
- C1: value C -> 1u
- C2, C3: value C -> 4.7u
Connections:
- net RF renamed RF_OUT
- net RF_APRES_PI renamed RF_APRES_MATCH
Other:
- note added: "Input cap: 1 uF nominal Output cap: 1 uF nominal, 0.47 uF min, 22 uF max"
- moved on the sheet: C1, C2, C3, U1

Commit message: wip
Signed-off-by: Christopher Hoover <ch@murgatroid.com>
Parts:
- C1: value 1u -> 1u X7R
- C2, C3: value 4.7u -> 4.7u X7R
Other:
- note added: "TPS7A0533PDBZ Input cap: 1 uF nominal Output cap: 1 uF nominal, 0.47 uF min, 22 uF max"
- note removed: "Input cap: 1 uF nominal Output cap: 1 uF nominal, 0.47 uF min, 22 uF max"
- moved on the sheet: C1, C3
Changed lines of the file:
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@@
 	)
 	(junction
-		(at 40.64 148.59)
+		(at 41.91 148.59)
 		(diameter 0)
 		(color 0 0 0 0)
@@
 	(wire
 		(pts
-			(xy 96.52 143.51) (xy 96.52 147.32)
-		)
-		(stroke
-			(width 0)
-			(type default)
-		)
-	)
-	(wire
-		(pts
-			(xy 96.52 154.94) (xy 96.52 158.75)
-		)
-		(stroke
-			(width 0)
-			(type default)
-		)
-	)
-	(wire
-		(pts
-			(xy 40.64 157.48) (xy 40.64 158.75)
+			(xy 104.14 143.51) (xy 104.14 147.32)
+		)
+		(stroke
+			(width 0)
+			(type default)
+		)
+	)
+	(wire
+		(pts
+			(xy 104.14 154.94) (xy 104.14 158.75)
+		)
+		(stroke
+			(width 0)
+			(type default)
+		)
+	)
+	(wire
+		(pts
+			(xy 41.91 157.48) (xy 41.91 158.75)
 		)
 		(stroke
@@
 	(wire
 		(pts
-			(xy 40.64 143.51) (xy 40.64 148.59)
+			(xy 41.91 143.51) (xy 41.91 148.59)
 		)
 		(stroke
@@
 	(wire
 		(pts
-			(xy 40.64 148.59) (xy 40.64 149.86)
+			(xy 41.91 148.59) (xy 41.91 149.86)
 		)
 		(stroke
@@
 	(wire
 		(pts
-			(xy 49.53 148.59) (xy 40.64 148.59)
+			(xy 49.53 148.59) (xy 41.91 148.59)
 		)
 		(stroke
@@
 	(text "Place\nnear\nU1"
 		(exclude_from_sim no)
-		(at 102.616 151.13 0)
+		(at 110.236 151.13 0)
 		(effects
 			(font
@@
 		)
 	)
-	(text "Input cap: 1 uF nominal\nOutput cap: 1 uF nominal, 0.47 uF min, 22 uF max"
+	(text "TPS7A0533PDBZ\nInput cap: 1 uF nominal\nOutput cap: 1 uF nominal, 0.47 uF min, 22 uF max"
 		(exclude_from_sim no)
 		(at 38.1 169.164 0)
@@
 			)
 		)
-		(property "Value" "4.7u"
+		(property "Value" "4.7u X7R"
 			(at 73.66 154.9399 0)
 			(effects
@@
 	(symbol
 		(lib_id "power:+5V")
-		(at 40.64 143.51 0)
+		(at 41.91 143.51 0)
 		(unit 1)
 		(exclude_from_sim no)
@@
 		(fields_autoplaced yes)
 		(property "Reference" "#PWR03"
-			(at 40.64 147.32 0)
+			(at 41.91 147.32 0)
 			(effects
 				(font
@@
 		)
 		(property "Value" "+5V"
-			(at 40.64 138.43 0)
+			(at 41.91 138.43 0)
 			(effects
 				(font
@@
 		)
 		(property "Footprint" ""
-			(at 40.64 143.51 0)
+			(at 41.91 143.51 0)
 			(effects
 				(font
@@
 		)
 		(property "Datasheet" ""
-			(at 40.64 143.51 0)
+			(at 41.91 143.51 0)
 			(effects
 				(font
@@
 		)
 		(property "Description" "Power symbol creates a global label with name \"+5V\""
-			(at 40.64 143.51 0)
+			(at 41.91 143.51 0)
 			(effects
 				(font
@@
 	(symbol
 		(lib_id "Device:C")
-		(at 40.64 153.67 0)
+		(at 41.91 153.67 0)
 		(unit 1)
 		(exclude_from_sim no)
@@
 		(fields_autoplaced yes)
 		(property "Reference" "C1"
-			(at 44.45 152.3999 0)
+			(at 45.72 152.3999 0)
 			(effects
 				(font
@@
 			)
 		)
-		(property "Value" "1u"
-			(at 44.45 154.9399 0)
+		(property "Value" "1u X7R"
+			(at 45.72 154.9399 0)
 			(effects
 				(font
@@
 		)
 		(property "Footprint" "Capacitor_SMD:C_0805_2012Metric_Pad1.18x1.45mm_HandSolder"
-			(at 41.6052 157.48 0)
+			(at 42.8752 157.48 0)
 			(effects
 				(font
@@
 		)
 		(property "Datasheet" "~"
-			(at 40.64 153.67 0)
+			(at 41.91 153.67 0)
 			(effects
 				(font
@@
 		)
 		(property "Description" "Unpolarized capacitor"
-			(at 40.64 153.67 0)
+			(at 41.91 153.67 0)
 			(effects
 				(font
@@
 	(symbol
 		(lib_id "Device:C")
-		(at 96.52 151.13 0)
+		(at 104.14 151.13 0)
 		(unit 1)
 		(exclude_from_sim no)
@@
 		(dnp no)
 		(property "Reference" "C3"
-			(at 89.154 149.352 0)
+			(at 93.726 152.4 0)
 			(effects
 				(font
@@
 			)
 		)
-		(property "Value" "4.7u"
-			(at 89.154 151.892 0)
+		(property "Value" "4.7u X7R"
+			(at 93.472 154.94 0)
 			(effects
 				(font
@@
 		)
 		(property "Footprint" "Capacitor_SMD:C_0805_2012Metric_Pad1.18x1.45mm_HandSolder"
-			(at 97.4852 154.94 0)
+			(at 105.1052 154.94 0)
 			(effects
 				(font
@@
 		)
 		(property "Datasheet" "~"
-			(at 96.52 151.13 0)
+			(at 104.14 151.13 0)
 			(effects
 				(font
@@
 		)
 		(property "Description" "Unpolarized capacitor"
-			(at 96.52 151.13 0)
+			(at 104.14 151.13 0)
 			(effects
 				(font
@@
 	(symbol
 		(lib_id "power:GND")
-		(at 96.52 158.75 0)
+		(at 104.14 158.75 0)
 		(unit 1)
 		(exclude_from_sim no)
@@
 		(fields_autoplaced yes)
 		(property "Reference" "#PWR011"
-			(at 96.52 165.1 0)
+			(at 104.14 165.1 0)
 			(effects
 				(font
@@
 		)
 		(property "Value" "GND"
-			(at 96.52 163.83 0)
+			(at 104.14 163.83 0)
 			(effects
 				(font
@@
 		)
 		(property "Footprint" ""
-			(at 96.52 158.75 0)
+			(at 104.14 158.75 0)
 			(effects
 				(font
@@
 		)
 		(property "Datasheet" ""
-			(at 96.52 158.75 0)
+			(at 104.14 158.75 0)
 			(effects
 				(font
@@
 		)
 		(property "Description" "Power symbol creates a global label with name \"GND\" , ground"
-			(at 96.52 158.75 0)
+			(at 104.14 158.75 0)
 			(effects
 				(font
@@
 	(symbol
 		(lib_id "power:+3.3VP")
-		(at 96.52 143.51 0)
+		(at 104.14 143.51 0)
 		(unit 1)
 		(exclude_from_sim no)
@@
 		(fields_autoplaced yes)
 		(property "Reference" "#PWR010"
-			(at 100.33 144.78 0)
+			(at 107.95 144.78 0)
 			(effects
 				(font
@@
 		)
 		(property "Value" "+3.3VP"
-			(at 96.52 138.43 0)
+			(at 104.14 138.43 0)
 			(effects
 				(font
@@
 		)
 		(property "Footprint" ""
-			(at 96.52 143.51 0)
+			(at 104.14 143.51 0)
 			(effects
 				(font
@@
 		)
 		(property "Datasheet" ""
-			(at 96.52 143.51 0)
+			(at 104.14 143.51 0)
 			(effects
 				(font
@@
 		)
 		(property "Description" "Power symbol creates a global label with name \"+3.3VP\""
-			(at 96.52 143.51 0)
+			(at 104.14 143.51 0)
 			(effects
 				(font
@@
 	(symbol
 		(lib_id "power:GND")
-		(at 40.64 158.75 0)
+		(at 41.91 158.75 0)
 		(unit 1)
 		(exclude_from_sim no)
@@
 		(fields_autoplaced yes)
 		(property "Reference" "#PWR04"
-			(at 40.64 165.1 0)
+			(at 41.91 165.1 0)
 			(effects
 				(font
@@
 		)
 		(property "Value" "GND"
-			(at 40.64 163.83 0)
+			(at 41.91 163.83 0)
 			(effects
 				(font
@@
 		)
 		(property "Footprint" ""
-			(at 40.64 158.75 0)
+			(at 41.91 158.75 0)
 			(effects
 				(font
@@
 		)
 		(property "Datasheet" ""
-			(at 40.64 158.75 0)
+			(at 41.91 158.75 0)
 			(effects
 				(font
@@
 		)
 		(property "Description" "Power symbol creates a global label with name \"GND\" , ground"
-			(at 40.64 158.75 0)
-			(effects
-				(font
+			(at 41.91 158.75 0)
+			(effects
+				(font

Commit message: wip
Signed-off-by: Christopher Hoover <ch@murgatroid.com>
Parts:
- added J3, J4: Conn_Coaxial, Connector_Coaxial:U.FL_Hirose_U.FL-R-SMT-1_Vertical, symbol Connector:Conn_Coaxial
- C4, C5: now not fitted; now left out of the parts list
Connections:
- net GND: now also J3.2 (Ext), J4.2 (Ext)
- new net RF_TEST: J3.1 (In), J4.1 (In)
Other:
- note added: "Test"
