File: projects/impulse_temp_tester/impulse_temp_tester.kicad_pcb (KiCad board)
At the start: 2 copper layers, 89.8 x 53.5 mm, 28 parts, among them J1 Conn_Coaxial, J10 Screw_Terminal_01x02, J2 Conn_Coaxial, J3 Conn_01x01_Pin, J4 Screw_Terminal_01x02, J5 7472524-SINGLE, J6 Conn_01x01_Pin, J7 Screw_Terminal_01x02, J8 Screw_Terminal_01x02, J9 5054481071

Commit message: wip
Parts:
- removed C1: 500n, Capacitor_SMD:C_0603_1608Metric_Pad1.08x0.95mm_HandSolder
- removed C2, C3: 1u, Capacitor_SMD:C_0603_1608Metric_Pad1.08x0.95mm_HandSolder
- removed J1, J2: Conn_Coaxial, Connector_Coaxial:SMA_Amphenol_132291-12_Vertical
- removed J10: Screw_Terminal_01x02, TerminalBlock_Phoenix:TerminalBlock_Phoenix_MKDS-3-2-5.08_1x02_P5.08mm_Horizontal
- removed J3, J6: Conn_01x01_Pin, impulse_temp_tester:2.5sqmm_D2.5mm
- removed J4, J7, J8: Screw_Terminal_01x02, TerminalBlock_Phoenix:TerminalBlock_Phoenix_MPT-0,5-2-2.54_1x02_P2.54mm_Horizontal
- removed J9: 5054481071, impulse_temp_tester:MOLEX_5054481071
- removed R1, R4: 100K, Resistor_SMD:R_0805_2012Metric_Pad1.20x1.40mm_HandSolder
- removed R10, R11, R9: 0, Resistor_SMD:R_0805_2012Metric_Pad1.20x1.40mm_HandSolder
- removed R2, R3: 2000, Resistor_SMD:R_0805_2012Metric_Pad1.20x1.40mm_HandSolder
- removed R5, R6, R7, R8: R, Resistor_SMD:R_2512_6332Metric_Pad1.40x3.35mm_HandSolder
Routing:
- net /HEAT_P: track 70.2 -> 0.00 mm, vias 2 -> 0
- net /HEAT_N: track 68.9 -> 0.00 mm, vias 4 -> 0
- net /AIN2/2_P: track 61.1 -> 0.00 mm
- net +VDC: track 48.9 -> 0.00 mm
- net /AIN0/0_P: track 47.7 -> 0.00 mm
- net /AIN1/0_N: track 42.9 -> 0.00 mm, vias 2 -> 0
- net /SHIELD: track 12.0 -> 0.00 mm, vias 2 -> 0
- net GND: track 6.28 -> 0.00 mm, vias 25 -> 0
- net /12V_SHIELD: track 2.96 -> 0.00 mm
- removed copper zone on F.Cu, net +VDC
- removed copper zone on B.Cu, net /AIN1/0_N
- removed copper zone on B.Cu, net /HEAT_N
- removed copper zone on F.Cu, net /HEAT_N
- removed copper zone on F.Cu, net /HEAT_P
- removed copper zone on F.Cu, net GND
Other:
- board text removed: "GND"
- board text removed: "GND V+"
- board text removed: "H+"
- board text removed: "H-"
- board text removed: "Impulse Labs HEB Power Cal v1.2c ch@"
- board text removed: "dV"
- board text removed: "lpf(dV)"
