File: projects/ddf_big_array/ddf_big_array_antsw/ddf_big_array_antsw.kicad_pcb (KiCad board)
At the start: 4 copper layers, 90 x 90 mm, 50 parts, among them J1 Conn_Coaxial, J2 Conn_Coaxial, J3 Conn_Coaxial, J4 Conn_Coaxial, J5 Conn_Coaxial, J6 RJ45_Shielded, J7 5_Port_50Z_RF_Junction, U1 SMDA05

Commit message: checkpoint
Parts:
- removed C1, C2, C3, C4: 390p NP0 50V, Capacitor_SMD:C_0603_1608Metric
- removed C5, C6, C7, C8: 1n NP0 50V, Capacitor_SMD:C_0603_1608Metric
- removed C9: DNP, Capacitor_SMD:C_0603_1608Metric
- removed D1, D2, D3, D4: SMP1340, Diode_SMD:D_SOD-523
- removed J7: 5_Port_50Z_RF_Junction, ch:5 Port 50Z RF Junction
- removed L1, L2, L3, L4: 560n, ch:IMC1008
- removed L5: 0R, Inductor_SMD:L_0402_1005Metric_Pad0.77x0.64mm_HandSolder
- added U2: SKY13414-485LF, RF:Skyworks_SKY13575_639LF, F.Cu at (126.3, 87.1)
- added U3: STM32G0B1CBT, Package_QFP:LQFP-48_7x7mm_P0.5mm, F.Cu at (148.3, 102.5)
Connections:
- U1 pad 1: Net-(FB1-Pad2) -> Net-(U1-A1)
- U1 pad 2: Net-(FB2-Pad2) -> Net-(U1-B1)
- U1 pad 3: Net-(FB3-Pad2) -> Net-(U1-C1)
- U1 pad 4: Net-(FB4-Pad2) -> Net-(U1-D1)
Routing:
- net /RF_OUT: track 44.3 -> 7.38 mm
- net Net-(C8-Pad1): track 40.0 -> 3.34 mm, vias 2 -> 0
- net Net-(C7-Pad1): track 34.6 -> 1.29 mm, vias 2 -> 0
- net Net-(C5-Pad1): track 27.3 -> 1.29 mm, vias 2 -> 0
- net /E_IN: track 25.8 -> 0.00 mm
- net /S_IN: track 25.8 -> 0.00 mm
- net /N_IN: track 25.8 -> 0.00 mm
- net /W_IN: track 25.5 -> 0.00 mm
- net Net-(C6-Pad1): track 15.9 -> 1.29 mm, vias 2 -> 0
- net GND: track 18.5 -> 12.2 mm, vias 312 -> 307
- net /E_SW_DCB: track 5.48 -> 0.00 mm
- net /S_SW_DCB: track 5.45 -> 0.00 mm
- net /W_SW_DCB: track 5.45 -> 0.00 mm
- net /N_SW_DCB: track 5.45 -> 0.00 mm
- net /E_SW: track 4.53 -> 0.00 mm
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