File: projects/ddf_big_array/ddf_big_array_antsw/ddf_big_array_antsw.kicad_sch (KiCad schematic)
At the start: 50 parts, among them J1 Conn_Coaxial, J2 Conn_Coaxial, J3 Conn_Coaxial, J4 Conn_Coaxial, J5 Conn_Coaxial, J6 RJ45_Shielded, J7 5_Port_50Z_RF_Junction, U1 SMDA05

Commit message: checkpoint
Parts:
- removed C1, C2, C3, C4: 390p NP0 50V, Capacitor_SMD:C_0603_1608Metric, symbol Device:C
- removed C5, C6, C7, C8: 1n NP0 50V, Capacitor_SMD:C_0603_1608Metric, symbol Device:C
- removed C9: DNP, Capacitor_SMD:C_0603_1608Metric, symbol Device:C
- removed D1, D2, D3, D4: SMP1340, Diode_SMD:D_SOD-523, symbol Device:D
- removed D5, D6, D7, D8, D9: ESD7951ST5G, Diode_SMD:D_SOD-923, symbol Device:D_TVS
- removed J7: 5_Port_50Z_RF_Junction, ch:5 Port 50Z RF Junction, symbol ch:5_Port_50Z_RF_Junction
- removed L1, L2, L3, L4: 560n, ch:IMC1008, symbol Device:L
- removed L5: 0R, Inductor_SMD:L_0402_1005Metric_Pad0.77x0.64mm_HandSolder, symbol Device:L
- removed R1, R3, R5, R7, R9: 100K, Resistor_SMD:R_0603_1608Metric, symbol Device:R
- removed R2, R4, R6, R8: 270, Resistor_SMD:R_0603_1608Metric_Pad0.98x0.95mm_HandSolder, symbol Device:R
- added U2: SKY13414-485LF, RF:Skyworks_SKY13575_639LF, symbol ddf_big_array:SKY13575-639LF
- C10: footprint Capacitor_SMD:C_0603_1608Metric -> (none); LCSC C77026 -> (none); MFG Murata -> (none); MPN GRM1885C1H102JA01D -> (none)
- FB1, FB2, FB3, FB4: footprint Inductor_SMD:L_0603_1608Metric -> (none); LCSC C94375 -> (none); MFG Sunlord -> (none); MPN GZ1608D601TF -> (none)
- H1, H2, H3, H4: footprint MountingHole:MountingHole_3.2mm_M3_Pad_TopBottom -> (none)
- J1, J2, J3, J4, J5: footprint ch:SMA_Horizontal -> (none); LCSC C1509208 -> (none)
- J6: footprint Connector_RJ:RJ45_Amphenol_RJHSE5380 -> (none); LCSC C464586 -> (none)
- R10: footprint Resistor_SMD:R_0603_1608Metric -> (none); LCSC C14675 -> (none); MFG Yageo -> (none); MPN RC0603FR-07100KL -> (none)
Connections:
- net GND: now also U2.15 (GND)
- net E_IN renamed AntChannel_E/ANT_IN
- net N_IN renamed AntChannel_N/ANT_IN
- net RF_OUT renamed SwitcherOutput/SW_OUT
- net S_IN renamed AntChannel_S/ANT_IN
- net W_IN renamed AntChannel_W/ANT_IN
- new net AntChannel_E/ANT_OUT: U2.9 (RF2)
- new net AntChannel_N/ANT_OUT: U2.3 (RF1)
- new net AntChannel_S/ANT_OUT: U2.2 (RF3)
- new net AntChannel_W/ANT_OUT: U2.10 (RF4)
- new net SwitcherOutput/SW_OUT_IN: U2.13 (RFC)
Other:
- added sheet AntChannel_E (ant_channel.kicad_sch)
- added sheet AntChannel_N (ant_channel.kicad_sch)
- added sheet AntChannel_S (ant_channel.kicad_sch)
- added sheet AntChannel_W (ant_channel.kicad_sch)
- added sheet SwitcherOutput (switcher_ouput.kicad_sch)
- added sheet mcu (mcu.kicad_sch)
- note removed: "560nH @ 144MHz => Z=506Ω 560nH @ 440MHz => Z=1547Ω 390pF @ 144MHz => Z=2.84Ω 390pF @ 440MHz => Z=0.928Ω"
- moved on the sheet: H1, H2, H3, H4, J1, J2, J3, J4, J5
