File: projects/rpi_hat_templates/rpi_hat_template_uhat_smt_bot/rpi_hat_template_uhat_smt_bot.kicad_pcb (KiCad board)
At the start: 2 copper layers, 65 x 27 mm, 5 parts, among them J1 Harwin M20-7812045-R

Commit message: Fixes border outlines
Other:
- board size 65 x 27 mm -> 65 x 30.5 mm
