File: projects/iso_xfmr/iso_xfmr.kicad_pcb (KiCad board)
At the start: 2 copper layers, 76.2 x 50.8 mm, 13 parts, among them J1 Conn_Coaxial, J2 Conn_Coaxial, J3 Conn_02x03_Odd_Even

Commit message: Small fix ups
Parts:
- TR1: footprint triad_magnetics:Untitled -> triad_magnetics:ty-145p
Changed lines of the file:
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@@
 		(embedded_fonts no)
 	)
-	(footprint "triad_magnetics:Untitled"
+	(footprint "triad_magnetics:ty-145p"
 		(layer "F.Cu")
 		(at 146.05 95.25)
 		(property "Reference" "TR1"
-			(at 7.62 -12.065 0)
+			(at 0 -12.7 0)
 			(unlocked yes)
 			(layer "F.SilkS")
@@
 		(sheetname "/")
 		(sheetfile "iso_xfmr.kicad_sch")
-		(attr smd)
+		(attr through_hole)
 		(fp_rect
 			(start -9.525 -11.43)
