File: projects/iso_xfmr/iso_xfmr.kicad_sch (KiCad schematic)
At the start: 13 parts, among them J1 Conn_Coaxial, J2 Conn_Coaxial, J3 Conn_02x03_Odd_Even

Commit message: Small fix ups
Parts:
- TR1: footprint triad_magnetics:Untitled -> triad_magnetics:ty-145p
Changed lines of the file:
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@@
 			)
 		)
-		(property "Footprint" "triad_magnetics:Untitled"
+		(property "Footprint" "triad_magnetics:ty-145p"
 			(at 69.088 67.564 0)
 			(effects
