File: projects/canob/canob.kicad_sch (KiCad schematic)
At the start: 45 parts, among them J1 USB_C_Receptacle_USB2.0, J2 5054481071, J4 Conn_01x02, J6 5054481071, U1 STM32G0B1CBT, U2 TPSM53602RDA, U3 TJA1051T-3, U4 TLV493D, Y1 Crystal_GND24_Small

Commit message: wip
Parts:
- removed C4: 100n, Capacitor_SMD:C_0603_1608Metric, symbol Device:C
- removed D5, D6: D_Schottky, symbol Device:D_Schottky
- removed J4: Conn_01x02, Connector_PinHeader_2.54mm:PinHeader_1x03_P2.54mm_Vertical, symbol Connector_Generic:Conn_01x03
- removed U3: TJA1051T-3, Package_SO:SOIC-8_3.9x4.9mm_P1.27mm, symbol Interface_CAN_LIN:TJA1051T-3
- added D5: 20CJQ045, Package_TO_SOT_SMD:SOT-223-3_TabPin2, symbol Device:D_Schottky_Dual_CommonCathode_AKA_Parallel
- added JP1: SolderJumper_2_Open, Jumper:SolderJumper-2_P1.3mm_Open_TrianglePad1.0x1.5mm, symbol Jumper:SolderJumper_2_Open
- added U3: TCAN337G, Package_TO_SOT_SMD:TSOT-23-8, symbol Interface_CAN_LIN:TCAN337G
- R14, R15: value 0 -> 0/DNI
Connections:
- net +12V: now also D5.1 (A)
- net +3V3: now also C10.1, U3.3 (VCC)
- net +5V: now also D5.3 (A); no longer C10.1
- net CAN1_H: now also JP1.2 (B), U3.7 (CANH)
- net CAN1_L: now also U3.6 (CANL)
- net CAN1_RX: now also U3.4 (RXD)
- net CAN1_S: now also U3.8 (S)
- net CAN1_TX: now also U3.1 (TXD)
- net GND: now also U3.2 (GND)
- net VIN: now reaches C11.1, C5.1, C6.1, U2.1 (VIN), U2.14 (VIN), U2.2 (EN)
- net VIN: now also D5.2 (K)
- net at R8.1: now also JP1.1 (A)
- net FB: now reaches R11.1, R7.2, U2.9 (FB)
- net SWDIO: no longer names the net of U1.35 (PA13)
- no-connect marks 35 -> 36
Other:
- moved on the sheet: C1, C10, C11, C12, C13, C2, C3, C5, C6, C7, C8, C9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

Commit message: wip
Parts:
- added R10, R16, R17, R9: 10K, Resistor_SMD:R_0402_1005Metric, symbol Device:R
- added SW1: SW_Coded_SH-7010, Button_Switch_SMD:Nidec_Copal_SH-7010A, symbol Switch:SW_Coded_SH-7010
- R1, R11, R12, R13, R2, R3, R4, R5, R6, R7: footprint Resistor_SMD:R_0603_1608Metric -> Resistor_SMD:R_0402_1005Metric
- R14, R15: footprint Resistor_SMD:R_1206_3216Metric -> Resistor_SMD:R_0402_1005Metric
Connections:
- net +3V3: now also R10.1, R16.1, R17.1, R9.1
- net GND: now also SW1.C
- net SW_B0: now reaches U1.22 (PB10)
- net SW_B0: now also R9.2, SW1.1
- net SW_B1: now reaches U1.23 (PB11)
- net SW_B1: now also R10.2, SW1.2
- net SW_B2: now reaches U1.24 (PB12)
- net SW_B2: now also R16.2, SW1.4
- net SW_B3: now reaches U1.25 (PB13)
- net SW_B3: now also R17.2, SW1.8
- no-connect marks 36 -> 32

Commit message: wip
Parts:
- removed C11: 47u X5R/X7R, Capacitor_SMD:C_2220_5750Metric, symbol Device:C
- removed R14: 0/DNI, Resistor_SMD:R_0402_1005Metric, symbol Device:R
- added C4: 10u X7R, Capacitor_SMD:C_1206_3216Metric, symbol Device:C
- added D6: NUP2105L, Package_TO_SOT_SMD:SOT-23, symbol Power_Protection:NUP2105L
- added JP2: SolderJumper_3_Bridged12, Jumper:SolderJumper-3_P1.3mm_Bridged12_Pad1.0x1.5mm, symbol Jumper:SolderJumper_3_Bridged12
- added R18: 10K, Resistor_SMD:R_0402_1005Metric, symbol Device:R
- C12: value 47u X5R/X7R -> 47u 6V3 X5R (C3225X5R0J476K); footprint Capacitor_SMD:C_2220_5750Metric -> Capacitor_SMD:C_1210_3225Metric
Connections:
- net +12V: now also JP2.2 (C); no longer J2.1, J2.3, J2.5, J6.1, J6.3, J6.5
- net +3V3: now also R18.1
- net CAN1_H: now also D6.1 (K)
- net CAN1_L: now also D6.2 (K)
- net GND: now also C4.2, D6.3 (A)
- net VIN: now also C4.1
- net CAN1_FAULT: now reaches U1.40 (PD2)
- net CAN1_FAULT: now also U3.5 (FAULT), R18.2
- net 12V_SHIELD renamed 12V_STBY
- net 12V_STBY: now also JP2.3 (B)
- new net 12V_PRI: J2.1, J2.3, J2.5, J6.1, J6.3, J6.5, JP2.1 (A)
- no-connect marks 32 -> 30
Other:
- moved on the sheet: C10, C12, C13, C5, C6, D4, D5, J2, J6, JP1, R10, R11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

Commit message: wip
Parts:
- removed C12: 47u 6V3 X5R (C3225X5R0J476K), Capacitor_SMD:C_1210_3225Metric, symbol Device:C
- removed JP2: SolderJumper_3_Bridged12, Jumper:SolderJumper-3_P1.3mm_Bridged12_Pad1.0x1.5mm, symbol Jumper:SolderJumper_3_Bridged12
- removed R11: 4K32, Resistor_SMD:R_0402_1005Metric, symbol Device:R
- removed R7: 10K, Resistor_SMD:R_0402_1005Metric, symbol Device:R
- removed U2: TPSM53602RDA, Package_DFN_QFN:Texas_B3QFN-14-1EP_5x5.5mm_P0.65mm_ThermalVia, symbol Converter_DCDC:TPSM53602RDA
- added R16, R17: 0, Resistor_SMD:R_0402_1005Metric, symbol Device:R
- added U2: TPSM265R1, canob:SIL0010C, symbol canob:TPSM265R1
- C10: renamed from C9; footprint Capacitor_SMD:C_0603_1608Metric -> Capacitor_SMD:C_0402_1005Metric
- C11: renamed from C13; footprint Capacitor_SMD:C_0603_1608Metric -> Capacitor_SMD:C_0402_1005Metric
- C4: value 10u X7R -> 4u7; footprint Capacitor_SMD:C_1206_3216Metric -> Capacitor_SMD:C_0603_1608Metric
- C5: renamed from C10; footprint Capacitor_SMD:C_0603_1608Metric -> Capacitor_SMD:C_0402_1005Metric
- D1: renamed from D5; value 20CJQ045 -> tbd; footprint Package_TO_SOT_SMD:SOT-223-3_TabPin2 -> Package_TO_SOT_SMD:SOT-323_SC-70
- D4: renamed from D1; footprint LED_SMD:LED_0603_1608Metric -> LED_SMD:LED_0402_1005Metric
- D5: renamed from D2; footprint LED_SMD:LED_0603_1608Metric -> LED_SMD:LED_0402_1005Metric
- D6: renamed from D3; footprint LED_SMD:LED_0603_1608Metric -> LED_SMD:LED_0402_1005Metric
- renumbered C5 to C1, C6 to C2, C2 to C3, C1 to C6, C3 to C7, C7 to C8, C8 to C9, D4 to D2, D6 to D3, J6 to J2, J2 to J3, R2 to R1, R9 to R10, R10 to R11, R16 to R12, R17 to R13, R12 to R14, R13 to R15, R4 to R2, R18 to R3, R6 to R4, R8 to R5, R15 to R6, R1 to R7, R3 to R8, R5 to R9, RV2 to RV1, RV1 to RV2
Connections:
- net +12V: now also R16.2, R17.1
- net +3V3: now also C4.1, U2.1 (VOUT), U2.8 (SENSE+_FB)
- net 12V_PRI: now also R16.1
- net 12V_STBY: now also R17.2
- net GND: now also U2.11 (GND), U2.3 (GND), U2.6 (GND)
- net SW_B0: now also U1.23 (PB11); no longer U1.22 (PB10)
- net SW_B1: now also U1.25 (PB13); no longer U1.23 (PB11)
- net SW_B3: now also U1.22 (PB10); no longer U1.25 (PB13)
- net VIN: now also U2.4 (VIN), U2.5 (VIN), U2.9 (EN); no longer C4.1
- net CAN1_H renamed CAN1_P
- net CAN1_P: now also D2.2 (K), D3.2 (K); no longer D2.1 (K), D3.1 (K)
- net CAN1_L renamed CAN1_N
- net CAN1_N: now also D2.1 (K), D3.1 (K); no longer D2.2 (K), D3.2 (K)
- no-connect marks 30 -> 31
Other:
- moved on the sheet: C1, C2, D1

Commit message: Draft release version.
Parts:
- D1: value tbd -> BAT54CWFILM
Other:
- note added: "If(max) = 300 mA"
- note added: "Iout(max) = 100 mA Vin = 3-65 V"
Changed lines of the file:
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@@
 	(generator_version "9.0")
 	(paper "B")
+	(text "Iout(max) = 100 mA\nVin = 3-65 V"
+		(exclude_from_sim no)
+		(at 288.544 62.484 0)
+		(effects
+			(font
+				(size 1.27 1.27)
+			)
+		)
+	)
 	(text "8 MHz 3225"
 		(exclude_from_sim no)
@@
 		)
 	)
+	(text "If(max) = 300 mA"
+		(exclude_from_sim no)
+		(at 207.264 40.132 0)
+		(effects
+			(font
+				(size 1.27 1.27)
+			)
+		)
+	)
 	(junction
 		(at 294.64 33.02)
@@
 			)
 		)
-		(property "Value" "tbd"
+		(property "Value" "BAT54CWFILM"
 			(at 212.0265 26.67 0)
 			(effects

Commit message: wip
Parts:
- removed U2: TPSM265R1, canob:SIL0010C, symbol canob:TPSM265R1
- added R18, R20: DNP, Resistor_SMD:R_0402_1005Metric, symbol Device:R
- added R19: 40K2, Resistor_SMD:R_0402_1005Metric, symbol Device:R
- added U2: TPSM82902SISR, canob:uSIP11_SIS_TEX, symbol canob:TPSM82902SISR
- C1: value 10u X7R -> 10u X7R 50V
- C2: value 10u X7R -> DNP; footprint Capacitor_SMD:C_1206_3216Metric -> Capacitor_SMD:C_0402_1005Metric; now not fitted
- C4: value 4u7 -> 22u X7R 10V; footprint Capacitor_SMD:C_0603_1608Metric -> Capacitor_SMD:C_1206_3216Metric
- D1: value BAT54CWFILM -> SB05W05C; footprint Package_TO_SOT_SMD:SOT-323_SC-70 -> Package_TO_SOT_SMD:SOT-23-3
Connections:
- net +3V3: now also R20.1, U2.10 (VOUT), U2.9 (VOUT)
- net GND: now also R18.2, R19.2, U2.11 (GND)
- net VIN: now also U2.1 (VIN), U2.2 (VIN), U2.3 (EN); no longer C2.1
- new net: R19.1, U2.4 (MODE/S-CONF)
- new net: C2.1, U2.5 (SS/TR)
- new net: R18.1, R20.2, U2.7 (FB/VSET)
- no-connect marks 31 -> 29
Other:
- note added: "40K2 => AUTO PFM/PWM w/ACE VSET Fsw=2.5 MHz No output discharge"
- note added: "Io(avg)=500 mA"
- note added: "Io(max) = 2A"
- note added: "SS/TR floating => fastest ramp"
- note added: "VSET open => 3V3"
- note removed: "If(max) = 300 mA"
- note removed: "Iout(max) = 100 mA Vin = 3-65 V"
- moved on the sheet: C4

Commit message: wip
Parts:
- removed R3: 10K, Resistor_SMD:R_0402_1005Metric, symbol Device:R
- removed U3: TCAN337G, Package_TO_SOT_SMD:TSOT-23-8, symbol Interface_CAN_LIN:TCAN337G
- added U3: TCAN330G, Package_TO_SOT_SMD:TSOT-23-8, symbol Interface_CAN_LIN:TCAN330G
- R9: value 330 -> 680
Connections:
- net +3V3: now also U3.3 (VCC)
- net CAN1_N: now also U3.6 (CANL)
- net CAN1_P: now also U3.7 (CANH)
- net CAN1_RX: now also U3.4 (RXD)
- net CAN1_S: now also U3.8 (S)
- net CAN1_TX: now also U3.1 (TXD)
- net GND: now also U3.2 (GND)
- net SW_B0: now also U1.22 (PB10); no longer U1.23 (PB11)
- net SW_B3: now also U1.23 (PB11); no longer U1.22 (PB10)
- net CAN1_FAULT: no longer names the net of U1.40 (PD2)
- no-connect marks 29 -> 31
Other:
- moved on the sheet: JP1, R10, R11, R12, R13, R16, R17, R5, SW1

Commit message: Removes LCSC field from symbols for passives and LEDs (several did not match the chosen footprint)
Parts:
- C10, C7: LCSC C14663 -> (none)
- D4: LCSC C9900012286 -> (none)
- D5: LCSC C3030991 -> (none)
- D6: LCSC C5252984 -> (none)
- R6: LCSC C473612 -> (none)
Changed lines of the file:
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@@
 			)
 		)
-		(property "LCSC" "C5252984"
+		(property "LCSC" ""
 			(at 62.23 203.2 90)
 			(effects
@@
 			)
 		)
-		(property "LCSC" "C14663"
+		(property "LCSC" ""
 			(at 67.31 143.51 0)
 			(effects
@@
 			)
 		)
-		(property "LCSC" "C14663"
+		(property "LCSC" ""
 			(at 46.99 111.76 0)
 			(effects
@@
 			)
 		)
-		(property "LCSC" "C9900012286"
+		(property "LCSC" ""
 			(at 35.56 203.2 90)
 			(effects
@@
 			)
 		)
-		(property "LCSC" "C473612"
+		(property "LCSC" ""
 			(at 325.12 144.78 0)
 			(effects
@@
 			)
 		)
-		(property "LCSC" "C3030991"
+		(property "LCSC" ""
 			(at 49.53 203.2 90)
 			(effects
