File: projects/tbox/kicad/control.kicad_sch (KiCad schematic)
At the start: 5 parts, among them J902 TO FRONT J901, J903 TO REAR J904

Commit message: Prep for board-coded annotation: page numbers 1x/2x/3x, Interconnect field on the ribbon connectors
Parts:
- J902: Interconnect (none) -> FC
- J903: Interconnect (none) -> CR
Changed lines of the file:
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@@
     (property "Reference" "J902" (at 66.04 106.68 0) (effects (font (size 1.27 1.27))))
     (property "Value" "TO FRONT J901" (at 66.04 109.22 0) (effects (font (size 1.27 1.27))))
+    (property "Interconnect" "FC" (at 66.04 106.68 0) (effects (font (size 1.27 1.27)) (hide yes)))
     (property "Footprint" "" (at 66.04 127 0) (effects (font (size 1.27 1.27)) (hide yes)))
     (property "Datasheet" "" (at 66.04 127 0) (effects (font (size 1.27 1.27)) (hide yes)))
@@
     (property "Reference" "J903" (at 200.66 106.68 0) (effects (font (size 1.27 1.27))))
     (property "Value" "TO REAR J904" (at 200.66 109.22 0) (effects (font (size 1.27 1.27))))
+    (property "Interconnect" "CR" (at 200.66 106.68 0) (effects (font (size 1.27 1.27)) (hide yes)))
     (property "Footprint" "" (at 200.66 127 0) (effects (font (size 1.27 1.27)) (hide yes)))
     (property "Datasheet" "" (at 200.66 127 0) (effects (font (size 1.27 1.27)) (hide yes)))
@@
     (pin "MUTE_B" output (at 83.82 50.8 0) (effects (font (size 1.27 1.27)) (justify right)))
     (pin "PTT_ACTIVE" output (at 83.82 55.88 0) (effects (font (size 1.27 1.27)) (justify right)))
-    (instances (project "tbox" (path "/6a29b3f1-3e67-482d-942d-4557fa8bc2d6/7885f5d1-bf3d-5361-a0a2-98a329efbaa8" (page "8"))))
+    (instances (project "tbox" (path "/6a29b3f1-3e67-482d-942d-4557fa8bc2d6/7885f5d1-bf3d-5361-a0a2-98a329efbaa8" (page "21"))))
   )
   (sheet (at 124.46 40.64) (size 45.72 22.86)
@@
     (pin "PTT_ACTIVE" input (at 124.46 55.88 180) (effects (font (size 1.27 1.27)) (justify left)))
     (pin "TX_MIX" output (at 170.18 45.72 0) (effects (font (size 1.27 1.27)) (justify right)))
-    (instances (project "tbox" (path "/6a29b3f1-3e67-482d-942d-4557fa8bc2d6/7885f5d1-bf3d-5361-a0a2-98a329efbaa8" (page "9"))))
+    (instances (project "tbox" (path "/6a29b3f1-3e67-482d-942d-4557fa8bc2d6/7885f5d1-bf3d-5361-a0a2-98a329efbaa8" (page "22"))))
   )
   (sheet (at 210.82 40.64) (size 45.72 27.94)
@@
     (pin "PH_B_L" output (at 256.54 55.88 0) (effects (font (size 1.27 1.27)) (justify right)))
     (pin "PH_B_R" output (at 256.54 60.96 0) (effects (font (size 1.27 1.27)) (justify right)))
-    (instances (project "tbox" (path "/6a29b3f1-3e67-482d-942d-4557fa8bc2d6/7885f5d1-bf3d-5361-a0a2-98a329efbaa8" (page "11"))))
+    (instances (project "tbox" (path "/6a29b3f1-3e67-482d-942d-4557fa8bc2d6/7885f5d1-bf3d-5361-a0a2-98a329efbaa8" (page "24"))))
   )
 )

Commit message: Annotate by board: KiCad annotator, first free after sheet number x100 (1xxx front, 2xxx control, 3xxx rear)
Parts:
- renumbered C911 to C2001, C912 to C2002, C913 to C2003, J902 to J2001, J903 to J2002

Commit message: Rename refdes mentions in notes and docs to the board-coded numbering
Table-driven: the old->new map was derived from symbol UUIDs across the
annotation commit (619 instances, checked one-to-one and per board), and
only exact whole tokens from that table were replaced, in sheet notes,
connector Values, DESIGN.md, TODO.md and power_tree.json.  The one range
("J901-J904") and the one instance-specific ref in the shared Mute sheet
were rewritten by hand.  Power tree regenerated (loads now grouped by
board).  Netlist identical to the annotated baseline.
Parts:
- J2001: value TO FRONT J901 -> TO FRONT J1005
- J2002: value TO REAR J904 -> TO REAR J3001
Other:
- note added: "J2001: ribbon to the front board (J1005). J2002: ribbon to the rear board (J3001). GAIN_x_HI / BIAS_x pass straight through from J2002 to J2001."
- note removed: "J902: ribbon to the front board (J901). J903: ribbon to the rear board (J904). GAIN_x_HI / BIAS_x pass straight through from J903 to J902."
Changed lines of the file:
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@@
 		)
 	)
-	(text "J902: ribbon to the front board (J901). J903: ribbon to the rear board (J904). GAIN_x_HI / BIAS_x pass straight through from J903 to J902."
+	(text "J2001: ribbon to the front board (J1005). J2002: ribbon to the rear board (J3001). GAIN_x_HI / BIAS_x pass straight through from J2002 to J2001."
 		(exclude_from_sim no)
 		(at 20.32 24.13 0)
@@
 			)
 		)
-		(property "Value" "TO FRONT J901"
+		(property "Value" "TO FRONT J1005"
 			(at 66.04 109.22 0)
 			(show_name no)
@@
 			)
 		)
-		(property "Value" "TO REAR J904"
+		(property "Value" "TO REAR J3001"
 			(at 200.66 109.22 0)
 			(show_name no)
