File: projects/tbox/kicad/rear.kicad_sch (KiCad schematic)
At the start: 1 part, among them J904 TO CTRL J903

Commit message: Prep for board-coded annotation: page numbers 1x/2x/3x, Interconnect field on the ribbon connectors
Parts:
- J904: Interconnect (none) -> CR
Changed lines of the file:
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@@
     (property "Reference" "J904" (at 66.04 119.38 0) (effects (font (size 1.27 1.27))))
     (property "Value" "TO CTRL J903" (at 66.04 121.92 0) (effects (font (size 1.27 1.27))))
+    (property "Interconnect" "CR" (at 66.04 119.38 0) (effects (font (size 1.27 1.27)) (hide yes)))
     (property "Footprint" "" (at 66.04 139.7 0) (effects (font (size 1.27 1.27)) (hide yes)))
     (property "Datasheet" "" (at 66.04 139.7 0) (effects (font (size 1.27 1.27)) (hide yes)))
@@
     (property "Sheetname" "Supply" (at 38.1 37.14 0) (effects (font (size 1.27 1.27)) (justify left bottom)))
     (property "Sheetfile" "supply.kicad_sch" (at 38.1 39.64 0) (effects (font (size 1.27 1.27)) (justify left bottom)))
-    (instances (project "tbox" (path "/6a29b3f1-3e67-482d-942d-4557fa8bc2d6/6aedcaa5-d555-5688-b8e3-a5d8be255c1c" (page "13"))))
+    (instances (project "tbox" (path "/6a29b3f1-3e67-482d-942d-4557fa8bc2d6/6aedcaa5-d555-5688-b8e3-a5d8be255c1c" (page "31"))))
   )
   (sheet (at 124.46 40.64) (size 45.72 38.1)
@@
     (pin "PTT_A_IN" output (at 170.18 66.04 0) (effects (font (size 1.27 1.27)) (justify right)))
     (pin "PTT_B_IN" output (at 170.18 71.12 0) (effects (font (size 1.27 1.27)) (justify right)))
-    (instances (project "tbox" (path "/6a29b3f1-3e67-482d-942d-4557fa8bc2d6/6aedcaa5-d555-5688-b8e3-a5d8be255c1c" (page "14"))))
+    (instances (project "tbox" (path "/6a29b3f1-3e67-482d-942d-4557fa8bc2d6/6aedcaa5-d555-5688-b8e3-a5d8be255c1c" (page "32"))))
   )
   (sheet (at 210.82 40.64) (size 45.72 22.86)
@@
     (pin "RX_R_BUS" input (at 210.82 50.8 180) (effects (font (size 1.27 1.27)) (justify left)))
     (pin "TX_MIX" input (at 210.82 55.88 180) (effects (font (size 1.27 1.27)) (justify left)))
-    (instances (project "tbox" (path "/6a29b3f1-3e67-482d-942d-4557fa8bc2d6/6aedcaa5-d555-5688-b8e3-a5d8be255c1c" (page "15"))))
+    (instances (project "tbox" (path "/6a29b3f1-3e67-482d-942d-4557fa8bc2d6/6aedcaa5-d555-5688-b8e3-a5d8be255c1c" (page "33"))))
   )
   (sheet (at 210.82 106.68) (size 45.72 22.86)
@@
     (pin "RX_L_BUS" output (at 256.54 111.76 0) (effects (font (size 1.27 1.27)) (justify right)))
     (pin "RX_R_BUS" output (at 256.54 116.84 0) (effects (font (size 1.27 1.27)) (justify right)))
-    (instances (project "tbox" (path "/6a29b3f1-3e67-482d-942d-4557fa8bc2d6/6aedcaa5-d555-5688-b8e3-a5d8be255c1c" (page "16"))))
+    (instances (project "tbox" (path "/6a29b3f1-3e67-482d-942d-4557fa8bc2d6/6aedcaa5-d555-5688-b8e3-a5d8be255c1c" (page "34"))))
   )
 )

Commit message: Annotate by board: KiCad annotator, first free after sheet number x100 (1xxx front, 2xxx control, 3xxx rear)
Parts:
- renumbered J904 to J3001

Commit message: Rename refdes mentions in notes and docs to the board-coded numbering
Table-driven: the old->new map was derived from symbol UUIDs across the
annotation commit (619 instances, checked one-to-one and per board), and
only exact whole tokens from that table were replaced, in sheet notes,
connector Values, DESIGN.md, TODO.md and power_tree.json.  The one range
("J901-J904") and the one instance-specific ref in the shared Mute sheet
were rewritten by hand.  Power tree regenerated (loads now grouped by
board).  Netlist identical to the annotated baseline.
Parts:
- J3001: value TO CTRL J903 -> TO CTRL J2002
Other:
- note added: "J3001: ribbon to the control board (J2002). The Powerpole is panel-mount, wired to J3101 on the Supply sheet."
- note removed: "J904: ribbon to the control board (J903). The Powerpole is panel-mount, wired to J1 on the Supply sheet."
Changed lines of the file:
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@@
 		(company "TBox")
 	)
-	(text "J904: ribbon to the control board (J903). The Powerpole is panel-mount, wired to J1 on the Supply sheet."
+	(text "J3001: ribbon to the control board (J2002). The Powerpole is panel-mount, wired to J3101 on the Supply sheet."
 		(exclude_from_sim no)
 		(at 20.32 24.13 0)
@@
 			)
 		)
-		(property "Value" "TO CTRL J903"
+		(property "Value" "TO CTRL J2002"
 			(at 66.04 121.92 0)
 			(show_name no)
