File: projects/tbox/kicad/txsum.kicad_sch (KiCad schematic)
At the start: 26 parts, among them Q2201 MMBT3904, Q2202 2N7002, SW2201 INTERCOM, U2201 OPA1678

Commit message: Rename refdes mentions in notes and docs to the board-coded numbering
Table-driven: the old->new map was derived from symbol UUIDs across the
annotation commit (619 instances, checked one-to-one and per board), and
only exact whole tokens from that table were replaced, in sheet notes,
connector Values, DESIGN.md, TODO.md and power_tree.json.  The one range
("J901-J904") and the one instance-specific ref in the shared Mute sheet
were rewritten by hand.  Power tree regenerated (loads now grouped by
board).  Netlist identical to the annotated baseline.
Other:
- note added: "Level pots RV2201/RV2202 (top panel) live here: PRE_x_OUT arrives at line level over the ribbon; the wiper feeds the sum locally."
- note added: "R2207 isolates the cap load"
- note removed: "Level pots RV201/RV301 (top panel) live here: PRE_x_OUT arrives at line level over the ribbon; the wiper feeds the sum locally."
- note removed: "R404 isolates the cap load"
Changed lines of the file:
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@@
 		(company "TBox")
 	)
-	(text "R404 isolates the cap load"
+	(text "R2207 isolates the cap load"
 		(exclude_from_sim no)
 		(at 20.32 83.82 0)
@@
 		)
 	)
-	(text "Level pots RV201/RV301 (top panel) live here: PRE_x_OUT arrives at line level over the ribbon; the wiper feeds the sum locally."
+	(text "Level pots RV2201/RV2202 (top panel) live here: PRE_x_OUT arrives at line level over the ribbon; the wiper feeds the sum locally."
 		(exclude_from_sim no)
 		(at 20.32 186.69 0)

Commit message: Footprint pass: every board part has a footprint, chosen parts carry MPNs
0603 base for R and C <= 1 uF, 0805 for 4u7, 1206 for 10 uF ceramics
(including the three non-polar coupling caps), 1210 for the 47 uF X7R;
electrolytics by can size; Keystone 5015 test points.  Panel parts per
the discussion: Switchcraft 35RAPC(2A/2B)H3 and Neutrik NRJ6HM-1-PRE
where the sleeve must bond to the panel, CUI SJ1-353xNG and Rean
NRJ6HF-1 where it must not; Alpha 9 mm pots, Bourns 3386 side-adjust
trims, C&K 7101 AV2 / 7201 V-bracket toggles, C&K PVA buttons, IDC
2x13 headers (vertical on front/rear, right-angle on control), JST XH
for the Powerpole pigtail (through-hole on purpose), Triad TY-250P
transformers, 0805 LEDs with light pipes.  J3207 (GND post) is a
panel part: on_board no.

kicad/tbox.pretty holds the four footprints with no stock equivalent,
each drawn from the vendor drawing and saying so in its description:
Switchcraft 35RAPC__H3 (rev J), C&K 7101 AV2 and 7201 V-bracket
patterns, Triad TY-250P (pads mapped to the Transformer_1P_1S symbol,
6-7 tied on copper for 1:1).

tools/check_footprints.py enforces the invariant.  Netlist unchanged
apart from J3207 leaving the board.
Parts:
- C2201, C2202, C2203, C2204, C2205: footprint (none) -> Capacitor_SMD:C_0603_1608Metric
- D2201: footprint (none) -> LED_SMD:LED_0805_2012Metric
- Q2201: footprint (none) -> Package_TO_SOT_SMD:SOT-23; MPN (none) -> MMBT3904
- Q2202: footprint (none) -> Package_TO_SOT_SMD:SOT-23; MPN (none) -> 2N7002
- R2201, R2202, R2203, R2204, R2205, R2206, R2207, R2208, R2209, R2210, R2211: footprint (none) -> Resistor_SMD:R_0603_1608Metric
- RV2201, RV2202: footprint (none) -> Potentiometer_THT:Potentiometer_Alpha_RD901F-40-00D_Single_Vertical; MPN (none) -> RD901F-40-15R1-A10K
- SW2201: footprint (none) -> Button_Switch_THT:SW_Push_2P1T_Toggle_CK_PVA1xxH2xxxxxxV2; MPN (none) -> PVA1EEH2xxxxxxV2 (momentary; height at layout)
- TP2201, TP2202, TP2203: footprint (none) -> TestPoint:TestPoint_Keystone_5015_Micro_Mini; MPN (none) -> 5015
- U2201: footprint (none) -> Package_SO:SOIC-8_3.9x4.9mm_P1.27mm; MPN (none) -> OPA1678IDR
Changed lines of the file:
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@@
 			)
 		)
-		(property "Footprint" ""
+		(property "Footprint" "Potentiometer_THT:Potentiometer_Alpha_RD901F-40-00D_Single_Vertical"
 			(at 175.26 121.92 0)
 			(hide yes)
@@
 					(size 1.27 1.27)
 				)
+			)
+		)
+		(property "MPN" "RD901F-40-15R1-A10K"
+			(at 175.26 121.92 0)
+			(effects
+				(font
+					(size 1.27 1.27)
+				)
+				(hide yes)
 			)
 		)
@@
 			)
 		)
-		(property "Footprint" ""
+		(property "Footprint" "Resistor_SMD:R_0603_1608Metric"
 			(at 111.76 78.74 0)
 			(hide yes)
@@
 			)
 		)
-		(property "Footprint" ""
+		(property "Footprint" "Package_SO:SOIC-8_3.9x4.9mm_P1.27mm"
 			(at 114.3 144.78 0)
 			(hide yes)
@@
 					(size 1.27 1.27)
 				)
+			)
+		)
+		(property "MPN" "OPA1678IDR"
+			(at 114.3 144.78 0)
+			(effects
+				(font
+					(size 1.27 1.27)
+				)
+				(hide yes)
 			)
 		)
@@
 			)
 		)
-		(property "Footprint" ""
+		(property "Footprint" "Package_TO_SOT_SMD:SOT-23"
 			(at 109.22 97.79 0)
 			(hide yes)
@@
 					(size 1.27 1.27)
 				)
+			)
+		)
+		(property "MPN" "2N7002"
+			(at 109.22 97.79 0)
+			(effects
+				(font
+					(size 1.27 1.27)
+				)
+				(hide yes)
 			)
 		)
@@
 			)
 		)
-		(property "Footprint" ""
+		(property "Footprint" "Package_TO_SOT_SMD:SOT-23"
 			(at 78.74 104.14 0)
 			(hide yes)
@@
 					(size 1.27 1.27)
 				)
+			)
+		)
+		(property "MPN" "MMBT3904"
+			(at 78.74 104.14 0)
+			(effects
+				(font
+					(size 1.27 1.27)
+				)
+				(hide yes)
 			)
 		)
@@
 			)
 		)
-		(property "Footprint" ""
+		(property "Footprint" "Resistor_SMD:R_0603_1608Metric"
 			(at 99.06 96.52 0)
 			(hide yes)
@@
 			)
 		)
-		(property "Footprint" ""
+		(property "Footprint" "Package_SO:SOIC-8_3.9x4.9mm_P1.27mm"
 			(at 83.82 144.78 0)
 			(hide yes)
@@
 					(size 1.27 1.27)
 				)
+			)
+		)
+		(property "MPN" "OPA1678IDR"
+			(at 83.82 144.78 0)
+			(effects
+				(font
+					(size 1.27 1.27)
+				)
+				(hide yes)
 			)
 		)
@@
 			)
 		)
-		(property "Footprint" ""
+		(property "Footprint" "Resistor_SMD:R_0603_1608Metric"
 			(at 46.99 60.96 0)
 			(hide yes)
@@
 			)
 		)
-		(property "Footprint" ""
+		(property "Footprint" "Capacitor_SMD:C_0603_1608Metric"
 			(at 48.26 109.22 0)
 			(hide yes)
@@
 			)
 		)
-		(property "Footprint" ""
+		(property "Footprint" "TestPoint:TestPoint_Keystone_5015_Micro_Mini"
 			(at 132.08 50.8 0)
 			(hide yes)
@@
 					(size 1.27 1.27)
 				)
+			)
+		)
+		(property "MPN" "5015"
+			(at 132.08 50.8 0)
+			(effects
+				(font
+					(size 1.27 1.27)
+				)
+				(hide yes)
 			)
 		)
@@
 			)
 		)
-		(property "Footprint" ""
+		(property "Footprint" "Capacitor_SMD:C_0603_1608Metric"
 			(at 66.04 76.2 0)
 			(hide yes)
@@
 			)
 		)
-		(property "Footprint" ""
+		(property "Footprint" "Button_Switch_THT:SW_Push_2P1T_Toggle_CK_PVA1xxH2xxxxxxV2"
 			(at 35.56 104.14 0)
 			(hide yes)
@@
 					(size 1.27 1.27)
 				)
+			)
+		)
+		(property "MPN" "PVA1EEH2xxxxxxV2 (momentary; height at layout)"
+			(at 35.56 104.14 0)
+			(effects
+				(font
+					(size 1.27 1.27)
+				)
+				(hide yes)
 			)
 		)
@@
 			)
 		)
-		(property "Footprint" ""
+		(property "Footprint" "Potentiometer_THT:Potentiometer_Alpha_RD901F-40-00D_Single_Vertical"
 			(at 175.26 96.52 0)
 			(hide yes)
@@
 					(size 1.27 1.27)
 				)
+			)
+		)
+		(property "MPN" "RD901F-40-15R1-A10K"
+			(at 175.26 96.52 0)
+			(effects
+				(font
+					(size 1.27 1.27)
+				)
+				(hide yes)
 			)
 		)
@@
 			)
 		)
-		(property "Footprint" ""
+		(property "Footprint" "TestPoint:TestPoint_Keystone_5015_Micro_Mini"
 			(at 184.15 114.3 0)
 			(hide yes)
@@
 					(size 1.27 1.27)
 				)
+			)
+		)
+		(property "MPN" "5015"
+			(at 184.15 114.3 0)
+			(effects
+				(font
+					(size 1.27 1.27)
+				)
+				(hide yes)
 			)
 		)
@@
 			)
 		)
-		(property "Footprint" ""
+		(property "Footprint" "Capacitor_SMD:C_0603_1608Metric"
 			(at 105.41 140.97 0)
 			(hide yes)
@@
 			)
 		)
-		(property "Footprint" ""
+		(property "Footprint" "Capacitor_SMD:C_0603_1608Metric"
 			(at 36.83 60.96 0)
 			(hide yes)
@@
 			)
 		)
-		(property "Footprint" ""
+		(property "Footprint" "Resistor_SMD:R_0603_1608Metric"
 			(at 81.28 91.44 0)
 			(hide yes)
@@
 			)
 		)
-		(property "Footprint" ""
+		(property "Footprint" "Resistor_SMD:R_0603_1608Metric"
 			(at 43.18 99.06 0)
 			(hide yes)
@@
 			)
 		)
-		(property "Footprint" ""
+		(property "Footprint" "Resistor_SMD:R_0603_1608Metric"
 			(at 57.15 104.14 0)
 			(hide yes)
@@
 			)
 		)
-		(property "Footprint" ""
+		(property "Footprint" "Resistor_SMD:R_0603_1608Metric"
 			(at 127 55.88 0)
 			(hide yes)
@@
 			)
 		)
-		(property "Footprint" ""
+		(property "Footprint" "TestPoint:TestPoint_Keystone_5015_Micro_Mini"
 			(at 184.15 88.9 0)
 			(hide yes)
@@
 					(size 1.27 1.27)
 				)
+			)
+		)
+		(property "MPN" "5015"
+			(at 184.15 88.9 0)
+			(effects
+				(font
+					(size 1.27 1.27)
+				)
+				(hide yes)
 			)
 		)
@@
 			)
 		)
-		(property "Footprint" ""
+		(property "Footprint" "Resistor_SMD:R_0603_1608Metric"
 			(at 46.99 53.34 0)
 			(hide yes)
@@
 			)
 		)
-		(property "Footprint" ""
+		(property "Footprint" "Resistor_SMD:R_0603_1608Metric"
 			(at 66.04 66.04 0)
 			(hide yes)
@@
 			)
 		)
-		(property "Footprint" ""
+		(property "Footprint" "Resistor_SMD:R_0603_1608Metric"
 			(at 81.28 50.8 0)
 			(hide yes)
@@
 			)
 		)
-		(property "Footprint" ""
+		(property "Footprint" "Package_SO:SOIC-8_3.9x4.9mm_P1.27mm"
 			(at 66.04 50.8 0)
 			(hide yes)
@@
 					(size 1.27 1.27)
 				)
+			)
+		)
+		(property "MPN" "OPA1678IDR"
+			(at 66.04 50.8 0)
+			(effects
+				(font
+					(size 1.27 1.27)
+				)
+				(hide yes)
 			)
 		)
@@
 			)
 		)
-		(property "Footprint" ""
+		(property "Footprint" "LED_SMD:LED_0805_2012Metric"
 			(at 111.76 87.63 0)
 			(hide yes)
@@
 			)
 		)
-		(property "Footprint" ""
+		(property "Footprint" "Capacitor_SMD:C_0603_1608Metric"
 			(at 36.83 53.34 0)
 			(hide yes)
@@
 			)
 		)
-		(property "Footprint" ""
+		(property "Footprint" "Resistor_SMD:R_0603_1608Metric"
 			(at 73.66 96.52 0)
 			(hide yes)
