File: projects/tbox/kicad/tbox.kicad_pcb (KiCad board)
At the start: 4 copper layers, 300 x 270 mm, 355 parts, among them J1001 PHONES A 3.5, J1002 PHONES A 1/4, J1003 PHONES B 3.5, J1004 PHONES B 1/4, J1005 TO CTRL J2001, J1101 MIC 3.5, J1102 MIC 1/4, J1103 HEADSET, J1104 SPARE, J1301 MIC 3.5, J1302 MIC 1/4, J1303 HEADSET, J1304 SPARE, J2001 TO FRONT J1005, J2002 TO REAR J3001, J2501 PWR IN (panel Powerpole), J3001 TO CTRL J2002, J3201 PTT A 3.5, J3202 PTT A 1/4, J3203 PTT B 3.5, J3204 PTT B 1/4, J3205 CW SPARE, J3206 RIG DE-9, J3301 LINE L SRC, J3302 LINE R SRC, J3303 LINE OUT, Q2101 2N7002, Q2102 2N7002, Q2103 2N7002, Q2104 2N7002, Q2105 2N7002, Q2106 2N7002, Q2107 2N7002, Q2201 MMBT3904, Q2202 2N7002, Q3201 2N7002, SW2101 PTT A, SW2102 PTT B, SW2103 OVERRIDE, SW2104 MUTE A, SW2105 MUTE B, SW2201 INTERCOM, SW3201 GAIN A HI, SW3202 GAIN B HI, SW3203 BIAS A, SW3204 BIAS B, T3301 TY-250P, T3302 TY-250P, U1101 OPA1678, U1102 TS12A12511, U1201 TS12A12511, U1301 OPA1678, U1302 TS12A12511, U1401 TS12A12511, U2201 OPA1678, U2301 TS12A12511, U2401 NJM4556A, U2402 OPA1678, U2403 NJM4556A, U2501 ADP7142AUJZ-5.0, U2502 OPA1678, U2503 TPS7A4701, U3301 OPA1678, U3302 OPA1678, U3401 OPA1678

Commit message: Update PCB from Schematic: TY-250P pin names relinked
Connections:
- C3310 pad 2: Net-(T3301-AA) -> Net-(T3301-P1)
- C3311 pad 2: Net-(T3302-AA) -> Net-(T3302-P1)
- FB3301 pad 1: Net-(T3301-SB) -> Net-(T3301-S1)
- FB3302 pad 1: Net-(T3302-SB) -> Net-(T3302-S1)
- T3301 pad 3: (no net) -> unconnected-(T3301-CT-Pad3)
- T3302 pad 3: (no net) -> unconnected-(T3302-CT-Pad3)
Changed lines of the file:
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@@
 			(layers "F.Cu" "F.Mask" "F.Paste")
 			(roundrect_rratio 0.15625)
-			(net "Net-(T3302-AA)")
+			(net "Net-(T3302-P1)")
 			(pintype "passive")
 		)
@@
 			)
 		)
+		(property "MPN" "TY-250P"
+			(at 0 0 0)
+			(unlocked yes)
+			(layer "F.Fab")
+			(hide yes)
+			(effects
+				(font
+					(size 1 1)
+					(thickness 0.15)
+				)
+			)
+		)
 		(sheetname "/Rear Board/Rig Out/")
 		(sheetfile "rigout.kicad_sch")
+		(units
+			(unit
+				(name "A")
+				(pins "2" "3" "4" "5" "6" "7" "8")
+			)
+		)
 		(attr through_hole)
 		(duplicate_pad_numbers_are_jumpers no)
@@
 			(remove_unused_layers no)
 			(net "Net-(T3302-P1)")
+			(pinfunction "P1_2")
+			(pintype "passive")
 		)
 		(pad "3" thru_hole circle
@@
 			(layers "*.Cu" "*.Mask")
 			(remove_unused_layers no)
+			(net "unconnected-(T3302-CT-Pad3)")
+			(pinfunction "CT_3")
+			(pintype "passive+no_connect")
 		)
 		(pad "4" thru_hole circle
@@
 			(remove_unused_layers no)
 			(net "GND")
+			(pinfunction "P2_4")
+			(pintype "passive")
 		)
 		(pad "5" thru_hole circle
@@
 			(remove_unused_layers no)
 			(net "Net-(T3302-S1)")
+			(pinfunction "S1_5")
+			(pintype "passive")
 		)
 		(pad "6" thru_hole circle
@@
 			(remove_unused_layers no)
 			(net "Net-(T3302-S1b)")
+			(pinfunction "S1b_6")
+			(pintype "passive")
 		)
 		(pad "7" thru_hole circle
@@
 			(remove_unused_layers no)
 			(net "Net-(T3302-S1b)")
+			(pinfunction "S2b_7")
+			(pintype "passive")
 		)
 		(pad "8" thru_hole circle
@@
 			(remove_unused_layers no)
 			(net "/Rear Board/Rig Out/LOUT_RET")
+			(pinfunction "S2_8")
+			(pintype "passive")
 		)
 		(embedded_fonts no)
@@
 			(layers "F.Cu" "F.Mask" "F.Paste")
 			(roundrect_rratio 0.25)
-			(net "Net-(T3302-SB)")
+			(net "Net-(T3302-S1)")
 			(pintype "passive")
 		)
@@
 			)
 		)
+		(property "MPN" "TY-250P"
+			(at 0 0 0)
+			(unlocked yes)
+			(layer "F.Fab")
+			(hide yes)
+			(effects
+				(font
+					(size 1 1)
+					(thickness 0.15)
+				)
+			)
+		)
 		(sheetname "/Rear Board/Rig Out/")
 		(sheetfile "rigout.kicad_sch")
+		(units
+			(unit
+				(name "A")
+				(pins "2" "3" "4" "5" "6" "7" "8")
+			)
+		)
 		(attr through_hole)
 		(duplicate_pad_numbers_are_jumpers no)
@@
 			(remove_unused_layers no)
 			(net "Net-(T3301-P1)")
+			(pinfunction "P1_2")
+			(pintype "passive")
 		)
 		(pad "3" thru_hole circle
@@
 			(layers "*.Cu" "*.Mask")
 			(remove_unused_layers no)
+			(net "unconnected-(T3301-CT-Pad3)")
+			(pinfunction "CT_3")
+			(pintype "passive+no_connect")
 		)
 		(pad "4" thru_hole circle
@@
 			(remove_unused_layers no)
 			(net "GND")
+			(pinfunction "P2_4")
+			(pintype "passive")
 		)
 		(pad "5" thru_hole circle
@@
 			(remove_unused_layers no)
 			(net "Net-(T3301-S1)")
+			(pinfunction "S1_5")
+			(pintype "passive")
 		)
 		(pad "6" thru_hole circle
@@
 			(remove_unused_layers no)
 			(net "Net-(T3301-S1b)")
+			(pinfunction "S1b_6")
+			(pintype "passive")
 		)
 		(pad "7" thru_hole circle
@@
 			(remove_unused_layers no)
 			(net "Net-(T3301-S1b)")
+			(pinfunction "S2b_7")
+			(pintype "passive")
 		)
 		(pad "8" thru_hole circle
@@
 			(remove_unused_layers no)
 			(net "/Rear Board/Rig Out/LOUT_RET")
+			(pinfunction "S2_8")
+			(pintype "passive")
 		)
 		(embedded_fonts no)
@@
 			(layers "F.Cu" "F.Mask" "F.Paste")
 			(roundrect_rratio 0.25)
-			(net "Net-(T3301-SB)")
+			(net "Net-(T3301-S1)")
 			(pintype "passive")
 		)
@@
 			(layers "F.Cu" "F.Mask" "F.Paste")
 			(roundrect_rratio 0.15625)
-			(net "Net-(T3301-AA)")
+			(net "Net-(T3301-P1)")
 			(pintype "passive")
 		)
