File: projects/tbox/kicad/reario.kicad_sch (KiCad schematic)
At the start: 42 parts, among them J3201 PTT A 3.5, J3202 PTT A 1/4, J3203 PTT B 3.5, J3204 PTT B 1/4, J3205 CW SPARE, J3206 RIG DE-9, J3207 GND POST, Q3201 2N7002, SW3201 GAIN A HI, SW3202 GAIN B HI, SW3203 BIAS A, SW3204 BIAS B

Commit message: Review design changes: chassis returns, OPA1622 phones amps, RX-in protection, supervisor, mute fade, gains, BLEND buffer, jack-side protection, mic-jack bias
Decisions Q1-Q9 from the 2026-09-08 adversarial review:
- Q1 (D): phones jack sleeves and TRRS ring 2 on CHASSIS; GND-CHASSIS
  ties per board (NT1001 front at the headset jacks, NT2401 control at
  the phones amps, NT3201 rear) with chassis studs H1001/H2401; phones
  return rides the chassis, never the ribbon ground.
- Q2 (B'): U2401/U2403 NJM4556A -> OPA1622 (new tbox symbol, VSON-10),
  build-out 10R -> 3R3, EN from PWR_OK.
- Q3 (A+C): RX-in coupling caps non-polar 10u, 2k2 series, 1N4148W
  clamps to the rails at the op-amp inputs (SMAJ15CA stays at the jack).
- Q4 (B): TPS3808G01 supervisor on +9 V (7.5 V, ~1.2 s) -> PWR_OK;
  MUTE_HOLD inverter replaces the RC hold, shunts PTT_ACTIVE; Q3201 gets
  a 100k gate pull-down.
- Q5 (A): mute fades (2k2 + back-to-back 2N7002 shunt to Vref, ~5 ms)
  before the TS12A12511 switches (~30 ms, immediate release).
- Q6 (A): preamp LO +28 / HI +40 dB (R1104 430R, R1106 3k3).
- Q7 (A): BLEND is an inverting summer on U3301B (R3318 22k, C3317).
- Q8 (C): phones RF filters move to the front board at the jacks; SP724
  arrays on every front jack contact and the rear PTT inputs; SMAJ15CA
  across each isolated line-out secondary.
- Q9 (B'): 3.5 mm mic jack tip carries the mic, tip and ring both get
  2k2 bias (R1109/C1109).
DESIGN.md, LEVELS.md and TODO.md updated; ERC 0, check_sch/boards/
footprints/power clean; power tree regenerated.
Parts:
- added R3211: 100k, Resistor_SMD:R_0603_1608Metric, symbol Device:R
- added U3201: SP724, Package_TO_SOT_SMD:SOT-23-6, symbol tbox:SP724
Connections:
- net +9V: now also U3201.5 (V+)
- net GND: now also R3211.2, U3201.2 (V-)
- net PTT_A_IN: now also U3201.1 (IN1)
- net PTT_B_IN: now also U3201.3 (IN2)
- net Q3201_G: now reaches Q3201.1 (G), R3203.2
- net Q3201_G: now also R3211.1
- no-connect marks 0 -> 2

Commit message: Review 2: load maxima and the resistor rule
- Op-amp maxima from the datasheets: OPA1678 duals 4/6 (5.6 mA IQ over
  temperature), line drivers 4/10, OPA1622 6/101 (8.4 mA IQ + two
  145 mA-peak class-B channels).
- Every resistor with an end on a rail now needs Load_mA (Vref returns
  and the ADP7142 output RC exempt): R2122, R2501, R2505, R2507,
  R3209/R3210 (1k gain-select pull-ups, 9 mA each when closed),
  R3201/R3202 PTT pull-ups annotated.
- Load_mA syntax is strict (n or n/m).
- RAW_13V8 capability 400 mA (1812L050 hold at 50 C), not 500.
- C3401/C3402 10u X7R 25V, GRM31CR71E106KA12L.
Parts:
- R3201, R3202: Load_mA (none) -> 0/0.9; Load_rail (none) -> +9V
- R3209, R3210: Load_mA (none) -> 0/9
Changed lines of the file:
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@@
 			)
 		)
+		(property "Load_mA" "0/9"
+			(at 189.23 128.27 0)
+			(show_name no)
+			(do_not_autoplace no)
+			(hide yes)
+			(effects
+				(font
+					(size 1.27 1.27)
+				)
+			)
+		)
 		(property "Footprint" "Resistor_SMD:R_0603_1608Metric"
 			(at 189.23 128.27 0)
@@
 			)
 		)
+		(property "Load_mA" "0/0.9"
+			(at 52.07 93.98 0)
+			(show_name no)
+			(do_not_autoplace no)
+			(hide yes)
+			(effects
+				(font
+					(size 1.27 1.27)
+				)
+			)
+		)
+		(property "Load_rail" "+9V"
+			(at 52.07 93.98 0)
+			(show_name no)
+			(do_not_autoplace no)
+			(hide yes)
+			(effects
+				(font
+					(size 1.27 1.27)
+				)
+			)
+		)
 		(property "Footprint" "Resistor_SMD:R_0603_1608Metric"
 			(at 52.07 93.98 0)
@@
 			)
 		)
+		(property "Load_mA" "0/9"
+			(at 189.23 138.43 0)
+			(show_name no)
+			(do_not_autoplace no)
+			(hide yes)
+			(effects
+				(font
+					(size 1.27 1.27)
+				)
+			)
+		)
 		(property "Footprint" "Resistor_SMD:R_0603_1608Metric"
 			(at 189.23 138.43 0)
@@
 			)
 		)
+		(property "Load_mA" "0/0.9"
+			(at 52.07 53.34 0)
+			(show_name no)
+			(do_not_autoplace no)
+			(hide yes)
+			(effects
+				(font
+					(size 1.27 1.27)
+				)
+			)
+		)
+		(property "Load_rail" "+9V"
+			(at 52.07 53.34 0)
+			(show_name no)
+			(do_not_autoplace no)
+			(hide yes)
+			(effects
+				(font
+					(size 1.27 1.27)
+				)
+			)
+		)

Commit message: Review 2 design decisions: mute cell sequencing, phones precharge, non-inverting BLEND, chassis RF returns, SP724 bypass and placement, TVS ahead of the bead, load and level updates
Q1  Mute cell: MUTE is a source-only OR with a 100k pull-down; a 2N7002
    inverter (Q1203) and sink (Q1204) pull SW_CTL hard low on release so
    the SPDT reconnects under the shunt, the fade gate charges through
    D1201/47k and bleeds through 470k (~50 ms); nothing discharges
    through MUTE any more.
Q2  1k from Vref on each OPA1622 output node (R2425-R2428) precharges
    the 470u phones caps during the hold.
Q3  Fade resistor 220R (all three instances): 0.2 dB insertion, TX_MIX
    level within 0.3 dB of the line-out jumpering.
Q4  LO stays +28 dB; -28 dBV desk mics declared out of scope in LEVELS.
Q5  SP724s stay on the rails, each with its own 100n (C1110/C1111/C1007/
    C3208 + B copies), placed behind their jack (place_panel ATTACH,
    check_placement 20 mm rule); mic RF caps C1101/C1109 return to
    CHASSIS.
Q6  Supply source envelope documented (bench/rig PSU, fused at source);
    SMBJ18A moved to the post-Schottky node ahead of FB2501; TODO for
    mobile use.
Q7  BLEND is a non-inverting summer (22k/22k into +IN, R3319 22k to Vref
    for a gain of 2), in phase with the RX selections.
Q8  Key-inhibit delay through MUTE_HOLD accepted and documented.
Q9  Beads are Murata BLM21PG601SN1D (600 R, 1.4 A, 0.14 R; datasheet
    added); PVA ordering code TODO names the panel gap that sets it.
Also: setup_pcb cuts the SJ-43514 4.5 x 1.3 mm edge notches at the jacks
on the board; supervisor hold text 1.3 s.
Parts:
- added C3208: 100n, Capacitor_SMD:C_0603_1608Metric, symbol Device:C
- FB3201, FB3202, FB3203, FB3204, FB3205, FB3206, FB3207: MPN (none) -> BLM21PG601SN1D
Connections:
- net +9V: now also C3208.1
- net GND: now also C3208.2
